File: ecad/helios/LED_driver/_saved_LED_driver.sch (KiCad schematic (older format))
At the start: 21 parts, among them J1 Conn_02x04_Top_Bottom, J2 Conn_02x03_Top_Bottom, J3 Conn_02x04_Top_Bottom, U1 UA9637

Commit message: Adds Pull-Down resistor
We do not want the LEDs to be turned ON on a UC reset.
Parts:
- gave numbers to parts that had none: 2
Changed lines of the file:
@@
 $EndComp
 $Comp
-L GND #PWR01
+L GND #PWR11
 U 1 1 5AAA77E2
 P 7100 4250
-F 0 "#PWR01" H 7100 4000 50  0001 C CNN
+F 0 "#PWR11" H 7100 4000 50  0001 C CNN
 F 1 "GND" H 7100 4100 50  0000 C CNN
 F 2 "" H 7100 4250 50  0001 C CNN
@@
 $EndComp
 $Comp
-L GND #PWR02
+L GND #PWR16
 U 1 1 5AAA7DD2
 P 7100 5050
-F 0 "#PWR02" H 7100 4800 50  0001 C CNN
+F 0 "#PWR16" H 7100 4800 50  0001 C CNN
 F 1 "GND" H 7100 4900 50  0000 C CNN
 F 2 "" H 7100 5050 50  0001 C CNN
@@
 $EndComp
 $Comp
-L GND #PWR03
+L GND #PWR19
 U 1 1 5AAA81A1
 P 7100 5850
-F 0 "#PWR03" H 7100 5600 50  0001 C CNN
+F 0 "#PWR19" H 7100 5600 50  0001 C CNN
 F 1 "GND" H 7100 5700 50  0000 C CNN
 F 2 "" H 7100 5850 50  0001 C CNN
@@
 $EndComp
 $Comp
-L GND #PWR04
+L GND #PWR12
 U 1 1 5AAAA97D
 P 7500 4250
-F 0 "#PWR04" H 7500 4000 50  0001 C CNN
+F 0 "#PWR12" H 7500 4000 50  0001 C CNN
 F 1 "GND" H 7500 4100 50  0000 C CNN
 F 2 "" H 7500 4250 50  0001 C CNN
@@
 $EndComp
 $Comp
-L GND #PWR05
+L GND #PWR17
 U 1 1 5AAAAB6E
 P 7500 5050
-F 0 "#PWR05" H 7500 4800 50  0001 C CNN
+F 0 "#PWR17" H 7500 4800 50  0001 C CNN
 F 1 "GND" H 7500 4900 50  0000 C CNN
 F 2 "" H 7500 5050 50  0001 C CNN
@@
 $EndComp
 $Comp
-L GND #PWR06
+L GND #PWR20
 U 1 1 5AAAACC3
 P 7500 5850
-F 0 "#PWR06" H 7500 5600 50  0001 C CNN
+F 0 "#PWR20" H 7500 5600 50  0001 C CNN
 F 1 "GND" H 7500 5700 50  0000 C CNN
 F 2 "" H 7500 5850 50  0001 C CNN
@@
 $EndSheet
 $Comp
-L +36V #PWR07
+L +36V #PWR9
 U 1 1 5AB15ABE
 P 6300 3550
-F 0 "#PWR07" H 6300 3400 50  0001 C CNN
+F 0 "#PWR9" H 6300 3400 50  0001 C CNN
 F 1 "+36V" H 6300 3690 50  0000 C CNN
 F 2 "" H 6300 3550 50  0001 C CNN
@@
 $EndComp
 $Comp
-L GND #PWR08
+L GND #PWR3
 U 1 1 5AB4B54E
 P 3350 3150
-F 0 "#PWR08" H 3350 2900 50  0001 C CNN
+F 0 "#PWR3" H 3350 2900 50  0001 C CNN
 F 1 "GND" H 3350 3000 50  0000 C CNN
 F 2 "" H 3350 3150 50  0001 C CNN
@@
 $EndComp
 $Comp
-L GND #PWR09
+L GND #PWR13
 U 1 1 5AB4B6FD
 P 3350 4400
-F 0 "#PWR09" H 3350 4150 50  0001 C CNN
+F 0 "#PWR13" H 3350 4150 50  0001 C CNN
 F 1 "GND" H 3350 4250 50  0000 C CNN
 F 2 "" H 3350 4400 50  0001 C CNN
@@
 $EndComp
 $Comp
-L +5V #PWR010
+L +5V #PWR8
 U 1 1 5AB4B802
 P 3350 3550
-F 0 "#PWR010" H 3350 3400 50  0001 C CNN
+F 0 "#PWR8" H 3350 3400 50  0001 C CNN
 F 1 "+5V" H 3350 3690 50  0000 C CNN
 F 2 "" H 3350 3550 50  0001 C CNN
@@
 $EndComp
 $Comp
-L +5V #PWR011
+L +5V #PWR1
 U 1 1 5AB4BE6D
 P 3350 2300
-F 0 "#PWR011" H 3350 2150 50  0001 C CNN
+F 0 "#PWR1" H 3350 2150 50  0001 C CNN
 F 1 "+5V" H 3350 2440 50  0000 C CNN
 F 2 "" H 3350 2300 50  0001 C CNN
@@
 $EndComp
 $Comp
-L GND #PWR012
+L GND #PWR2
 U 1 1 5AB4C0C2
 P 3950 2500
-F 0 "#PWR012" H 3950 2250 50  0001 C CNN
+F 0 "#PWR2" H 3950 2250 50  0001 C CNN
 F 1 "GND" H 3950 2350 50  0000 C CNN
 F 2 "" H 3950 2500 50  0001 C CNN
@@
 $EndComp
 $Comp
-L GND #PWR013
+L GND #PWR10
 U 1 1 5AB4CC17
 P 3950 3750
-F 0 "#PWR013" H 3950 3500 50  0001 C CNN
+F 0 "#PWR10" H 3950 3500 50  0001 C CNN
 F 1 "GND" H 3950 3600 50  0000 C CNN
 F 2 "" H 3950 3750 50  0001 C CNN
@@
 	1550 2850 2850 2850
 $Comp
-L GND #PWR014
+L GND #PWR18
 U 1 1 5AB53D95
 P 3950 5550
-F 0 "#PWR014" H 3950 5300 50  0001 C CNN
+F 0 "#PWR18" H 3950 5300 50  0001 C CNN
 F 1 "GND" H 3950 5400 50  0000 C CNN
 F 2 "" H 3950 5550 50  0001 C CNN
@@
 	2650 5850 3250 5850
 $Comp
-L GND #PWR015
+L GND #PWR21
 U 1 1 5AB57015
 P 3950 6150
-F 0 "#PWR015" H 3950 5900 50  0001 C CNN
+F 0 "#PWR21" H 3950 5900 50  0001 C CNN
 F 1 "GND" H 3950 6000 50  0000 C CNN
 F 2 "" H 3950 6150 50  0001 C CNN
@@
 Connection ~ 2300 2850
 $Comp
-L GND #PWR016
+L GND #PWR4
 U 1 1 5AB95930
 P 2300 3350
-F 0 "#PWR016" H 2300 3100 50  0001 C CNN
+F 0 "#PWR4" H 2300 3100 50  0001 C CNN
 F 1 "GND" H 2300 3200 50  0000 C CNN
 F 2 "" H 2300 3350 50  0001 C CNN
@@
 	2300 3350 2300 3250
 $Comp
-L GND #PWR017
+L GND #PWR5
 U 1 1 5AB95ABB
 P 2600 3350
-F 0 "#PWR017" H 2600 3100 50  0001 C CNN
+F 0 "#PWR5" H 2600 3100 50  0001 C CNN
 F 1 "GND" H 2600 3200 50  0000 C CNN
 F 2 "" H 2600 3350 50  0001 C CNN
@@
 $EndComp
 $Comp
-L GND #PWR018
+L GND #PWR14
 U 1 1 5AB964BA
 P 2300 4600
-F 0 "#PWR018" H 2300 4350 50  0001 C CNN
+F 0 "#PWR14" H 2300 4350 50  0001 C CNN
 F 1 "GND" H 2300 4450 50  0000 C CNN
 F 2 "" H 2300 4600 50  0001 C CNN
@@
 	2300 4600 2300 4500
 $Comp
-L GND #PWR019
+L GND #PWR15
 U 1 1 5AB964C1
 P 2600 4600
-F 0 "#PWR019" H 2600 4350 50  0001 C CNN
+F 0 "#PWR15" H 2600 4350 50  0001 C CNN
 F 1 "GND" H 2600 4450 50  0000 C CNN
 F 2 "" H 2600 4600 50  0001 C CNN
@@
 Connection ~ 2300 4100
 $Comp
-L R R?
+L R R19
 U 1 1 5ABBCBC8
 P 6950 3250
-F 0 "R?" V 7030 3250 50  0000 C CNN
+F 0 "R19" V 7030 3250 50  0000 C CNN
 F 1 "100k" V 6950 3250 50  0000 C CNN
 F 2 "Resistors_SMD:R_0603" V 6880 3250 50  0001 C CNN
@@
 $EndComp
 $Comp
-L R R?
+L R R26
 U 1 1 5ABBD07A
 P 7250 3250
-F 0 "R?" V 7330 3250 50  0000 C CNN
+F 0 "R26" V 7330 3250 50  0000 C CNN
 F 1 "100k" V 7250 3250 50  0000 C CNN
 F 2 "Resistors_SMD:R_0603" V 7180 3250 50  0001 C CNN
@@
 Connection ~ 7250 2950
 $Comp
-L GND #PWR?
+L GND #PWR6
 U 1 1 5ABBD303
 P 6950 3450
-F 0 "#PWR?" H 6950 3200 50  0001 C CNN
+F 0 "#PWR6" H 6950 3200 50  0001 C CNN
 F 1 "GND" H 6950 3300 50  0000 C CNN
 F 2 "" H 6950 3450 50  0001 C CNN
@@
 $EndComp
 $Comp
-L GND #PWR?
+L GND #PWR7
 U 1 1 5ABBD3DA
 P 7250 3450
-F 0 "#PWR?" H 7250 3200 50  0001 C CNN
+F 0 "#PWR7" H 7250 3200 50  0001 C CNN
 F 1 "GND" H 7250 3300 50  0000 C CNN
 F 2 "" H 7250 3450 50  0001 C CNN
