File: ecad/helios/LED_driver/Controller.sch (KiCad schematic (older format))
At the start: 14 parts, among them J4 M20-8760342, SW1 SW_Push, U7 ATMEGA328PB-AU, Y1 16MHz

Commit message: wip LED Driver revB
Parts:
- Y1: value 16MHz -> 20MHz; footprint Crystals:Crystal_SMD_SeikoEpson_FA238-4pin_3.2x2.5mm -> Crystals:Crystal_SMD_Abracon_ABM8G-4pin_3.2x2.5mm; Part Number FA-238 16.0000MB-C3 -> ABM8G-20.000MHZ-18-D2Y-T
Connections:
- net EN36V: now also U7.10 ((OC0A/AIN0/PTCXY)PD6); no longer U7.9 ((OC0B/T1/PTCXY)PD5)
- net FLASH_IN: now also U7.32 ((OC3B/OC4B/INT0/PTCXY)PD2)
- net IR_ON: now also U7.9 ((OC0B/T1/PTCXY)PD5); no longer U7.10 ((OC0A/AIN0/PTCXY)PD6)
Changed lines of the file:
@@
 Wire Wire Line
 	4400 3300 5450 3300
+Text HLabel 4750 5200 2    60   Output ~ 0
+IR_ON
 Text HLabel 4750 5300 2    60   Output ~ 0
-IR_ON
-Text HLabel 4750 5200 2    60   Output ~ 0
 EN36V
 Connection ~ 10000 3600
@@
 V36_MEASURE
 Wire Wire Line
-	4400 5200 4750 5200
+	4400 5300 4750 5300
 Wire Wire Line
 	6100 4250 10000 4250
@@
 	10000 4250 10000 3350
 Wire Wire Line
-	4400 5300 4750 5300
+	4400 5200 4750 5200
 Wire Wire Line
 	4400 4700 4800 4700
@@
 P 6700 3650
 F 0 "Y1" V 6950 3750 50  0000 L CNN
-F 1 "16MHz" V 6850 3750 50  0000 L CNN
-F 2 "Crystals:Crystal_SMD_SeikoEpson_FA238-4pin_3.2x2.5mm" H 6700 3650 50  0001 C CNN
+F 1 "20MHz" V 6850 3750 50  0000 L CNN
+F 2 "Crystals:Crystal_SMD_Abracon_ABM8G-4pin_3.2x2.5mm" H 6700 3650 50  0001 C CNN
 F 3 "" H 6700 3650 50  0001 C CNN
-F 4 "FA-238 16.0000MB-C3" H 6700 3650 60  0001 C CNN "Part Number"
+F 4 "ABM8G-20.000MHZ-18-D2Y-T" H 6700 3650 60  0001 C CNN "Part Number"
 	1    6700 3650
 	0    1    1    0
@@
 Text Label 5650 3700 0    60   ~ 0
 XTAL-
+Wire Wire Line
+	4400 4900 4550 4900
+Wire Wire Line
+	4550 4900 4550 5000
+Connection ~ 4550 5000
 $EndSCHEMATC
