File: ecad/helios/LED_driver/Power_Management.sch (KiCad schematic (older format))
At the start: 15 parts, among them Q1 Q_PMOS_GDS, Q2 Q_PMOS_GDS, U5 TPS1H100AQ, U6 LM2936-5.0

Commit message: Finishes the schematics
Parts:
- D7: footprint (none) -> FORT:D_SOT-23_KAN; Part Number LM4040 -> LM4040DIM3X-10/NOPB
- U5: footprint (none) -> FORT:HTSSOP-14-1EP_4.4x6.5mm_Pitch0.65mm_ThermalPad; Part Number (none) -> TPS1H100AQPWPRQ1
- U6: footprint (none) -> TO_SOT_Packages_SMD:SOT-223-3Lead_TabPin2; Part Number (none) -> LM2936MPX-5.0/NOPB
Changed lines of the file:
@@
 F 0 "U5" H 5250 1700 60  0000 C CNN
 F 1 "TPS1H100AQ" H 5450 2750 60  0000 C CNN
-F 2 "" H 5400 2350 60  0001 C CNN
+F 2 "FORT:HTSSOP-14-1EP_4.4x6.5mm_Pitch0.65mm_ThermalPad" H 5400 2350 60  0001 C CNN
 F 3 "" H 5400 2350 60  0001 C CNN
+F 4 "TPS1H100AQPWPRQ1" H 5450 2250 60  0001 C CNN "Part Number"
 	1    5450 2250
 	1    0    0    -1
 $EndComp
 $Comp
-L GND #PWR021
+L GND #PWR022
 U 1 1 5AB122DC
 P 5400 3300
-F 0 "#PWR021" H 5400 3050 50  0001 C CNN
+F 0 "#PWR022" H 5400 3050 50  0001 C CNN
 F 1 "GND" H 5400 3150 50  0000 C CNN
 F 2 "" H 5400 3300 50  0001 C CNN
@@
 F 0 "D7" H 3400 1600 50  0000 C CNN
 F 1 "10V" H 3400 1400 50  0000 C CNN
-F 2 "" H 3400 1500 50  0001 C CNN
+F 2 "FORT:D_SOT-23_KAN" H 3400 1500 50  0001 C CNN
 F 3 "" H 3400 1500 50  0001 C CNN
-F 4 "LM4040" H 3400 1500 60  0001 C CNN "Part Number"
+F 4 "LM4040DIM3X-10/NOPB" H 3400 1500 60  0001 C CNN "Part Number"
 	1    3400 1500
 	0    1    1    0
 $EndComp
 $Comp
-L GND #PWR022
+L GND #PWR023
 U 1 1 5AB12A91
 P 2950 2300
-F 0 "#PWR022" H 2950 2050 50  0001 C CNN
+F 0 "#PWR023" H 2950 2050 50  0001 C CNN
 F 1 "GND" H 2950 2150 50  0000 C CNN
 F 2 "" H 2950 2300 50  0001 C CNN
@@
 F 0 "U6" H 4500 5725 50  0000 C CNN
 F 1 "LM2936-5.0" H 4650 5725 50  0000 L CNN
-F 2 "" H 4650 5825 50  0001 C CIN
+F 2 "TO_SOT_Packages_SMD:SOT-223-3Lead_TabPin2" H 4650 5825 50  0001 C CIN
 F 3 "" H 4650 5550 50  0001 C CNN
+F 4 "LM2936MPX-5.0/NOPB" H 4650 5600 60  0001 C CNN "Part Number"
 	1    4650 5600
 	1    0    0    -1
@@
 VS6
 $Comp
-L GND #PWR023
+L GND #PWR024
 U 1 1 5AB3DBC2
 P 4850 6400
-F 0 "#PWR023" H 4850 6150 50  0001 C CNN
+F 0 "#PWR024" H 4850 6150 50  0001 C CNN
 F 1 "GND" H 4850 6250 50  0000 C CNN
 F 2 "" H 4850 6400 50  0001 C CNN
@@
 $EndComp
 $Comp
-L +5V #PWR024
+L +5V #PWR025
 U 1 1 5AB3EB47
 P 5850 5450
-F 0 "#PWR024" H 5850 5300 50  0001 C CNN
+F 0 "#PWR025" H 5850 5300 50  0001 C CNN
 F 1 "+5V" H 5850 5590 50  0000 C CNN
 F 2 "" H 5850 5450 50  0001 C CNN
@@
 $EndComp
 $Comp
-L +36V #PWR025
+L +36V #PWR026
 U 1 1 5AB403B2
 P 8300 1200
-F 0 "#PWR025" H 8300 1050 50  0001 C CNN
+F 0 "#PWR026" H 8300 1050 50  0001 C CNN
 F 1 "+36V" H 8300 1340 50  0000 C CNN
 F 2 "" H 8300 1200 50  0001 C CNN

Commit message: layouted the board
Parts:
- removed Q2: Q_PMOS_GDS, TO_SOT_Packages_SMD:TO-252-2, symbol Q_PMOS_GDS
- added Q2: PMV48XP,215, TO_SOT_Packages_SMD:SOT-23, symbol Q_PMOS_GSD
- Q1: value Q_PMOS_GDS -> IRF9Z34NPbF; footprint TO_SOT_Packages_SMD:TO-252-2 -> TO_SOT_Packages_THT:TO-220_Vertical; Part Number AOD4189 -> IRF9Z34NPbF
- R28: footprint Resistors_SMD:R_0603 -> FORT:R_S-5; Part Number RMCF0603FT5K11 -> S5-47RF1
Connections:
- net VS6: now also Q2.3 (D)
- net V36_PROTECTED: now reaches D7.1 (K), Q1.3 (S), R28.1, U5.10 (VS), U5.8 (VS), U5.9 (VS)
- net V6_PROTECTED: now reaches C34.1, R35.1, U6.1 (VI)
- net V6_PROTECTED: now also Q2.1 (G), Q2.2 (S)
Changed lines of the file:
@@
 F 0 "R28" V 5480 1200 50  0000 C CNN
 F 1 "47, 4W" V 5300 1200 50  0000 C CNN
-F 2 "Resistors_SMD:R_0603" V 5330 1200 50  0001 C CNN
+F 2 "FORT:R_S-5" V 5330 1200 50  0001 C CNN
 F 3 "" H 5400 1200 50  0001 C CNN
-F 4 "RMCF0603FT5K11" H 5400 1200 60  0001 C CNN "Part Number"
+F 4 "S5-47RF1" H 5400 1200 60  0001 C CNN "Part Number"
 	1    5400 1200
 	0    -1   -1   0
@@
 U 1 1 5AB1266D
 P 2950 1300
-F 0 "Q1" H 3150 1350 50  0000 L CNN
-F 1 "Q_PMOS_GDS" H 3150 1250 50  0000 L CNN
-F 2 "TO_SOT_Packages_SMD:TO-252-2" H 3150 1400 50  0001 C CNN
+F 0 "Q1" V 3300 1300 50  0000 L CNN
+F 1 "IRF9Z34NPbF" V 3200 1300 50  0000 L CNN
+F 2 "TO_SOT_Packages_THT:TO-220_Vertical" H 3150 1400 50  0001 C CNN
 F 3 "" H 2950 1300 50  0001 C CNN
-F 4 "AOD4189" H 2950 1300 60  0001 C CNN "Part Number"
+F 4 "IRF9Z34NPbF" H 2950 1300 60  0001 C CNN "Part Number"
 	1    2950 1300
 	0    -1   -1   0
@@
 $EndComp
 $Comp
-L Q_PMOS_GDS Q2
-U 1 1 5AB3F8DC
-P 3400 5700
-F 0 "Q2" H 3600 5750 50  0000 L CNN
-F 1 "Q_PMOS_GDS" H 3600 5650 50  0000 L CNN
-F 2 "TO_SOT_Packages_SMD:TO-252-2" H 3600 5800 50  0001 C CNN
-F 3 "" H 3400 5700 50  0001 C CNN
-F 4 "AOD4189" H 3400 5700 60  0001 C CNN "Part Number"
-	1    3400 5700
-	0    -1   -1   0
-$EndComp
-$Comp
 L R R35
 U 1 1 5AB3FBD1
@@
 	3850 2200 3850 2650
 Connection ~ 3850 2200
+$Comp
+L Q_PMOS_GSD Q2
+U 1 1 5AB5D20E
+P 3400 5700
+F 0 "Q2" V 3650 5750 50  0000 L CNN
+F 1 "PMV48XP,215" V 3750 5700 50  0000 L CNN
+F 2 "TO_SOT_Packages_SMD:SOT-23" H 3600 5800 50  0001 C CNN
+F 3 "" H 3400 5700 50  0001 C CNN
+F 4 "PMV48XP,215" H 3400 5700 60  0001 C CNN "Part Number"
+	1    3400 5700
+	0    -1   -1   0
+$EndComp
+Text Label 3650 1200 0    60   ~ 0
+V36_PROTECTED
+Text Label 3650 5600 0    60   ~ 0
+V6_PROTECTED
 $EndSCHEMATC

Commit message: Improves the layout
Parts:
- R28: value 47, 4W -> 47, 5W; footprint FORT:R_S-5 -> Resistors_THT:R_Radial_Power_L13.0mm_W9.0mm_P5.00mm; Part Number S5-47RF1 -> SQP500JB-47R
Changed lines of the file:
@@
 $EndComp
 $Comp
-L GND #PWR022
+L GND #PWR026
 U 1 1 5AB122DC
 P 5400 3300
-F 0 "#PWR022" H 5400 3050 50  0001 C CNN
+F 0 "#PWR026" H 5400 3050 50  0001 C CNN
 F 1 "GND" H 5400 3150 50  0000 C CNN
 F 2 "" H 5400 3300 50  0001 C CNN
@@
 P 5400 1200
 F 0 "R28" V 5480 1200 50  0000 C CNN
-F 1 "47, 4W" V 5300 1200 50  0000 C CNN
-F 2 "FORT:R_S-5" V 5330 1200 50  0001 C CNN
+F 1 "47, 5W" V 5300 1200 50  0000 C CNN
+F 2 "Resistors_THT:R_Radial_Power_L13.0mm_W9.0mm_P5.00mm" V 5330 1200 50  0001 C CNN
 F 3 "" H 5400 1200 50  0001 C CNN
-F 4 "S5-47RF1" H 5400 1200 60  0001 C CNN "Part Number"
+F 4 "SQP500JB-47R" H 5400 1200 60  0001 C CNN "Part Number"
 	1    5400 1200
 	0    -1   -1   0
@@
 $EndComp
 $Comp
-L GND #PWR023
+L GND #PWR027
 U 1 1 5AB12A91
 P 2950 2300
-F 0 "#PWR023" H 2950 2050 50  0001 C CNN
+F 0 "#PWR027" H 2950 2050 50  0001 C CNN
 F 1 "GND" H 2950 2150 50  0000 C CNN
 F 2 "" H 2950 2300 50  0001 C CNN
@@
 VS6
 $Comp
-L GND #PWR024
+L GND #PWR028
 U 1 1 5AB3DBC2
 P 4850 6400
-F 0 "#PWR024" H 4850 6150 50  0001 C CNN
+F 0 "#PWR028" H 4850 6150 50  0001 C CNN
 F 1 "GND" H 4850 6250 50  0000 C CNN
 F 2 "" H 4850 6400 50  0001 C CNN
@@
 $EndComp
 $Comp
-L +5V #PWR025
+L +5V #PWR029
 U 1 1 5AB3EB47
 P 5850 5450
-F 0 "#PWR025" H 5850 5300 50  0001 C CNN
+F 0 "#PWR029" H 5850 5300 50  0001 C CNN
 F 1 "+5V" H 5850 5590 50  0000 C CNN
 F 2 "" H 5850 5450 50  0001 C CNN
@@
 $EndComp
 $Comp
-L +36V #PWR026
+L +36V #PWR030
 U 1 1 5AB403B2
 P 8300 1200
-F 0 "#PWR026" H 8300 1050 50  0001 C CNN
+F 0 "#PWR030" H 8300 1050 50  0001 C CNN
 F 1 "+36V" H 8300 1340 50  0000 C CNN
 F 2 "" H 8300 1200 50  0001 C CNN

Commit message: Adds a nice master board
Parts:
- removed C35: 10uF, Capacitors_SMD:C_0603, symbol C
- removed R34: 500m, Resistors_SMD:R_0603, symbol R
- removed U6: LM2936-5.0, TO_SOT_Packages_SMD:SOT-223-3Lead_TabPin2, symbol LM2936-5.0
- added C15: 1uF, Capacitors_SMD:C_0603, symbol C
- added C25: 0.01uF, Capacitors_SMD:C_0603, symbol C
- added U?: LP3985IM5-5.0/NOPB, TO_SOT_Packages_SMD:SOT-23-5, symbol LP3985IM5-5.0/NOPB
- C34: value 100nF -> 1uF; Part Number 06035C104KAT2A -> 0603YD105KAT2A
- R29, R35: value 100k -> 100K; Part Number RMCF0603FT100k -> RMCF0603FT100K
Connections:
- net +5V: now also C15.1, U?.5 (OUT)
- net GND: now also C15.2, C25.2, U?.2 (GND)
- net V6_PROTECTED: now also U?.1 (IN), U?.3 (EN)
- new net: C25.1, U?.4 (BYPASS)
Other:
- moved on the sheet: C34, Q2, R35
Changed lines of the file:
@@
 $EndComp
 $Comp
-L GND #PWR026
+L GND #PWR031
 U 1 1 5AB122DC
 P 5400 3300
-F 0 "#PWR026" H 5400 3050 50  0001 C CNN
+F 0 "#PWR031" H 5400 3050 50  0001 C CNN
 F 1 "GND" H 5400 3150 50  0000 C CNN
 F 2 "" H 5400 3300 50  0001 C CNN
@@
 P 2950 1900
 F 0 "R29" V 3030 1900 50  0000 C CNN
-F 1 "100k" V 2950 1900 50  0000 C CNN
+F 1 "100K" V 2950 1900 50  0000 C CNN
 F 2 "Resistors_SMD:R_0603" V 2880 1900 50  0001 C CNN
 F 3 "" H 2950 1900 50  0001 C CNN
-F 4 "RMCF0603FT100k" H 2950 1900 60  0001 C CNN "Part Number"
+F 4 "RMCF0603FT100K" H 2950 1900 60  0001 C CNN "Part Number"
 	1    2950 1900
 	1    0    0    -1
@@
 $EndComp
 $Comp
-L GND #PWR027
+L GND #PWR032
 U 1 1 5AB12A91
 P 2950 2300
-F 0 "#PWR027" H 2950 2050 50  0001 C CNN
+F 0 "#PWR032" H 2950 2050 50  0001 C CNN
 F 1 "GND" H 2950 2150 50  0000 C CNN
 F 2 "" H 2950 2300 50  0001 C CNN
@@
 	0    1    1    0
 $EndComp
-$Comp
-L LM2936-5.0 U6
-U 1 1 5AB3D855
-P 4650 5600
-F 0 "U6" H 4500 5725 50  0000 C CNN
-F 1 "LM2936-5.0" H 4650 5725 50  0000 L CNN
-F 2 "TO_SOT_Packages_SMD:SOT-223-3Lead_TabPin2" H 4650 5825 50  0001 C CIN
-F 3 "" H 4650 5550 50  0001 C CNN
-F 4 "LM2936MPX-5.0/NOPB" H 4650 5600 60  0001 C CNN "Part Number"
-	1    4650 5600
-	1    0    0    -1
-$EndComp
-Text HLabel 2650 5600 0    60   Input ~ 0
+Text HLabel 2300 4800 0    60   Input ~ 0
 VS6
-$Comp
-L GND #PWR028
-U 1 1 5AB3DBC2
-P 4850 6400
-F 0 "#PWR028" H 4850 6150 50  0001 C CNN
-F 1 "GND" H 4850 6250 50  0000 C CNN
-F 2 "" H 4850 6400 50  0001 C CNN
-F 3 "" H 4850 6400 50  0001 C CNN
-	1    4850 6400
-	1    0    0    -1
-$EndComp
-$Comp
-L C C35
-U 1 1 5AB3DCD0
-P 5500 6150
-F 0 "C35" H 5525 6250 50  0000 L CNN
-F 1 "10uF" H 5525 6050 50  0000 L CNN
-F 2 "Capacitors_SMD:C_0603" H 5538 6000 50  0001 C CNN
-F 3 "" H 5500 6150 50  0001 C CNN
-F 4 "0805ZD106MAT2A" H 5500 6150 60  0001 C CNN "Part Number"
-	1    5500 6150
-	1    0    0    -1
-$EndComp
-$Comp
-L R R34
-U 1 1 5AB3DDAE
-P 5500 5800
-F 0 "R34" V 5580 5800 50  0000 C CNN
-F 1 "500m" V 5500 5800 50  0000 C CNN
-F 2 "Resistors_SMD:R_0603" V 5430 5800 50  0001 C CNN
-F 3 "" H 5500 5800 50  0001 C CNN
-F 4 "CSR0603FKR500" H 5500 5800 60  0001 C CNN "Part Number"
-	1    5500 5800
-	1    0    0    -1
-$EndComp
 $Comp
 L C C34
 U 1 1 5AB3E3D4
-P 4050 5800
-F 0 "C34" H 4075 5900 50  0000 L CNN
-F 1 "100nF" H 4075 5700 50  0000 L CNN
-F 2 "Capacitors_SMD:C_0603" H 4088 5650 50  0001 C CNN
-F 3 "" H 4050 5800 50  0001 C CNN
-F 4 "06035C104KAT2A" H 4050 5800 60  0001 C CNN "Part Number"
-	1    4050 5800
-	1    0    0    -1
-$EndComp
-$Comp
-L +5V #PWR029
+P 3700 5000
+F 0 "C34" H 3725 5100 50  0000 L CNN
+F 1 "1uF" H 3725 4900 50  0000 L CNN
+F 2 "Capacitors_SMD:C_0603" H 3738 4850 50  0001 C CNN
+F 3 "" H 3700 5000 50  0001 C CNN
+F 4 "0603YD105KAT2A" H 3700 5000 60  0001 C CNN "Part Number"
+	1    3700 5000
+	1    0    0    -1
+$EndComp
+$Comp
+L +5V #PWR033
 U 1 1 5AB3EB47
-P 5850 5450
-F 0 "#PWR029" H 5850 5300 50  0001 C CNN
-F 1 "+5V" H 5850 5590 50  0000 C CNN
-F 2 "" H 5850 5450 50  0001 C CNN
-F 3 "" H 5850 5450 50  0001 C CNN
-	1    5850 5450
+P 6100 4650
+F 0 "#PWR033" H 6100 4500 50  0001 C CNN
+F 1 "+5V" H 6100 4790 50  0000 C CNN
+F 2 "" H 6100 4650 50  0001 C CNN
+F 3 "" H 6100 4650 50  0001 C CNN
+	1    6100 4650
 	1    0    0    -1
 $EndComp
@@
 L R R35
 U 1 1 5AB3FBD1
-P 3400 6150
-F 0 "R35" V 3480 6150 50  0000 C CNN
-F 1 "100k" V 3400 6150 50  0000 C CNN
-F 2 "Resistors_SMD:R_0603" V 3330 6150 50  0001 C CNN
-F 3 "" H 3400 6150 50  0001 C CNN
-F 4 "RMCF0603FT100k" H 3400 6150 60  0001 C CNN "Part Number"
-	1    3400 6150
-	1    0    0    -1
-$EndComp
-$Comp
-L +36V #PWR030
+P 3050 5350
+F 0 "R35" V 3130 5350 50  0000 C CNN
+F 1 "100K" V 3050 5350 50  0000 C CNN
+F 2 "Resistors_SMD:R_0603" V 2980 5350 50  0001 C CNN
+F 3 "" H 3050 5350 50  0001 C CNN
+F 4 "RMCF0603FT100K" H 3050 5350 60  0001 C CNN "Part Number"
+	1    3050 5350
+	1    0    0    -1
+$EndComp
+$Comp
+L +36V #PWR034
 U 1 1 5AB403B2
 P 8300 1200
-F 0 "#PWR030" H 8300 1050 50  0001 C CNN
+F 0 "#PWR034" H 8300 1050 50  0001 C CNN
 F 1 "+36V" H 8300 1340 50  0000 C CNN
 F 2 "" H 8300 1200 50  0001 C CNN
@@
 Connection ~ 7250 1900
 Wire Wire Line
-	4950 5600 5850 5600
-Wire Wire Line
-	3600 5600 4350 5600
-Connection ~ 4050 5600
-Connection ~ 5500 5600
-Wire Wire Line
-	5850 5600 5850 5450
-Wire Wire Line
-	5500 5950 5500 6000
-Wire Wire Line
-	5500 5650 5500 5600
-Wire Wire Line
-	5500 6350 5500 6300
-Wire Wire Line
-	3400 6350 5500 6350
-Wire Wire Line
-	4050 6350 4050 5950
-Wire Wire Line
-	4650 5900 4650 6350
-Connection ~ 4650 6350
-Wire Wire Line
-	4850 6350 4850 6400
-Connection ~ 4850 6350
-Wire Wire Line
-	4050 5600 4050 5650
-Wire Wire Line
-	3400 6350 3400 6300
-Connection ~ 4050 6350
-Wire Wire Line
-	3400 5900 3400 6000
-Wire Wire Line
-	3750 5600 3750 5950
-Wire Wire Line
-	3750 5950 3400 5950
-Connection ~ 3400 5950
-Connection ~ 3750 5600
-Wire Wire Line
-	3200 5600 2650 5600
+	5200 4800 6100 4800
+Wire Wire Line
+	3250 4800 4200 4800
+Connection ~ 3700 4800
+Connection ~ 5750 4800
+Wire Wire Line
+	6100 4800 6100 4650
+Wire Wire Line
+	5750 4800 5750 4950
+Wire Wire Line
+	3700 5150 3700 5600
+Wire Wire Line
+	3700 4800 3700 4850
+Wire Wire Line
+	3050 5500 3050 5700
+Wire Wire Line
+	3050 5100 3050 5200
+Wire Wire Line
+	3400 4800 3400 5150
+Wire Wire Line
+	3400 5150 3050 5150
+Connection ~ 3050 5150
+Connection ~ 3400 4800
+Wire Wire Line
+	2850 4800 2300 4800
 Wire Wire Line
 	8300 1900 8300 1200
@@
 L Q_PMOS_GSD Q2
 U 1 1 5AB5D20E
-P 3400 5700
-F 0 "Q2" V 3650 5750 50  0000 L CNN
-F 1 "PMV48XP,215" V 3750 5700 50  0000 L CNN
-F 2 "TO_SOT_Packages_SMD:SOT-23" H 3600 5800 50  0001 C CNN
-F 3 "" H 3400 5700 50  0001 C CNN
-F 4 "PMV48XP,215" H 3400 5700 60  0001 C CNN "Part Number"
-	1    3400 5700
+P 3050 4900
+F 0 "Q2" V 3300 4950 50  0000 L CNN
+F 1 "PMV48XP,215" V 3400 4900 50  0000 L CNN
+F 2 "TO_SOT_Packages_SMD:SOT-23" H 3250 5000 50  0001 C CNN
+F 3 "" H 3050 4900 50  0001 C CNN
+F 4 "PMV48XP,215" H 3050 4900 60  0001 C CNN "Part Number"
+	1    3050 4900
 	0    -1   -1   0
 $EndComp
 Text Label 3650 1200 0    60   ~ 0
 V36_PROTECTED
-Text Label 3650 5600 0    60   ~ 0
+Text Label 3300 4800 0    60   ~ 0
 V6_PROTECTED
+$Comp
+L C C15
+U 1 1 5AC62A8E
+P 5750 5100
+F 0 "C15" H 5775 5200 50  0000 L CNN
+F 1 "1uF" H 5775 5000 50  0000 L CNN
+F 2 "Capacitors_SMD:C_0603" H 5788 4950 50  0001 C CNN
+F 3 "" H 5750 5100 50  0001 C CNN
+F 4 "0603YD105KAT2A" H 5750 5100 60  0001 C CNN "Part Number"
+	1    5750 5100
+	1    0    0    -1
+$EndComp
+$Comp
+L C C25
+U 1 1 5AC62C30
+P 5400 5350
+F 0 "C25" H 5425 5450 50  0000 L CNN
+F 1 "0.01uF" H 5425 5250 50  0000 L CNN
+F 2 "Capacitors_SMD:C_0603" H 5438 5200 50  0001 C CNN
+F 3 "" H 5400 5350 50  0001 C CNN
+F 4 "06035C103KAT4A" H 5400 5350 60  0001 C CNN "Part Number"
+	1    5400 5350
+	1    0    0    -1
+$EndComp
+Wire Wire Line
+	4200 5000 4050 5000
+Wire Wire Line
+	4050 5000 4050 4800
+Connection ~ 4050 4800
+$Comp
+L GND #PWR035
+U 1 1 5AC62CF7
+P 3050 5700
+F 0 "#PWR035" H 3050 5450 50  0001 C CNN
+F 1 "GND" H 3050 5550 50  0000 C CNN
+F 2 "" H 3050 5700 50  0001 C CNN
+F 3 "" H 3050 5700 50  0001 C CNN
+	1    3050 5700
+	1    0    0    -1
+$EndComp
+Wire Wire Line
+	3050 5600 5750 5600
+Connection ~ 3050 5600
+Wire Wire Line
+	4700 5600 4700 5550
+Connection ~ 3700 5600
+Wire Wire Line
+	5400 5600 5400 5500
+Connection ~ 4700 5600
+Wire Wire Line
+	5200 5000 5400 5000
+Wire Wire Line
+	5400 5000 5400 5200
+Wire Wire Line
+	5750 5600 5750 5250
+Connection ~ 5400 5600
+$Comp
+L LP3985IM5-5.0/NOPB U?
+U 1 1 5AC5F4CF
+P 4700 5000
+F 0 "U?" H 4450 4600 60  0000 C CNN
+F 1 "LP3985IM5-5.0/NOPB" H 4700 5350 60  0000 C CNN
+F 2 "TO_SOT_Packages_SMD:SOT-23-5" H 4650 5000 60  0001 C CNN
+F 3 "" H 4650 5000 60  0001 C CNN
+F 4 "LP3985IM5-5.0/NOPB" H 4700 5000 60  0001 C CNN "Part Number"
+	1    4700 5000
+	1    0    0    -1
+$EndComp
 $EndSCHEMATC

Commit message: wip
Parts:
- gave numbers to parts that had none: 1
Changed lines of the file:
@@
 Connection ~ 5400 5600
 $Comp
-L LP3985IM5-5.0/NOPB U?
+L LP3985IM5-5.0/NOPB U6
 U 1 1 5AC5F4CF
 P 4700 5000
-F 0 "U?" H 4450 4600 60  0000 C CNN
+F 0 "U6" H 4450 4600 60  0000 C CNN
 F 1 "LP3985IM5-5.0/NOPB" H 4700 5350 60  0000 C CNN
 F 2 "TO_SOT_Packages_SMD:SOT-23-5" H 4650 5000 60  0001 C CNN

Commit message: wip
Parts:
- C25: value 0.01uF -> 10nF, 50V
- U5: value TPS1H100AQ -> TPS1H100AQPWPRQ1
Changed lines of the file:
@@
 P 5450 2250
 F 0 "U5" H 5250 1700 60  0000 C CNN
-F 1 "TPS1H100AQ" H 5450 2750 60  0000 C CNN
+F 1 "TPS1H100AQPWPRQ1" H 5450 2750 60  0000 C CNN
 F 2 "FORT:HTSSOP-14-1EP_4.4x6.5mm_Pitch0.65mm_ThermalPad" H 5400 2350 60  0001 C CNN
 F 3 "" H 5400 2350 60  0001 C CNN
@@
 P 5400 5350
 F 0 "C25" H 5425 5450 50  0000 L CNN
-F 1 "0.01uF" H 5425 5250 50  0000 L CNN
+F 1 "10nF, 50V" H 4950 5250 50  0000 L CNN
 F 2 "Capacitors_SMD:C_0603" H 5438 5200 50  0001 C CNN
 F 3 "" H 5400 5350 50  0001 C CNN
