File: ecad/helios/LED_driver/UV_LEDs.sch (KiCad schematic (older format))
At the start: 10 parts, among them J5 LED HDR, J6 LED HDR, J7 LED PLUG, J8 LED PLUG, Q3 BSS138L

Commit message: Makes all electronics production ready
Parts:
- R40: value 100K -> 100k
Other:
- note added: "© 2018 Université de Lausanne\n\nThis documentation describes Open Hardware and is licensed under the\nCERN OHL v. 1.2.\n\nYou may redistribute and modify this documentation under the terms of\nthe CERN OHL v.1.2. (http://ohwr.org/cernohl). This documentation is\ndistributed WITHOUT ANY EXPRESS OR IMPLIED WARRANTY,\nINCLUDING OF MERCHANTABILITY, SATISFACTORY QUALITY AND\nFITNESS FOR A PARTICULAR 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"
Changed lines of the file:
@@
 encoding utf-8
 Sheet 9 9
-Title ""
-Date ""
-Rev ""
-Comp ""
-Comment1 ""
-Comment2 ""
+Title "Helios - Module - UV Illumination"
+Date "12/10/2018"
+Rev "C"
+Comp "Université de Lausanne"
+Comment1 "Author: Alexandre Tuleu"
+Comment2 "Licensed under the CERN OHL v1.2"
 Comment3 ""
 Comment4 ""
@@
 AR Path="/5C214647/5C217CCB" Ref="R40"  Part="1"
 F 0 "R40" V 5930 4450 50  0000 C CNN
-F 1 "100K" V 5850 4450 50  0000 C CNN
+F 1 "100k" V 5850 4450 50  0000 C CNN
 F 2 "Resistor_SMD:R_0603_1608Metric" V 5780 4450 50  0001 C CNN
 F 3 "" H 5850 4450 50  0001 C CNN
@@
 	4150 4250 5850 4250
 Connection ~ 5850 4250
+Text Notes 550  7750 0    60   ~ 0
+© 2018 Université de Lausanne\n\nThis documentation describes Open Hardware and is licensed under the\nCERN OHL v. 1.2.\n\nYou may redistribute and modify this documentation under the terms of\nthe CERN OHL v.1.2. (http://ohwr.org/cernohl). This documentation is\ndistributed WITHOUT ANY EXPRESS OR IMPLIED WARRANTY,\nINCLUDING OF MERCHANTABILITY, SATISFACTORY QUALITY AND\nFITNESS FOR A PARTICULAR PURPOSE. Please see the CERN OHL v.1.2\nfor applicable conditions
 $EndSCHEMATC
