File: ecad/climate/pleiades/UC.sch (KiCad schematic (older format))
At the start: 16 parts, among them J4 M20-8760342, SW1 1825910-6, U2 AT90CAN128-16AU, Y1 16MHz

Commit message: Makes Pleiades KiCad 5 compatible
Parts:
- C10, C11, C7, C8, C9: footprint Capacitors_SMD:C_0603 -> Capacitor_SMD:C_0603_1608Metric; symbol C -> Device:C
- D3, D6: footprint LEDs:LED_0603 -> LED_SMD:LED_0603_1608Metric; symbol LED -> Device:LED
- D4: symbol D_Schottky -> Device:D_Schottky
- J4: footprint Pin_Headers:Pin_Header_Straight_2x03_Pitch2.54mm_SMD -> Connector_PinHeader_2.54mm:PinHeader_2x03_P2.54mm_Vertical_SMD; symbol Conn_02x03_Odd_Even -> Connector_Generic:Conn_02x03_Odd_Even
- R4, R5, R8, R9: footprint Resistors_SMD:R_0603 -> Resistor_SMD:R_0603_1608Metric; symbol R -> Device:R
- SW1: footprint Buttons_Switches_THT:SW_PUSH_6mm -> Button_Switch_THT:SW_PUSH_6mm; symbol SW_Push -> Switch:SW_Push
- U2: footprint Housings_QFP:TQFP-64_14x14mm_Pitch0.8mm -> Package_QFP:TQFP-64_14x14mm_P0.8mm; symbol AT90CAN128-16AU -> MCU_Microchip_AVR:AT90CAN128-16AU
- Y1: footprint Crystals:Crystal_SMD_SeikoEpson_FA238-4pin_3.2x2.5mm -> Crystal:Crystal_SMD_SeikoEpson_FA238-4Pin_3.2x2.5mm; symbol Crystal_GND24 -> Device:Crystal_GND24
Connections:
- wire segments 71 -> 81
Other:
- moved on the sheet: C7, C8, C9, R4

Commit message: Makes one board that fit them all
Bad Idea, will revert the changes soon
Parts:
- added J14, J15: 68000-212HLF, Connector_PinHeader_2.54mm:PinHeader_1x12_P2.54mm_Vertical, symbol Connector_Generic:Conn_01x12
Connections:
- net labels added: +12V, +3V3, RELAY_1, RELAY_2
- wire segments 81 -> 115
- no-connect marks 42 -> 24
Changed lines of the file:
@@
 $Descr A4 11693 8268
 encoding utf-8
-Sheet 6 8
+Sheet 6 12
 Title ""
 Date ""
@@
 Text HLabel 7400 3750 2    60   Output ~ 0
 HEAT2
-$Comp
-L MCU_Microchip_AVR:AT90CAN128-16AU U2
-U 1 1 5BA92DFF
-P 5800 3950
-F 0 "U2" H 5300 5900 50  0000 L BNN
-F 1 "AT90CAN128-16AU" H 6950 2000 50  0000 R BNN
-F 2 "Package_QFP:TQFP-64_14x14mm_P0.8mm" H 5850 3950 50  0001 C CNN
-F 3 "" H 5800 3950 50  0001 C CNN
-F 4 "AT90CAN128-16AU" H 5800 3950 60  0001 C CNN "Part Number"
-	1    5800 3950
-	1    0    0    -1
-$EndComp
 $Comp
 L power:GND #PWR034
@@
 Text HLabel 7800 4950 2    60   Output ~ 0
 SCL_5V
-NoConn ~ 6400 2250
-NoConn ~ 6400 2350
-NoConn ~ 6400 2450
-NoConn ~ 6400 2550
-NoConn ~ 6400 2650
-NoConn ~ 6400 2750
-NoConn ~ 6400 2850
-NoConn ~ 6400 2950
 NoConn ~ 6400 3150
 NoConn ~ 6400 3350
@@
 NoConn ~ 6400 3550
 NoConn ~ 6400 3850
-NoConn ~ 6400 4050
-NoConn ~ 6400 4150
-NoConn ~ 6400 4250
-NoConn ~ 6400 4350
-NoConn ~ 6400 4450
-NoConn ~ 6400 4550
-NoConn ~ 6400 4650
-NoConn ~ 6400 4750
 NoConn ~ 6400 5150
 NoConn ~ 6400 5250
@@
 NoConn ~ 5200 4450
 NoConn ~ 5200 4550
-NoConn ~ 5200 4650
-NoConn ~ 5200 4750
 NoConn ~ 5200 5150
 NoConn ~ 5200 5450
@@
 	4150 5550 5200 5550
 Wire Wire Line
-	6400 5550 7450 5550
-Wire Wire Line
-	6400 5450 7450 5450
-Wire Wire Line
-	6400 4950 7800 4950
-Wire Wire Line
-	6400 5050 7800 5050
-Wire Wire Line
-	6400 3750 7400 3750
-Wire Wire Line
-	6400 3650 7400 3650
-Wire Wire Line
-	6400 3250 7700 3250
-Wire Wire Line
 	5150 1250 5150 1350
 Wire Wire Line
@@
 Wire Wire Line
 	5800 6450 5800 6400
+$Comp
+L Connector_Generic:Conn_01x12 J14
+U 1 1 5BB5BBE4
+P 10450 2450
+F 0 "J14" H 10530 2442 50  0000 L CNN
+F 1 "68000-212HLF" H 10530 2351 50  0000 L CNN
+F 2 "Connector_PinHeader_2.54mm:PinHeader_1x12_P2.54mm_Vertical" H 10450 2450 50  0001 C CNN
+F 3 "~" H 10450 2450 50  0001 C CNN
+F 4 "68000-212HLF" H 10450 2450 50  0001 C CNN "Part Number"
+	1    10450 2450
+	1    0    0    -1
+$EndComp
+$Comp
+L MCU_Microchip_AVR:AT90CAN128-16AU U2
+U 1 1 5BA92DFF
+P 5800 3950
+F 0 "U2" H 5300 5900 50  0000 L BNN
+F 1 "AT90CAN128-16AU" H 6950 2000 50  0000 R BNN
+F 2 "Package_QFP:TQFP-64_14x14mm_P0.8mm" H 5850 3950 50  0001 C CNN
+F 3 "" H 5800 3950 50  0001 C CNN
+F 4 "AT90CAN128-16AU" H 5800 3950 60  0001 C CNN "Part Number"
+	1    5800 3950
+	1    0    0    -1
+$EndComp
+Wire Wire Line
+	6400 5550 7450 5550
+Wire Wire Line
+	6400 5450 7450 5450
+Wire Wire Line
+	6400 4950 7800 4950
+Wire Wire Line
+	6400 5050 7800 5050
+Wire Wire Line
+	6400 3750 7400 3750
+Wire Wire Line
+	6400 3650 7400 3650
+Wire Wire Line
+	6400 3250 7700 3250
+$Comp
+L Connector_Generic:Conn_01x12 J15
+U 1 1 5BB63291
+P 10450 4250
+F 0 "J15" H 10530 4242 50  0000 L CNN
+F 1 "68000-212HLF" H 10530 4151 50  0000 L CNN
+F 2 "Connector_PinHeader_2.54mm:PinHeader_1x12_P2.54mm_Vertical" H 10450 4250 50  0001 C CNN
+F 3 "~" H 10450 4250 50  0001 C CNN
+F 4 "68000-212HLF" H 10450 4250 50  0001 C CNN "Part Number"
+	1    10450 4250
+	1    0    0    -1
+$EndComp
+Wire Wire Line
+	6400 2250 10250 2250
+Wire Wire Line
+	6400 2350 10250 2350
+Wire Wire Line
+	6400 2450 10250 2450
+Wire Wire Line
+	6400 2550 10250 2550
+Wire Wire Line
+	6400 2650 10250 2650
+Wire Wire Line
+	6400 2750 10250 2750
+Wire Wire Line
+	6400 2850 10250 2850
+Wire Wire Line
+	6400 2950 10250 2950
+Wire Wire Line
+	6400 4050 10250 4050
+Wire Wire Line
+	6400 4150 10250 4150
+Wire Wire Line
+	6400 4250 10250 4250
+Wire Wire Line
+	6400 4350 10250 4350
+Wire Wire Line
+	6400 4450 10250 4450
+Wire Wire Line
+	6400 4550 10250 4550
+Wire Wire Line
+	6400 4650 10250 4650
+Wire Wire Line
+	6400 4750 10250 4750
+$Comp
+L power:GND #PWR0101
+U 1 1 5BB6711B
+P 10100 3150
+F 0 "#PWR0101" H 10100 2900 50  0001 C CNN
+F 1 "GND" H 10105 2977 50  0000 C CNN
+F 2 "" H 10100 3150 50  0001 C CNN
+F 3 "" H 10100 3150 50  0001 C CNN
+	1    10100 3150
+	1    0    0    -1
+$EndComp
+Wire Wire Line
+	10100 3050 10250 3050
+$Comp
+L power:GND #PWR0102
+U 1 1 5BB69978
+P 10100 5000
+F 0 "#PWR0102" H 10100 4750 50  0001 C CNN
+F 1 "GND" H 10105 4827 50  0000 C CNN
+F 2 "" H 10100 5000 50  0001 C CNN
+F 3 "" H 10100 5000 50  0001 C CNN
+	1    10100 5000
+	1    0    0    -1
+$EndComp
+Wire Wire Line
+	10100 5000 10100 4850
+Wire Wire Line
+	10100 4850 10250 4850
+$Comp
+L power:+12V #PWR0103
+U 1 1 5BB6C373
+P 10100 1800
+F 0 "#PWR0103" H 10100 1650 50  0001 C CNN
+F 1 "+12V" H 10115 1973 50  0000 C CNN
+F 2 "" H 10100 1800 50  0001 C CNN
+F 3 "" H 10100 1800 50  0001 C CNN
+	1    10100 1800
+	1    0    0    -1
+$EndComp
+Wire Wire Line
+	10100 1800 10100 1950
+Wire Wire Line
+	10100 1950 10250 1950
+$Comp
+L power:+5V #PWR0104
+U 1 1 5BB6EEB4
+P 9900 1800
+F 0 "#PWR0104" H 9900 1650 50  0001 C CNN
+F 1 "+5V" H 9915 1973 50  0000 C CNN
+F 2 "" H 9900 1800 50  0001 C CNN
+F 3 "" H 9900 1800 50  0001 C CNN
+	1    9900 1800
+	1    0    0    -1
+$EndComp
+$Comp
+L power:+3V3 #PWR0105
+U 1 1 5BB71A1D
+P 9650 1800
+F 0 "#PWR0105" H 9650 1650 50  0001 C CNN
+F 1 "+3V3" H 9665 1973 50  0000 C CNN
+F 2 "" H 9650 1800 50  0001 C CNN
+F 3 "" H 9650 1800 50  0001 C CNN
+	1    9650 1800
+	1    0    0    -1
+$EndComp
+Wire Wire Line
+	9650 1800 9650 2150
+Wire Wire Line
+	9650 2150 10250 2150
+Wire Wire Line
+	10250 2050 9900 2050
+Wire Wire Line
+	9900 2050 9900 1800
+$Comp
+L power:+12V #PWR0106
+U 1 1 5BB77434
+P 10100 3600
+F 0 "#PWR0106" H 10100 3450 50  0001 C CNN
+F 1 "+12V" H 10115 3773 50  0000 C CNN
+F 2 "" H 10100 3600 50  0001 C CNN
+F 3 "" H 10100 3600 50  0001 C CNN
+	1    10100 3600
+	1    0    0    -1
+$EndComp
+Wire Wire Line
+	10100 3600 10100 3750
+Wire Wire Line
+	10100 3750 10250 3750
+$Comp
+L power:+5V #PWR0107
+U 1 1 5BB7743C
+P 9900 3600
+F 0 "#PWR0107" H 9900 3450 50  0001 C CNN
+F 1 "+5V" H 9915 3773 50  0000 C CNN
+F 2 "" H 9900 3600 50  0001 C CNN
+F 3 "" H 9900 3600 50  0001 C CNN
+	1    9900 3600
+	1    0    0    -1
+$EndComp
+$Comp
+L power:+3V3 #PWR0108
+U 1 1 5BB77442
+P 9650 3600
+F 0 "#PWR0108" H 9650 3450 50  0001 C CNN
+F 1 "+3V3" H 9665 3773 50  0000 C CNN
+F 2 "" H 9650 3600 50  0001 C CNN
+F 3 "" H 9650 3600 50  0001 C CNN
+	1    9650 3600
+	1    0    0    -1
+$EndComp
+Wire Wire Line
+	9650 3600 9650 3950
+Wire Wire Line
+	9650 3950 10250 3950
+Wire Wire Line
+	10250 3850 9900 3850
+Wire Wire Line
+	9900 3850 9900 3600
+Wire Wire Line
+	10100 3150 10100 3050
+Text HLabel 4600 4650 0    50   Output ~ 0
+RELAY_1
+Text HLabel 4600 4750 0    50   Output ~ 0
+RELAY_2
+Wire Wire Line
+	4600 4650 5200 4650
+Wire Wire Line
+	4600 4750 5200 4750
 $EndSCHEMATC
