File: ecad/climate/pleiades/i2c_mux.sch (KiCad schematic (older format))
At the start: 15 parts, among them U5 TCA9544A

Commit message: Makes Pleiades KiCad 5 compatible
Parts:
- C4: footprint Capacitors_SMD:C_0603 -> Capacitor_SMD:C_0603_1608Metric; symbol C -> Device:C
- R1, R10, R11, R12, R13, R14, R15, R16, R17, R18, R19, R2, R3: footprint Resistors_SMD:R_0603 -> Resistor_SMD:R_0603_1608Metric; symbol R -> Device:R
- U5: footprint Housings_SSOP:TSSOP-20_4.4x6.5mm_Pitch0.65mm -> Package_SO:SSOP-20_4.4x6.5mm_P0.65mm; symbol TCA9544A -> Interface_Expansion:TCA9544A; Part Number (none) -> TCA9544A
Changed lines of the file:
@@
-EESchema Schematic File Version 2
-LIBS:power
-LIBS:device
-LIBS:switches
-LIBS:relays
-LIBS:motors
-LIBS:transistors
-LIBS:conn
-LIBS:linear
-LIBS:regul
-LIBS:74xx
-LIBS:cmos4000
-LIBS:adc-dac
-LIBS:memory
-LIBS:xilinx
-LIBS:microcontrollers
-LIBS:dsp
-LIBS:microchip
-LIBS:analog_switches
-LIBS:motorola
-LIBS:texas
-LIBS:intel
-LIBS:audio
-LIBS:interface
-LIBS:digital-audio
-LIBS:philips
-LIBS:display
-LIBS:cypress
-LIBS:siliconi
-LIBS:opto
-LIBS:atmel
-LIBS:contrib
-LIBS:valves
-LIBS:fort
-LIBS:Oscillators
-LIBS:nxp
-LIBS:zeus-cache
-EELAYER 25 0
+EESchema Schematic File Version 4
+LIBS:pleiades-cache
+EELAYER 26 0
 EELAYER END
 $Descr A4 11693 8268
@@
 $EndDescr
 $Comp
-L TCA9544A U5
+L Interface_Expansion:TCA9544A U5
 U 1 1 5BAB6C8F
 P 5450 3950
 F 0 "U5" H 5250 4750 50  0000 L CNN
 F 1 "TCA9544A" H 5550 4750 50  0000 L CNN
-F 2 "Housings_SSOP:TSSOP-20_4.4x6.5mm_Pitch0.65mm" H 6450 3050 50  0001 C CNN
+F 2 "Package_SO:SSOP-20_4.4x6.5mm_P0.65mm" H 6450 3050 50  0001 C CNN
 F 3 "" H 5500 4200 50  0000 C CNN
+F 4 "TCA9544A" H 5450 3950 50  0001 C CNN "Part Number"
 	1    5450 3950
 	1    0    0    -1
 $EndComp
 $Comp
-L +5V #PWR040
+L power:+5V #PWR040
 U 1 1 5BAB6C96
 P 5450 2500
@@
 $EndComp
 $Comp
-L C C4
+L Device:C C4
 U 1 1 5BAB6C9D
 P 5700 2700
 F 0 "C4" H 5725 2800 50  0000 L CNN
 F 1 "100nF" H 5725 2600 50  0000 L CNN
-F 2 "Capacitors_SMD:C_0603" H 5738 2550 50  0001 C CNN
+F 2 "Capacitor_SMD:C_0603_1608Metric" H 5738 2550 50  0001 C CNN
 F 3 "" H 5700 2700 50  0001 C CNN
 F 4 "06035C104KAT2A" H 5700 2700 60  0001 C CNN "Part Number"
@@
 $EndComp
 $Comp
-L GND #PWR041
+L power:GND #PWR041
 U 1 1 5BAB6CA4
 P 5700 2900
@@
 $EndComp
 $Comp
-L GND #PWR042
+L power:GND #PWR042
 U 1 1 5BAB6CAA
 P 5450 5050
@@
 NoConn ~ 5950 4550
 $Comp
-L R R11
+L Device:R R11
 U 1 1 5BAB6CBB
 P 6500 4650
 F 0 "R11" V 6580 4650 50  0000 C CNN
 F 1 "10k" V 6500 4650 50  0000 C CNN
-F 2 "Resistors_SMD:R_0603" V 6430 4650 50  0001 C CNN
+F 2 "Resistor_SMD:R_0603_1608Metric" V 6430 4650 50  0001 C CNN
 F 3 "" H 6500 4650 50  0001 C CNN
 F 4 "GPR060310K" H 6500 4650 60  0001 C CNN "Part Number"
@@
 $EndComp
 $Comp
-L +3.3V #PWR043
+L pleiades-rescue:+3.3V #PWR043
 U 1 1 5BAB6CC8
 P 6750 4650
@@
 ~INT0
 $Comp
-L R R13
+L Device:R R13
 U 1 1 5BABCAD6
 P 7700 3000
 F 0 "R13" V 7780 3000 50  0000 C CNN
 F 1 "10k" V 7700 3000 50  0000 C CNN
-F 2 "Resistors_SMD:R_0603" V 7630 3000 50  0001 C CNN
+F 2 "Resistor_SMD:R_0603_1608Metric" V 7630 3000 50  0001 C CNN
 F 3 "" H 7700 3000 50  0001 C CNN
 F 4 "GPR060310K" H 7700 3000 60  0001 C CNN "Part Number"
@@
 $EndComp
 $Comp
-L R R14
+L Device:R R14
 U 1 1 5BABCB3A
 P 7900 3000
 F 0 "R14" V 7980 3000 50  0000 C CNN
 F 1 "10k" V 7900 3000 50  0000 C CNN
-F 2 "Resistors_SMD:R_0603" V 7830 3000 50  0001 C CNN
+F 2 "Resistor_SMD:R_0603_1608Metric" V 7830 3000 50  0001 C CNN
 F 3 "" H 7900 3000 50  0001 C CNN
 F 4 "GPR060310K" H 7900 3000 60  0001 C CNN "Part Number"
@@
 $EndComp
 $Comp
-L R R15
+L Device:R R15
 U 1 1 5BABCB73
 P 8100 3000
 F 0 "R15" V 8180 3000 50  0000 C CNN
 F 1 "10k" V 8100 3000 50  0000 C CNN
-F 2 "Resistors_SMD:R_0603" V 8030 3000 50  0001 C CNN
+F 2 "Resistor_SMD:R_0603_1608Metric" V 8030 3000 50  0001 C CNN
 F 3 "" H 8100 3000 50  0001 C CNN
 F 4 "GPR060310K" H 8100 3000 60  0001 C CNN "Part Number"
@@
 $EndComp
 $Comp
-L R R2
+L Device:R R2
 U 1 1 5BABCBB7
 P 6200 3000
 F 0 "R2" V 6280 3000 50  0000 C CNN
 F 1 "4k99" V 6200 3000 50  0000 C CNN
-F 2 "Resistors_SMD:R_0603" V 6130 3000 50  0001 C CNN
+F 2 "Resistor_SMD:R_0603_1608Metric" V 6130 3000 50  0001 C CNN
 F 3 "" H 6200 3000 50  0001 C CNN
 F 4 "GPR06034K99" H 6200 3000 60  0001 C CNN "Part Number"
@@
 $EndComp
 $Comp
-L R R3
+L Device:R R3
 U 1 1 5BABCC22
 P 6400 3000
 F 0 "R3" V 6480 3000 50  0000 C CNN
 F 1 "4k99" V 6400 3000 50  0000 C CNN
-F 2 "Resistors_SMD:R_0603" V 6330 3000 50  0001 C CNN
+F 2 "Resistor_SMD:R_0603_1608Metric" V 6330 3000 50  0001 C CNN
 F 3 "" H 6400 3000 50  0001 C CNN
 F 4 "GPR06034K99" H 6400 3000 60  0001 C CNN "Part Number"
@@
 $EndComp
 $Comp
-L +3.3V #PWR044
+L pleiades-rescue:+3.3V #PWR044
 U 1 1 5BABCF2C
 P 6800 2700
@@
 $EndComp
 $Comp
-L R R1
+L Device:R R1
 U 1 1 5BAA344D
 P 4450 3000
 F 0 "R1" V 4530 3000 50  0000 C CNN
 F 1 "10k" V 4450 3000 50  0000 C CNN
-F 2 "Resistors_SMD:R_0603" V 4380 3000 50  0001 C CNN
+F 2 "Resistor_SMD:R_0603_1608Metric" V 4380 3000 50  0001 C CNN
 F 3 "" H 4450 3000 50  0001 C CNN
 F 4 "GPR060310K" H 4450 3000 60  0001 C CNN "Part Number"
@@
 $EndComp
 $Comp
-L R R16
+L Device:R R16
 U 1 1 5BAA3454
 P 4650 3000
 F 0 "R16" V 4730 3000 50  0000 C CNN
 F 1 "10k" V 4650 3000 50  0000 C CNN
-F 2 "Resistors_SMD:R_0603" V 4580 3000 50  0001 C CNN
+F 2 "Resistor_SMD:R_0603_1608Metric" V 4580 3000 50  0001 C CNN
 F 3 "" H 4650 3000 50  0001 C CNN
 F 4 "GPR060310K" H 4650 3000 60  0001 C CNN "Part Number"
@@
 $EndComp
 $Comp
-L R R17
+L Device:R R17
 U 1 1 5BAA345B
 P 4850 3000
 F 0 "R17" V 4930 3000 50  0000 C CNN
 F 1 "10k" V 4850 3000 50  0000 C CNN
-F 2 "Resistors_SMD:R_0603" V 4780 3000 50  0001 C CNN
+F 2 "Resistor_SMD:R_0603_1608Metric" V 4780 3000 50  0001 C CNN
 F 3 "" H 4850 3000 50  0001 C CNN
 F 4 "GPR060310K" H 4850 3000 60  0001 C CNN "Part Number"
@@
 $EndComp
 $Comp
-L R R10
+L Device:R R10
 U 1 1 5BAA4A0F
 P 6700 3000
 F 0 "R10" V 6780 3000 50  0000 C CNN
 F 1 "10k" V 6700 3000 50  0000 C CNN
-F 2 "Resistors_SMD:R_0603" V 6630 3000 50  0001 C CNN
+F 2 "Resistor_SMD:R_0603_1608Metric" V 6630 3000 50  0001 C CNN
 F 3 "" H 6700 3000 50  0001 C CNN
 F 4 "GPR060310K" H 6700 3000 60  0001 C CNN "Part Number"
@@
 $EndComp
 $Comp
-L R R12
+L Device:R R12
 U 1 1 5BAA4A16
 P 6900 3000
 F 0 "R12" V 6980 3000 50  0000 C CNN
 F 1 "10k" V 6900 3000 50  0000 C CNN
-F 2 "Resistors_SMD:R_0603" V 6830 3000 50  0001 C CNN
+F 2 "Resistor_SMD:R_0603_1608Metric" V 6830 3000 50  0001 C CNN
 F 3 "" H 6900 3000 50  0001 C CNN
 F 4 "GPR060310K" H 6900 3000 60  0001 C CNN "Part Number"
@@
 $EndComp
 $Comp
-L R R18
+L Device:R R18
 U 1 1 5BAA4A9A
 P 7200 3000
 F 0 "R18" V 7280 3000 50  0000 C CNN
 F 1 "10k" V 7200 3000 50  0000 C CNN
-F 2 "Resistors_SMD:R_0603" V 7130 3000 50  0001 C CNN
+F 2 "Resistor_SMD:R_0603_1608Metric" V 7130 3000 50  0001 C CNN
 F 3 "" H 7200 3000 50  0001 C CNN
 F 4 "GPR060310K" H 7200 3000 60  0001 C CNN "Part Number"
@@
 $EndComp
 $Comp
-L R R19
+L Device:R R19
 U 1 1 5BAA4AA1
 P 7400 3000
 F 0 "R19" V 7480 3000 50  0000 C CNN
 F 1 "10k" V 7400 3000 50  0000 C CNN
-F 2 "Resistors_SMD:R_0603" V 7330 3000 50  0001 C CNN
+F 2 "Resistor_SMD:R_0603_1608Metric" V 7330 3000 50  0001 C CNN
 F 3 "" H 7400 3000 50  0001 C CNN
 F 4 "GPR060310K" H 7400 3000 60  0001 C CNN "Part Number"
@@
 $EndComp
 Wire Wire Line
-	5450 2500 5450 3050
-Wire Wire Line
-	4450 2550 5700 2550
+	5450 2500 5450 2550
+Wire Wire Line
+	4450 2550 4650 2550
 Connection ~ 5450 2550
 Wire Wire Line
-	5450 4950 5450 5050
+	5450 4950 5450 5000
 Wire Wire Line
 	6650 4650 6750 4650
@@
 	5050 4450 5000 4450
 Wire Wire Line
-	5000 4450 5000 5000
+	5000 4450 5000 4550
 Wire Wire Line
 	5000 4550 5050 4550
@@
 	5700 2850 5700 2900
 Wire Wire Line
-	4000 3450 5050 3450
-Wire Wire Line
-	4000 3250 5050 3250
-Wire Wire Line
-	4000 3350 5050 3350
-Wire Wire Line
-	5950 3250 8300 3250
-Wire Wire Line
-	5950 3650 8300 3650
-Wire Wire Line
-	5950 4050 8300 4050
-Wire Wire Line
-	5950 3350 8300 3350
-Wire Wire Line
-	5950 4150 8300 4150
-Wire Wire Line
-	5950 3750 8300 3750
-Wire Wire Line
-	5950 3850 8300 3850
-Wire Wire Line
-	5950 4250 8300 4250
+	4000 3450 4850 3450
+Wire Wire Line
+	4000 3250 4450 3250
+Wire Wire Line
+	4000 3350 4650 3350
+Wire Wire Line
+	5950 3250 6200 3250
+Wire Wire Line
+	5950 3650 6700 3650
+Wire Wire Line
+	5950 4050 7200 4050
+Wire Wire Line
+	5950 3350 6400 3350
+Wire Wire Line
+	5950 4150 7400 4150
+Wire Wire Line
+	5950 3750 6900 3750
+Wire Wire Line
+	5950 3850 7900 3850
+Wire Wire Line
+	5950 4250 8100 4250
 Wire Wire Line
 	5950 4650 6350 4650
 Wire Wire Line
-	5950 3450 8300 3450
+	5950 3450 7700 3450
 Wire Wire Line
 	6800 2700 6800 2800
 Wire Wire Line
-	6200 2800 8100 2800
+	6200 2800 6400 2800
 Wire Wire Line
 	6200 2800 6200 2850
@@
 	7400 3150 7400 4150
 Connection ~ 7400 4150
+Wire Wire Line
+	5450 2550 5450 3050
+Wire Wire Line
+	5450 2550 5700 2550
+Wire Wire Line
+	5000 4550 5000 4650
+Wire Wire Line
+	5000 4650 5000 5000
+Wire Wire Line
+	5450 5000 5450 5050
+Wire Wire Line
+	6400 2800 6700 2800
+Wire Wire Line
+	6700 2800 6800 2800
+Wire Wire Line
+	6800 2800 6900 2800
+Wire Wire Line
+	6900 2800 7200 2800
+Wire Wire Line
+	7700 2800 7900 2800
+Wire Wire Line
+	7900 2800 8100 2800
+Wire Wire Line
+	7700 3450 8300 3450
+Wire Wire Line
+	7900 3850 8300 3850
+Wire Wire Line
+	8100 4250 8300 4250
+Wire Wire Line
+	6900 3750 8300 3750
+Wire Wire Line
+	6700 3650 8300 3650
+Wire Wire Line
+	6400 3350 8300 3350
+Wire Wire Line
+	6200 3250 8300 3250
+Wire Wire Line
+	4650 2550 4850 2550
+Wire Wire Line
+	4850 2550 5450 2550
+Wire Wire Line
+	4450 3250 5050 3250
+Wire Wire Line
+	4650 3350 5050 3350
+Wire Wire Line
+	4850 3450 5050 3450
+Wire Wire Line
+	7200 2800 7400 2800
+Wire Wire Line
+	7400 2800 7700 2800
+Wire Wire Line
+	7200 4050 8300 4050
+Wire Wire Line
+	7400 4150 8300 4150
 $EndSCHEMATC
