File: ecad/climate/celaeno/celeano.sch (KiCad schematic (older format))
At the start: 8 parts, among them J1 MCV 1,5/ 2-G-3,5, J2 MCV 1,5/ 2-G-3,5, J3 MCV 1,5/ 2-G-3,5, J5 47053-1000, J6 47053-1000, J7 Conn_01x04, J8 640454-2, J9 640454-2

Commit message: Small Correction for Production
Parts:
- J7: value Conn_01x04 -> PT 1,5/4-3,5-H; footprint (none) -> TerminalBlock_Phoenix:TerminalBlock_Phoenix_PT-1,5-4-3.5-H_1x04_P3.50mm_Horizontal; Part Number (none) -> PT 1,5/4-3,5-H
Changed lines of the file:
@@
 P 10300 1900
 F 0 "J7" H 10380 1892 50  0000 L CNN
-F 1 "Conn_01x04" H 10380 1801 50  0000 L CNN
-F 2 "" H 10300 1900 50  0001 C CNN
+F 1 "PT 1,5/4-3,5-H" H 10380 1801 50  0000 L CNN
+F 2 "TerminalBlock_Phoenix:TerminalBlock_Phoenix_PT-1,5-4-3.5-H_1x04_P3.50mm_Horizontal" H 10300 1900 50  0001 C CNN
 F 3 "~" H 10300 1900 50  0001 C CNN
+F 4 "PT 1,5/4-3,5-H" H 10300 1900 50  0001 C CNN "Part Number"
 	1    10300 1900
 	1    0    0    -1
@@
 F5 "SDA_5V" B R 4850 4200 60
 F6 "SCL_5V" O R 4850 4300 60
-F7 "LVL_0" I R 4850 3350 50
-F8 "LVL_1" I R 4850 3450 50
+F7 "LVL_0" I R 4850 3450 50
+F8 "LVL_1" I R 4850 3550 50
+F9 "RELAY" O R 4850 3250 50
 $EndSheet
 $Comp
@@
 	10400 3100 7700 3100
 Wire Wire Line
-	7700 3100 7700 3450
+	7600 2800 10400 2800
 Wire Wire Line
-	7700 3450 4850 3450
+	4850 3550 7700 3550
 Wire Wire Line
-	4850 3350 7600 3350
+	7700 3100 7700 3550
 Wire Wire Line
-	7600 3350 7600 2800
+	7600 3450 4850 3450
 Wire Wire Line
-	7600 2800 10400 2800
+	7600 2800 7600 3450
+Wire Wire Line
+	4850 3250 7500 3250
+Wire Wire Line
+	7500 3250 7500 2700
+Wire Wire Line
+	7500 2700 8400 2700
+Wire Wire Line
+	8400 2700 8400 1950
+Wire Wire Line
+	8400 1950 8700 1950
 $EndSCHEMATC

Commit message: Corrects Celaeno silkscreen
Parts:
- J7: Part Number PT 1,5/4-3,5-H -> 1984633
Changed lines of the file:
@@
 F 2 "TerminalBlock_Phoenix:TerminalBlock_Phoenix_PT-1,5-4-3.5-H_1x04_P3.50mm_Horizontal" H 10300 1900 50  0001 C CNN
 F 3 "~" H 10300 1900 50  0001 C CNN
-F 4 "PT 1,5/4-3,5-H" H 10300 1900 50  0001 C CNN "Part Number"
+F 4 "1984633" H 10300 1900 50  0001 C CNN "Part Number"
 	1    10300 1900
 	1    0    0    -1
