File: ecad/climate/celaeno/Relay.sch (KiCad schematic (older format))
At the start: 4 parts, among them K1 FINDER-32.21-x000, Q4 BSS138

Commit message: Small Correction for Production
Parts:
- removed K1: FINDER-32.21-x000, Relay_THT:Relay_SPST_Finder_32.21-x300, symbol Relay:FINDER-32.21-x000
- added K1: G5Q-1A4-EU DC5, Relay_THT:Relay_SPST_Omron-G5Q-1A, symbol Relay:G5Q-1A
- D2: value MCL4148 -> 1N4148WS; footprint Diode_SMD:D_MicroMELF -> Diode_SMD:D_SOD-323F; Part Number MCL4148-TR -> 1N4148WS
Connections:
- no-connect marks 1 -> 0
Changed lines of the file:
@@
 $Descr A4 11693 8268
 encoding utf-8
-Sheet 11 8
+Sheet 7 8
 Title ""
 Date ""
@@
 $EndDescr
 $Comp
-L Relay:FINDER-32.21-x000 K?
-U 1 1 5BB41828
-P 5850 3450
-AR Path="/5BB4177A/5BB41828" Ref="K?"  Part="1"
-AR Path="/5BB53554/5BB41828" Ref="K?"  Part="1"
-AR Path="/5BB4D604/5BB41828" Ref="K1"  Part="1"
-F 0 "K1" H 6280 3496 50  0000 L CNN
-F 1 "FINDER-32.21-x000" H 6280 3405 50  0000 L CNN
-F 2 "Relay_THT:Relay_SPST_Finder_32.21-x300" H 7120 3420 50  0001 C CNN
-F 3 "https://gfinder.findernet.com/assets/Series/355/S32EN.pdf" H 5850 3450 50  0001 C CNN
-F 4 "32.21.7.005.4000" H 5850 3450 50  0001 C CNN "Part Number"
-	1    5850 3450
-	1    0    0    -1
-$EndComp
-$Comp
 L Device:D D?
 U 1 1 5BB41B1C
@@
 AR Path="/5BB4D604/5BB41B1C" Ref="D2"  Part="1"
 F 0 "D2" H 5200 3500 50  0000 C CNN
-F 1 "MCL4148" H 5200 3300 50  0000 C CNN
-F 2 "Diode_SMD:D_MicroMELF" H 5200 3400 50  0001 C CNN
+F 1 "1N4148WS" H 5200 3300 50  0000 C CNN
+F 2 "Diode_SMD:D_SOD-323F" H 5200 3400 50  0001 C CNN
 F 3 "" H 5200 3400 50  0001 C CNN
-F 4 "MCL4148-TR" H 5200 3400 60  0001 C CNN "Part Number"
+F 4 "1N4148WS" H 5200 3400 60  0001 C CNN "Part Number"
 	1    5200 3400
 	0    1    1    0
@@
 AR Path="/5BB4177A/5BB45131" Ref="#PWR?"  Part="1"
 AR Path="/5BB53554/5BB45131" Ref="#PWR?"  Part="1"
-AR Path="/5BB4D604/5BB45131" Ref="#PWR0101"  Part="1"
-F 0 "#PWR0101" H 5650 2600 50  0001 C CNN
+AR Path="/5BB4D604/5BB45131" Ref="#PWR0106"  Part="1"
+F 0 "#PWR0106" H 5650 2600 50  0001 C CNN
 F 1 "+5V" H 5665 2923 50  0000 C CNN
 F 2 "" H 5650 2750 50  0001 C CNN
@@
 AR Path="/5BB4177A/5BB45528" Ref="#PWR?"  Part="1"
 AR Path="/5BB53554/5BB45528" Ref="#PWR?"  Part="1"
-AR Path="/5BB4D604/5BB45528" Ref="#PWR0102"  Part="1"
-F 0 "#PWR0102" H 5650 4700 50  0001 C CNN
+AR Path="/5BB4D604/5BB45528" Ref="#PWR0107"  Part="1"
+F 0 "#PWR0107" H 5650 4700 50  0001 C CNN
 F 1 "GND" H 5655 4777 50  0000 C CNN
 F 2 "" H 5650 4950 50  0001 C CNN
@@
 Connection ~ 5650 4800
 Connection ~ 5200 4200
-NoConn ~ 5950 3150
 Text HLabel 4400 4200 0    50   Input ~ 0
 CMD
 Wire Wire Line
 	4400 4200 5200 4200
+Text HLabel 6500 3900 2    50   BiDi ~ 0
+A
 Text HLabel 6500 2950 2    50   BiDi ~ 0
-A
-Text HLabel 6500 3900 2    50   BiDi ~ 0
 B
 Wire Wire Line
@@
 Wire Wire Line
 	6050 3900 6050 3750
+$Comp
+L Relay:G5Q-1A K1
+U 1 1 5BB5DA17
+P 5850 3450
+F 0 "K1" H 6250 3300 50  0000 R CNN
+F 1 "G5Q-1A4-EU DC5" H 6850 3600 50  0000 R CNN
+F 2 "Relay_THT:Relay_SPST_Omron-G5Q-1A" H 6200 3400 50  0001 L CNN
+F 3 "https://www.omron.com/ecb/products/pdf/en-g5q.pdf" H 6950 3150 50  0001 C CNN
+F 4 "G5Q-1A4-EU DC5" H 5850 3450 50  0001 C CNN "Part Number"
+	1    5850 3450
+	1    0    0    1
+$EndComp
 Wire Wire Line
-	6150 3150 6150 2950
+	6050 3150 6050 2950
 Wire Wire Line
-	6150 2950 6500 2950
+	6050 2950 6500 2950
 $EndSCHEMATC

Commit message: Licenses Climate PCB under OHL v1.2
Other:
- note added: "© 2018 Université de Lausanne\n\nThis documentation describes Open Hardware and is licensed under the\nCERN OHL v. 1.2.\n\nYou may redistribute and modify this documentation under the terms of\nthe CERN OHL v.1.2. (http://ohwr.org/cernohl). This documentation is\ndistributed WITHOUT ANY EXPRESS OR IMPLIED WARRANTY,\nINCLUDING OF MERCHANTABILITY, SATISFACTORY QUALITY AND\nFITNESS FOR A PARTICULAR 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"
Changed lines of the file:
@@
 EESchema Schematic File Version 4
-LIBS:celeano-cache
+LIBS:celaeno-cache
 EELAYER 26 0
 EELAYER END
@@
 encoding utf-8
 Sheet 7 8
-Title ""
-Date ""
-Rev ""
-Comp ""
-Comment1 ""
-Comment2 ""
+Title "230V 5A Relay"
+Date "06/11/2018"
+Rev "A"
+Comp "Université de Lausanne"
+Comment1 "Author: Alexandre Tuleu"
+Comment2 "Licensed under the CERN OHL v1.2"
 Comment3 ""
 Comment4 ""
@@
 Wire Wire Line
 	6050 2950 6500 2950
+Text Notes 550  7750 0    50   ~ 0
+© 2018 Université de Lausanne\n\nThis documentation describes Open Hardware and is licensed under the\nCERN OHL v. 1.2.\n\nYou may redistribute and modify this documentation under the terms of\nthe CERN OHL v.1.2. (http://ohwr.org/cernohl). This documentation is\ndistributed WITHOUT ANY EXPRESS OR IMPLIED WARRANTY,\nINCLUDING OF MERCHANTABILITY, SATISFACTORY QUALITY AND\nFITNESS FOR A PARTICULAR PURPOSE. Please see the CERN OHL v.1.2\nfor applicable conditions
 $EndSCHEMATC

Commit message: Updates board for manufacturing
Parts:
- R13: value 47k5 -> 47k; Part Number GPR060347k5 -> GPR060347K0
Changed lines of the file:
@@
 AR Path="/5BB4D604/5BB45339" Ref="R13"  Part="1"
 F 0 "R13" V 5280 4550 50  0000 C CNN
-F 1 "47k5" V 5200 4550 50  0000 C CNN
+F 1 "47k" V 5200 4550 50  0000 C CNN
 F 2 "Resistor_SMD:R_0603_1608Metric" V 5130 4550 50  0001 C CNN
 F 3 "" H 5200 4550 50  0001 C CNN
-F 4 "GPR060347k5" H 5200 4550 60  0001 C CNN "Part Number"
+F 4 "GPR060347K0" H 5200 4550 60  0001 C CNN "Part Number"
 	1    5200 4550
 	-1   0    0    1
