File: ecad/climate/celaeno/i2c_level_shifter.kicad_sch (KiCad schematic)
At the start: 9 parts, among them Q1 BSS138, Q2 BSS138, Q3 BSS138

Commit message: Updates Celaeno for production
Parts:
- Q1, Q2, Q3: MPN (none) -> BSS138
- R1, R10, R11, R12, R2, R3: MPN (none) -> GPR060310K
Changed lines of the file:
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@@
 			)
 		)
-		(property "MPN" ""
+		(property "MPN" "BSS138"
 			(at 147.32 95.25 0)
 			(effects
@@
 			)
 		)
-		(property "MPN" ""
+		(property "MPN" "BSS138"
 			(at 160.02 86.36 0)
 			(effects
@@
 			)
 		)
-		(property "MPN" ""
+		(property "MPN" "BSS138"
 			(at 172.72 77.47 0)
 			(effects
@@
 			)
 		)
-		(property "MPN" ""
+		(property "MPN" "GPR060310K"
 			(at 121.92 63.5 0)
 			(effects
@@
 			)
 		)
-		(property "MPN" ""
+		(property "MPN" "GPR060310K"
 			(at 129.54 63.5 0)
 			(effects
@@
 			)
 		)
-		(property "MPN" ""
+		(property "MPN" "GPR060310K"
 			(at 135.89 63.5 0)
 			(effects
@@
 			)
 		)
-		(property "MPN" ""
+		(property "MPN" "GPR060310K"
 			(at 184.15 63.5 0)
 			(effects
@@
 			)
 		)
-		(property "MPN" ""
+		(property "MPN" "GPR060310K"
 			(at 191.77 63.5 0)
 			(effects
@@
 			)
 		)
-		(property "MPN" ""
+		(property "MPN" "GPR060310K"
 			(at 198.12 63.5 0)
 			(effects
