File: ecad/common/12V5VDCDC_LDO.sch (KiCad schematic (older format))
At the start: 15 parts, among them U4 MIC4680YM, U5 LP3985IM5-5.0_NOPB

Commit message: Small Correction for Production
Parts:
- U5: Part Number (none) -> LP3985IM5-5.0/NOPB
Changed lines of the file:
@@
 F 2 "Package_TO_SOT_SMD:SOT-23-5" H 5400 4750 60  0001 C CNN
 F 3 "" H 5400 4750 60  0001 C CNN
+F 4 "LP3985IM5-5.0/NOPB" H 5450 4750 50  0001 C CNN "Part Number"
 	1    5450 4750
 	1    0    0    -1

Commit message: Licenses Climate PCB under OHL v1.2
Other:
- note added: "© 2018 Université de Lausanne\n\nThis documentation describes Open Hardware and is licensed under the\nCERN OHL v. 1.2.\n\nYou may redistribute and modify this documentation under the terms of\nthe CERN OHL v.1.2. (http://ohwr.org/cernohl). This documentation is\ndistributed WITHOUT ANY EXPRESS OR IMPLIED WARRANTY,\nINCLUDING OF MERCHANTABILITY, SATISFACTORY QUALITY AND\nFITNESS FOR A PARTICULAR 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"
Changed lines of the file:
@@
 EESchema Schematic File Version 4
-LIBS:celeano-cache
+LIBS:celaeno-cache
 EELAYER 26 0
 EELAYER END
@@
 encoding utf-8
 Sheet 4 8
-Title ""
-Date ""
-Rev ""
-Comp ""
-Comment1 ""
-Comment2 ""
+Title "5V Bulk Converter w/ LDO"
+Date "06/11/2018"
+Rev "A"
+Comp "Université de Lausanne"
+Comment1 "Author: Alexandre Tuleu"
+Comment2 "Licensed under the CERN OHL v1.2"
 Comment3 ""
 Comment4 ""
@@
 	1    0    0    -1
 $EndComp
+Text Notes 550  7750 0    50   ~ 0
+© 2018 Université de Lausanne\n\nThis documentation describes Open Hardware and is licensed under the\nCERN OHL v. 1.2.\n\nYou may redistribute and modify this documentation under the terms of\nthe CERN OHL v.1.2. (http://ohwr.org/cernohl). This documentation is\ndistributed WITHOUT ANY EXPRESS OR IMPLIED WARRANTY,\nINCLUDING OF MERCHANTABILITY, SATISFACTORY QUALITY AND\nFITNESS FOR A PARTICULAR PURPOSE. Please see the CERN OHL v.1.2\nfor applicable conditions
 $EndSCHEMATC
