File: ecad/common/CAN_transceiver.sch (KiCad schematic (older format))
At the start: 2 parts, among them U3 MCP2561-E/SN

Commit message: Licenses Climate PCB under OHL v1.2
Other:
- note added: "© 2018 Université de Lausanne\n\nThis documentation describes Open Hardware and is licensed under the\nCERN OHL v. 1.2.\n\nYou may redistribute and modify this documentation under the terms of\nthe CERN OHL v.1.2. (http://ohwr.org/cernohl). This documentation is\ndistributed WITHOUT ANY EXPRESS OR IMPLIED WARRANTY,\nINCLUDING OF MERCHANTABILITY, SATISFACTORY QUALITY AND\nFITNESS FOR A PARTICULAR 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"
Changed lines of the file:
@@
 EESchema Schematic File Version 4
-LIBS:power
-LIBS:74xx
-LIBS:fort
-LIBS:arke-cache
+LIBS:zeus-cache
 EELAYER 26 0
 EELAYER END
 $Descr A4 11693 8268
 encoding utf-8
-Sheet 4 5
-Title ""
-Date ""
-Rev ""
-Comp ""
-Comment1 ""
-Comment2 ""
+Sheet 2 10
+Title "CAN Transceiver"
+Date "06/11/2018"
+Rev "A"
+Comp "Université de Lausanne"
+Comment1 "Author: Alexandre Tuleu"
+Comment2 "Licensed under the CERN OHL v1.2"
 Comment3 ""
 Comment4 ""
@@
 Wire Wire Line
 	5750 2650 5750 3400
+Text Notes 550  7750 0    50   ~ 0
+© 2018 Université de Lausanne\n\nThis documentation describes Open Hardware and is licensed under the\nCERN OHL v. 1.2.\n\nYou may redistribute and modify this documentation under the terms of\nthe CERN OHL v.1.2. (http://ohwr.org/cernohl). This documentation is\ndistributed WITHOUT ANY EXPRESS OR IMPLIED WARRANTY,\nINCLUDING OF MERCHANTABILITY, SATISFACTORY QUALITY AND\nFITNESS FOR A PARTICULAR PURPOSE. Please see the CERN OHL v.1.2\nfor applicable conditions
 $EndSCHEMATC

Commit message: Adds TVS diode on fan connector
Parts:
- renumbered C12 to C22, U3 to U9
Changed lines of the file:
@@
 EESchema Schematic File Version 4
-LIBS:arke-cache
+LIBS:master-cache
 EELAYER 26 0
 EELAYER END
 $Descr A4 11693 8268
 encoding utf-8
-Sheet 2 5
+Sheet 6 6
 Title "CAN Transceiver"
-Date "06/11/2018"
+Date "20/11/2018"
 Rev "A"
 Comp "Université de Lausanne"
@@
 $EndDescr
 $Comp
-L Interface_CAN_LIN:MCP2561-E-SN U3
+L Interface_CAN_LIN:MCP2561-E-SN U9
 U 1 1 5BA28540
 P 5750 3800
-F 0 "U3" H 5350 4150 50  0000 L CNN
+F 0 "U9" H 5350 4150 50  0000 L CNN
 F 1 "MCP2561-E/SN" H 5850 4150 50  0000 L CNN
 F 2 "Package_SO:SOIC-8_3.9x4.9mm_P1.27mm" H 5750 3300 50  0001 C CIN
@@
 	5750 4200 5750 4400
 $Comp
-L power:GND #PWR0101
+L power:GND #PWR020
 U 1 1 5BA285D4
 P 5750 4600
-F 0 "#PWR0101" H 5750 4350 50  0001 C CNN
+F 0 "#PWR020" H 5750 4350 50  0001 C CNN
 F 1 "GND" H 5750 4450 50  0000 C CNN
 F 2 "" H 5750 4600 50  0001 C CNN
@@
 Connection ~ 5750 4400
 $Comp
-L Device:C C12
+L Device:C C22
 U 1 1 5BA2863D
 P 5450 2900
-F 0 "C12" H 5475 3000 50  0000 L CNN
+F 0 "C22" H 5475 3000 50  0000 L CNN
 F 1 "100n" H 5475 2800 50  0000 L CNN
 F 2 "Capacitor_SMD:C_0603_1608Metric" H 5488 2750 50  0001 C CNN
@@
 $EndComp
 $Comp
-L power:GND #PWR0102
+L power:GND #PWR019
 U 1 1 5BA28644
 P 5450 3150
-F 0 "#PWR0102" H 5450 2900 50  0001 C CNN
+F 0 "#PWR019" H 5450 2900 50  0001 C CNN
 F 1 "GND" H 5450 3000 50  0000 C CNN
 F 2 "" H 5450 3150 50  0001 C CNN
@@
 	5750 2500 5750 2650
 $Comp
-L power:+5V #PWR0105
+L power:+5V #PWR016
 U 1 1 5BA2868E
 P 5750 2500
-F 0 "#PWR0105" H 5750 2350 50  0001 C CNN
+F 0 "#PWR016" H 5750 2350 50  0001 C CNN
 F 1 "+5V" H 5750 2640 50  0000 C CNN
 F 2 "" H 5750 2500 50  0001 C CNN

Commit message: Corrects anotation of Helios Master
Parts:
- renumbered C22 to C12, U9 to U3
Changed lines of the file:
@@
 $EndDescr
 $Comp
-L Interface_CAN_LIN:MCP2561-E-SN U9
+L Interface_CAN_LIN:MCP2561-E-SN U3
 U 1 1 5BA28540
 P 5750 3800
-F 0 "U9" H 5350 4150 50  0000 L CNN
+F 0 "U3" H 5350 4150 50  0000 L CNN
 F 1 "MCP2561-E/SN" H 5850 4150 50  0000 L CNN
 F 2 "Package_SO:SOIC-8_3.9x4.9mm_P1.27mm" H 5750 3300 50  0001 C CIN
@@
 Connection ~ 5750 4400
 $Comp
-L Device:C C22
+L Device:C C12
 U 1 1 5BA2863D
 P 5450 2900
-F 0 "C22" H 5475 3000 50  0000 L CNN
+F 0 "C12" H 5475 3000 50  0000 L CNN
 F 1 "100n" H 5475 2800 50  0000 L CNN
 F 2 "Capacitor_SMD:C_0603_1608Metric" H 5488 2750 50  0001 C CNN

Commit message: Makes all electronics production ready
Parts:
- C12: Part Number CC0603KRX7R8BB104 -> GPC0603104
Changed lines of the file:
@@
 $Descr A4 11693 8268
 encoding utf-8
-Sheet 6 6
+Sheet 6 8
 Title "CAN Transceiver"
 Date "20/11/2018"
@@
 F 2 "Capacitor_SMD:C_0603_1608Metric" H 5488 2750 50  0001 C CNN
 F 3 "" H 5450 2900 50  0001 C CNN
-F 4 "CC0603KRX7R8BB104" H 5450 2900 60  0001 C CNN "Part Number"
+F 4 "GPC0603104" H 5450 2900 60  0001 C CNN "Part Number"
 	1    5450 2900
 	1    0    0    -1
