File: ecad/common/Fan_controller.sch (KiCad schematic (older format))
At the start: 3 parts, among them U6 EMC2302-1-AIZL-TR, X1 32.768kHz

Commit message: Licenses Climate PCB under OHL v1.2
Other:
- note added: "© 2018 Université de Lausanne\n\nThis documentation describes Open Hardware and is licensed under the\nCERN OHL v. 1.2.\n\nYou may redistribute and modify this documentation under the terms of\nthe CERN OHL v.1.2. (http://ohwr.org/cernohl). This documentation is\ndistributed WITHOUT ANY EXPRESS OR IMPLIED WARRANTY,\nINCLUDING OF MERCHANTABILITY, SATISFACTORY QUALITY AND\nFITNESS FOR A PARTICULAR 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"
Changed lines of the file:
@@
 $Descr A4 11693 8268
 encoding utf-8
-Sheet 7 10
-Title ""
-Date ""
-Rev ""
-Comp ""
-Comment1 ""
-Comment2 ""
+Sheet 5 10
+Title "4 Wire PC FAN Controller"
+Date "06/11/2018"
+Rev "A"
+Comp "Université de Lausanne"
+Comment1 "Author: Alexandre Tuleu"
+Comment2 "Licensed under the CERN OHL v1.2"
 Comment3 ""
 Comment4 ""
@@
 Wire Wire Line
 	6000 4750 6000 4950
+Text Notes 550  7750 0    50   ~ 0
+© 2018 Université de Lausanne\n\nThis documentation describes Open Hardware and is licensed under the\nCERN OHL v. 1.2.\n\nYou may redistribute and modify this documentation under the terms of\nthe CERN OHL v.1.2. (http://ohwr.org/cernohl). This documentation is\ndistributed WITHOUT ANY EXPRESS OR IMPLIED WARRANTY,\nINCLUDING OF MERCHANTABILITY, SATISFACTORY QUALITY AND\nFITNESS FOR A PARTICULAR PURPOSE. Please see the CERN OHL v.1.2\nfor applicable conditions
 $EndSCHEMATC

Commit message: Updates climate board to rev B~dev
 * Changes all Power Connectors to MiniFit-JR 5566-02A to avoid
   someone pluging the power supply on the CAN bus as it will destroy
   all MCP2561 on the bus
 * Fixes issues in Arke:
 ** Crossed Rx/Tx lines
 ** Flipped DB9 connector
 * Fixes and Improvment in Celaeno/Zeus:
 ** Added missing pull-up resistor on tachometer inputs
 ** Removed unecessary 32.268kHz oscillators (they are not working
    properly with manual soldering)
 ** Removed I2C multiplexer as we can add a second EMC2302 with a
   different i2c address to do the same thing. Repaced it by an i2c
   level shifter (tested and working).

Many of these changes still need to be tested before going to
production
Parts:
- removed X1: 32.768kHz, Oscillator:Oscillator_SMD_Abracon_ASE-4Pin_3.2x2.5mm, symbol Oscillator:ASE-xxxMHz
- added R16, R17: 10k, Resistor_SMD:R_0603_1608Metric, symbol Device:R
Connections:
- net labels removed: 32K768_CLK
- wire segments 24 -> 22
- no-connect marks 0 -> 1
Changed lines of the file:
@@
 EESchema Schematic File Version 4
-LIBS:zeus-cache
+LIBS:celaeno-cache
 EELAYER 26 0
 EELAYER END
 $Descr A4 11693 8268
 encoding utf-8
-Sheet 5 10
+Sheet 5 8
 Title "4 Wire PC FAN Controller"
 Date "06/11/2018"
-Rev "A"
+Rev "B"
 Comp "Université de Lausanne"
 Comment1 "Author: Alexandre Tuleu"
@@
 Comment4 ""
 $EndDescr
-$Comp
-L fort:EMC2302-1-AIZL-TR U6
-U 1 1 5BA5AD00
-P 6000 3500
-AR Path="/5BA5AC9B/5BA5AD00" Ref="U6"  Part="1"
-AR Path="/5BAA713E/5BA5AD00" Ref="U61"  Part="1"
-F 0 "U6" H 5600 4050 60  0000 C CNN
-F 1 "EMC2302-1-AIZL-TR" H 6500 2950 60  0000 C CNN
-F 2 "Package_SO:MSOP-10_3x3mm_P0.5mm" H 6100 3500 60  0001 C CNN
-F 3 "" H 6100 3500 60  0001 C CNN
-F 4 "EMC2302-1-AIZL-TR" H 6100 3500 60  0001 C CNN "Part Number"
-	1    6000 3500
-	1    0    0    -1
-$EndComp
 $Comp
 L power:+3.3V #PWR017
@@
 	1    0    0    -1
 $EndComp
-Wire Wire Line
-	6000 4200 6000 4750
 Wire Wire Line
 	6000 2200 6000 2250
@@
 	5700 2700 5700 2600
 $Comp
-L Oscillator:ASE-xxxMHz X1
-U 1 1 5BA5AF21
-P 4750 4300
-AR Path="/5BA5AC9B/5BA5AF21" Ref="X1"  Part="1"
-AR Path="/5BAA713E/5BA5AF21" Ref="X2"  Part="1"
-F 0 "X1" H 4550 4550 50  0000 L CNN
-F 1 "32.768kHz" H 4800 4050 50  0000 L CNN
-F 2 "Oscillator:Oscillator_SMD_Abracon_ASE-4Pin_3.2x2.5mm" H 5450 3950 50  0001 C CNN
-F 3 "" H 4650 4300 50  0001 C CNN
-F 4 "ASEK-32.768KHZ-LRT" H 4750 4300 60  0001 C CNN "Part Number"
-	1    4750 4300
-	1    0    0    -1
-$EndComp
-$Comp
-L power:+3.3V #PWR019
-U 1 1 5BA5B077
-P 4750 3850
-AR Path="/5BA5AC9B/5BA5B077" Ref="#PWR019"  Part="1"
-AR Path="/5BAA713E/5BA5B077" Ref="#PWR038"  Part="1"
-AR Path="/5BA5B077" Ref="#PWR038"  Part="1"
-F 0 "#PWR019" H 4750 3700 50  0001 C CNN
-F 1 "+3.3V" H 4750 3990 50  0000 C CNN
-F 2 "" H 4750 3850 50  0001 C CNN
-F 3 "" H 4750 3850 50  0001 C CNN
-	1    4750 3850
-	1    0    0    -1
-$EndComp
-Wire Wire Line
-	4750 3850 4750 3900
-Wire Wire Line
-	4750 3900 4300 3900
-Wire Wire Line
-	4300 3900 4300 4300
-Wire Wire Line
-	4300 4300 4450 4300
-Connection ~ 4750 3900
-$Comp
 L power:GND #PWR020
 U 1 1 5BA5B0F5
@@
 	1    0    0    -1
 $EndComp
-Wire Wire Line
-	4750 4600 4750 4750
-Wire Wire Line
-	4750 4750 6000 4750
-Connection ~ 6000 4750
-Wire Wire Line
-	5200 4300 5050 4300
-Wire Wire Line
-	5200 3750 5200 4300
-Wire Wire Line
-	5200 3750 5350 3750
-Text HLabel 6900 3300 2    60   Output ~ 0
+Text HLabel 8150 3300 2    60   Output ~ 0
 PWM1
-Text HLabel 6900 3600 2    60   Output ~ 0
+Text HLabel 8150 3600 2    60   Output ~ 0
 PWM2
-Text HLabel 6900 3400 2    60   Input ~ 0
+Text HLabel 8150 3400 2    60   Input ~ 0
 TACH1
-Text HLabel 6900 3700 2    60   Input ~ 0
+Text HLabel 8150 3700 2    60   Input ~ 0
 TACH2
-Wire Wire Line
-	6650 3300 6900 3300
-Wire Wire Line
-	6650 3400 6900 3400
-Wire Wire Line
-	6650 3600 6900 3600
-Wire Wire Line
-	6650 3700 6900 3700
-Text HLabel 5150 3250 0    60   Output ~ 0
-~ALERT
 Text HLabel 5150 3450 0    60   BiDi ~ 0
 SDA
@@
 	5150 3450 5350 3450
 Wire Wire Line
-	5150 3250 5350 3250
-Text Label 5200 4300 0    60   ~ 0
-32K768_CLK
-Wire Wire Line
 	6000 2250 6000 2800
-Wire Wire Line
-	4750 3900 4750 4000
-Wire Wire Line
-	6000 4750 6000 4950
 Text Notes 550  7750 0    50   ~ 0
 © 2018 Université de Lausanne\n\nThis documentation describes Open Hardware and is licensed under the\nCERN OHL v. 1.2.\n\nYou may redistribute and modify this documentation under the terms of\nthe CERN OHL v.1.2. (http://ohwr.org/cernohl). This documentation is\ndistributed WITHOUT ANY EXPRESS OR IMPLIED WARRANTY,\nINCLUDING OF MERCHANTABILITY, SATISFACTORY QUALITY AND\nFITNESS FOR A PARTICULAR PURPOSE. Please see the CERN OHL v.1.2\nfor applicable conditions
+$Comp
+L Device:R R?
+U 1 1 5BE6233F
+P 7350 3050
+AR Path="/5BB3963A/5BE6233F" Ref="R?"  Part="1"
+AR Path="/5BA5AC9B/5BE6233F" Ref="R16"  Part="1"
+F 0 "R16" H 7420 3096 50  0000 L CNN
+F 1 "10k" H 7420 3005 50  0000 L CNN
+F 2 "Resistor_SMD:R_0603_1608Metric" V 7280 3050 50  0001 C CNN
+F 3 "~" H 7350 3050 50  0001 C CNN
+F 4 "GPR060310K" H 7350 3050 50  0001 C CNN "Part Number"
+	1    7350 3050
+	1    0    0    -1
+$EndComp
+$Comp
+L Device:R R?
+U 1 1 5BE6236B
+P 7650 3050
+AR Path="/5BB3963A/5BE6236B" Ref="R?"  Part="1"
+AR Path="/5BA5AC9B/5BE6236B" Ref="R17"  Part="1"
+F 0 "R17" H 7720 3096 50  0000 L CNN
+F 1 "10k" H 7720 3005 50  0000 L CNN
+F 2 "Resistor_SMD:R_0603_1608Metric" V 7580 3050 50  0001 C CNN
+F 3 "~" H 7650 3050 50  0001 C CNN
+F 4 "GPR060310K" H 7650 3050 50  0001 C CNN "Part Number"
+	1    7650 3050
+	1    0    0    -1
+$EndComp
+Wire Wire Line
+	7350 3200 7350 3400
+$Comp
+L power:+3.3V #PWR0108
+U 1 1 5BE6376D
+P 7500 2700
+AR Path="/5BA5AC9B/5BE6376D" Ref="#PWR0108"  Part="1"
+AR Path="/5BAA713E/5BE6376D" Ref="#PWR?"  Part="1"
+AR Path="/5BE6376D" Ref="#PWR?"  Part="1"
+F 0 "#PWR0108" H 7500 2550 50  0001 C CNN
+F 1 "+3.3V" H 7500 2840 50  0000 C CNN
+F 2 "" H 7500 2700 50  0001 C CNN
+F 3 "" H 7500 2700 50  0001 C CNN
+	1    7500 2700
+	1    0    0    -1
+$EndComp
+Wire Wire Line
+	7350 2900 7350 2800
+Wire Wire Line
+	7350 2800 7500 2800
+Wire Wire Line
+	7650 2900 7650 2800
+Wire Wire Line
+	7500 2800 7500 2700
+Connection ~ 7500 2800
+Wire Wire Line
+	7500 2800 7650 2800
+Wire Wire Line
+	7650 3200 7650 3700
+Wire Wire Line
+	6000 4200 6000 4950
+NoConn ~ 5350 3750
+Wire Wire Line
+	6650 3400 7350 3400
+Wire Wire Line
+	6650 3700 7650 3700
+Wire Wire Line
+	6650 3600 8150 3600
+Wire Wire Line
+	6650 3300 8150 3300
+Connection ~ 7350 3400
+Wire Wire Line
+	7350 3400 8150 3400
+Connection ~ 7650 3700
+Wire Wire Line
+	7650 3700 8150 3700
+Text HLabel 5150 3250 0    50   Output ~ 0
+~ALERT
+$Comp
+L fort:EMC2302-1-AIZL-TR U6
+U 1 1 5BA5AD00
+P 6000 3500
+AR Path="/5BA5AC9B/5BA5AD00" Ref="U6"  Part="1"
+AR Path="/5BAA713E/5BA5AD00" Ref="U61"  Part="1"
+F 0 "U6" H 5600 4050 60  0000 C CNN
+F 1 "EMC2302-1-AIZL-TR" H 6500 2950 60  0000 C CNN
+F 2 "Package_SO:MSOP-10_3x3mm_P0.5mm" H 6100 3500 60  0001 C CNN
+F 3 "" H 6100 3500 60  0001 C CNN
+F 4 "EMC2302-1-AIZL-TR" H 6100 3500 60  0001 C CNN "Part Number"
+	1    6000 3500
+	1    0    0    -1
+$EndComp
+Wire Wire Line
+	5150 3250 5350 3250
 $EndSCHEMATC

Commit message: Adds TVS diode on fan connector
Parts:
- added D5, D7: CPDT-5V0-HF, Package_TO_SOT_SMD:SOT-23, symbol Device:D_TVS_x2_AAC
- added R18, R19, R20, R21: 2k2, Resistor_SMD:R_0603_1608Metric, symbol Device:R
- R16, R17: value 10k -> 47k; Part Number GPR060310K -> GPR060347K0
Connections:
- net labels added: PWM1_PR, PWM2_PR, TACH1_PR, TACH2_PR
- wire segments 22 -> 59
Other:
- note added: "High Series resistor for ESD protection"
- moved on the sheet: C5

Commit message: Corrects anotation of Helios Master
Parts:
- D5, D7: value CPDT-5V0-HF -> CPDT-5V0USP-HF; Part Number CPDT-5V0-HF -> CPDT-5V0USP-HF
Changed lines of the file:
@@
 P 7100 4300
 F 0 "D5" H 7100 4516 50  0000 C CNN
-F 1 "CPDT-5V0-HF" H 7100 4425 50  0000 C CNN
+F 1 "CPDT-5V0USP-HF" H 7100 4425 50  0000 C CNN
 F 2 "Package_TO_SOT_SMD:SOT-23" H 6950 4300 50  0001 C CNN
 F 3 "~" H 6950 4300 50  0001 C CNN
-F 4 "CPDT-5V0-HF" H 7100 4300 50  0001 C CNN "Part Number"
+F 4 "CPDT-5V0USP-HF" H 7100 4300 50  0001 C CNN "Part Number"
 	1    7100 4300
 	1    0    0    -1
@@
 P 8050 4300
 F 0 "D7" H 8050 4516 50  0000 C CNN
-F 1 "CPDT-5V0-HF" H 8050 4425 50  0000 C CNN
+F 1 "CPDT-5V0USP-HF" H 8050 4425 50  0000 C CNN
 F 2 "Package_TO_SOT_SMD:SOT-23" H 7900 4300 50  0001 C CNN
 F 3 "~" H 7900 4300 50  0001 C CNN
-F 4 "CPDT-5V0-HF" H 8050 4300 50  0001 C CNN "Part Number"
+F 4 "CPDT-5V0USP-HF" H 8050 4300 50  0001 C CNN "Part Number"
 	1    8050 4300
 	1    0    0    -1

Commit message: Updates board for manufacturing
Parts:
- C5: value 100nF -> 100n; Part Number 06035C104KAT2A -> CC0603KRX7R8BB104
- R18, R19, R20, R21: Part Number GPR06032K20 -> GPR06032K2
- renumbered D5 to D1
Changed lines of the file:
@@
 AR Path="/5BF0B864/5BA5AE71" Ref="C1"  Part="1"
 F 0 "C5" H 3775 2500 50  0000 L CNN
-F 1 "100nF" H 3775 2300 50  0000 L CNN
+F 1 "100n" H 3775 2300 50  0000 L CNN
 F 2 "Capacitor_SMD:C_0603_1608Metric" H 3788 2250 50  0001 C CNN
 F 3 "" H 3750 2400 50  0001 C CNN
-F 4 "06035C104KAT2A" H 3750 2400 60  0001 C CNN "Part Number"
+F 4 "CC0603KRX7R8BB104" H 3750 2400 60  0001 C CNN "Part Number"
 	1    3750 2400
 	1    0    0    -1
@@
 F 1 "47k" H 5720 2955 50  0000 L CNN
 F 2 "Resistor_SMD:R_0603_1608Metric" V 5580 3000 50  0001 C CNN
-F 3 "~" H 5650 3000 50  0001 C CNN
+F 3 "" H 5650 3000 50  0001 C CNN
 F 4 "GPR060347K0" H 5650 3000 50  0001 C CNN "Part Number"
 	1    5650 3000
@@
 F 1 "47k" H 6020 2955 50  0000 L CNN
 F 2 "Resistor_SMD:R_0603_1608Metric" V 5880 3000 50  0001 C CNN
-F 3 "~" H 5950 3000 50  0001 C CNN
+F 3 "" H 5950 3000 50  0001 C CNN
 F 4 "GPR060347K0" H 5950 3000 50  0001 C CNN "Part Number"
 	1    5950 3000
@@
 F 2 "Resistor_SMD:R_0603_1608Metric" V 6480 3150 50  0001 C CNN
 F 3 "~" H 6550 3150 50  0001 C CNN
-F 4 "GPR06032K20" H 6550 3150 50  0001 C CNN "Part Number"
+F 4 "GPR06032K2" H 6550 3150 50  0001 C CNN "Part Number"
 	1    6550 3150
 	0    1    1    0
@@
 	5950 3650 4700 3650
 $Comp
-L Device:D_TVS_x2_AAC D5
+L Device:D_TVS_x2_AAC D1
 U 1 1 5BEFC8EC
 P 7100 4300
-F 0 "D5" H 7100 4516 50  0000 C CNN
+F 0 "D1" H 7100 4516 50  0000 C CNN
 F 1 "CPDT-5V0USP-HF" H 7100 4425 50  0000 C CNN
 F 2 "Package_TO_SOT_SMD:SOT-23" H 6950 4300 50  0001 C CNN
@@
 F 2 "Resistor_SMD:R_0603_1608Metric" V 6480 3350 50  0001 C CNN
 F 3 "~" H 6550 3350 50  0001 C CNN
-F 4 "GPR06032K20" H 6550 3350 50  0001 C CNN "Part Number"
+F 4 "GPR06032K2" H 6550 3350 50  0001 C CNN "Part Number"
 	1    6550 3350
 	0    1    1    0
@@
 F 2 "Resistor_SMD:R_0603_1608Metric" V 6480 3550 50  0001 C CNN
 F 3 "~" H 6550 3550 50  0001 C CNN
-F 4 "GPR06032K20" H 6550 3550 50  0001 C CNN "Part Number"
+F 4 "GPR06032K2" H 6550 3550 50  0001 C CNN "Part Number"
 	1    6550 3550
 	0    1    1    0
@@
 F 2 "Resistor_SMD:R_0603_1608Metric" V 6480 3750 50  0001 C CNN
 F 3 "~" H 6550 3750 50  0001 C CNN
-F 4 "GPR06032K20" H 6550 3750 50  0001 C CNN "Part Number"
+F 4 "GPR06032K2" H 6550 3750 50  0001 C CNN "Part Number"
 	1    6550 3750
 	0    1    1    0

Commit message: Makes all electronics production ready
Parts:
- C5: Part Number CC0603KRX7R8BB104 -> GPC0603104
Changed lines of the file:
@@
 F 2 "Capacitor_SMD:C_0603_1608Metric" H 3788 2250 50  0001 C CNN
 F 3 "" H 3750 2400 50  0001 C CNN
-F 4 "CC0603KRX7R8BB104" H 3750 2400 60  0001 C CNN "Part Number"
+F 4 "GPC0603104" H 3750 2400 60  0001 C CNN "Part Number"
 	1    3750 2400
 	1    0    0    -1
