File: ecad/common/12V5VDCDC.sch (KiCad schematic (older format))
At the start: 11 parts, among them U4 MIC4680YM

Commit message: Licenses Climate PCB under OHL v1.2
Other:
- note added: "© 2018 Université de Lausanne\n\nThis documentation describes Open Hardware and is licensed under the\nCERN OHL v. 1.2.\n\nYou may redistribute and modify this documentation under the terms of\nthe CERN OHL v.1.2. (http://ohwr.org/cernohl). This documentation is\ndistributed WITHOUT ANY EXPRESS OR IMPLIED WARRANTY,\nINCLUDING OF MERCHANTABILITY, SATISFACTORY QUALITY AND\nFITNESS FOR A PARTICULAR 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"
Changed lines of the file:
@@
 EESchema Schematic File Version 4
-LIBS:power
-LIBS:74xx
-LIBS:fort
-LIBS:arke-cache
+LIBS:zeus-cache
 EELAYER 26 0
 EELAYER END
 $Descr A4 11693 8268
 encoding utf-8
-Sheet 5 5
-Title ""
-Date ""
-Rev ""
-Comp ""
-Comment1 ""
-Comment2 ""
+Sheet 4 10
+Title "5V Buck Converter w/o LDO"
+Date "06/11/2018"
+Rev "A"
+Comp "Université de Lausanne"
+Comment1 "Author: Alexandre Tuleu"
+Comment2 "Licensed under the CERN OHL v1.2"
 Comment3 ""
 Comment4 ""
@@
 Wire Wire Line
 	5750 4450 6150 4450
+Text Notes 550  7750 0    50   ~ 0
+© 2018 Université de Lausanne\n\nThis documentation describes Open Hardware and is licensed under the\nCERN OHL v. 1.2.\n\nYou may redistribute and modify this documentation under the terms of\nthe CERN OHL v.1.2. (http://ohwr.org/cernohl). This documentation is\ndistributed WITHOUT ANY EXPRESS OR IMPLIED WARRANTY,\nINCLUDING OF MERCHANTABILITY, SATISFACTORY QUALITY AND\nFITNESS FOR A PARTICULAR PURPOSE. Please see the CERN OHL v.1.2\nfor applicable conditions
 $EndSCHEMATC

Commit message: Adds TVS diode on fan connector
Parts:
- renumbered C13 to C14, C14 to C15, C15 to C16, C16 to C17, D5 to D6, L1 to L2, L2 to L3, L3 to L4, R6 to R12, R7 to R13, U4 to U7
Changed lines of the file:
@@
 EESchema Schematic File Version 4
-LIBS:arke-cache
+LIBS:master-cache
 EELAYER 26 0
 EELAYER END
 $Descr A4 11693 8268
 encoding utf-8
-Sheet 4 5
+Sheet 4 6
 Title "5V Buck Converter w/o LDO"
-Date "06/11/2018"
+Date "20/11/2018"
 Rev "A"
 Comp "Université de Lausanne"
@@
 $EndDescr
 $Comp
-L fort:MIC4680YM U4
+L fort:MIC4680YM U7
 U 1 1 5BA10D91
 P 5150 3650
-F 0 "U4" H 4950 3150 60  0000 C CNN
+F 0 "U7" H 4950 3150 60  0000 C CNN
 F 1 "MIC4680YM" H 5150 4000 60  0000 C CNN
 F 2 "Package_SO:SOIC-8_3.9x4.9mm_P1.27mm" H 5050 3550 60  0001 C CNN
@@
 $EndComp
 $Comp
-L Device:D_Schottky D5
+L Device:D_Schottky D6
 U 1 1 5BA10E06
 P 6150 3850
-F 0 "D5" H 6150 3950 50  0000 C CNN
+F 0 "D6" H 6150 3950 50  0000 C CNN
 F 1 "B260, 60V, 2A" H 6150 3750 50  0000 C CNN
 F 2 "Diode_SMD:D_SMB" H 6150 3850 50  0001 C CNN
@@
 $EndComp
 $Comp
-L Device:L L2
+L Device:L L3
 U 1 1 5BA10FBE
 P 6700 3450
-F 0 "L2" V 6650 3450 50  0000 C CNN
+F 0 "L3" V 6650 3450 50  0000 C CNN
 F 1 "68uH, 560mA" V 6775 3450 50  0000 C CNN
 F 2 "Inductor_SMD:L_Wuerth_WE-PD2-Typ-MS" H 6700 3450 50  0001 C CNN
@@
 $EndComp
 $Comp
-L Device:R R6
+L Device:R R12
 U 1 1 5BA11005
 P 7250 3750
-F 0 "R6" V 7330 3750 50  0000 C CNN
+F 0 "R12" V 7330 3750 50  0000 C CNN
 F 1 "15k" V 7250 3750 50  0000 C CNN
 F 2 "Resistor_SMD:R_0603_1608Metric" V 7180 3750 50  0001 C CNN
@@
 $EndComp
 $Comp
-L Device:R R7
+L Device:R R13
 U 1 1 5BA1109C
 P 7250 4200
-F 0 "R7" V 7330 4200 50  0000 C CNN
+F 0 "R13" V 7330 4200 50  0000 C CNN
 F 1 "4k87" V 7250 4200 50  0000 C CNN
 F 2 "Resistor_SMD:R_0603_1608Metric" V 7180 4200 50  0001 C CNN
@@
 $EndComp
 $Comp
-L Device:CP C14
+L Device:CP C15
 U 1 1 5BA110CE
 P 7750 3800
-F 0 "C14" H 7775 3900 50  0000 L CNN
+F 0 "C15" H 7775 3900 50  0000 L CNN
 F 1 "470u, 6.3V" H 7775 3700 50  0000 L CNN
 F 2 "Capacitor_Tantalum_SMD:CP_EIA-7343-31_Kemet-D" H 7788 3650 50  0001 C CNN
@@
 $EndComp
 $Comp
-L Device:C C15
+L Device:C C16
 U 1 1 5BA11119
 P 8300 3800
-F 0 "C15" H 8325 3900 50  0000 L CNN
+F 0 "C16" H 8325 3900 50  0000 L CNN
 F 1 "4u7, 6.3V" H 8325 3700 50  0000 L CNN
 F 2 "Capacitor_SMD:C_0603_1608Metric" H 8338 3650 50  0001 C CNN
@@
 $EndComp
 $Comp
-L Device:C C16
+L Device:C C17
 U 1 1 5BA11162
 P 8850 3800
-F 0 "C16" H 8875 3900 50  0000 L CNN
+F 0 "C17" H 8875 3900 50  0000 L CNN
 F 1 "100n" H 8875 3700 50  0000 L CNN
 F 2 "Capacitor_SMD:C_0603_1608Metric" H 8888 3650 50  0001 C CNN
@@
 $EndComp
 $Comp
-L Device:C C13
+L Device:C C14
 U 1 1 5BA11196
 P 3850 3750
-F 0 "C13" H 3875 3850 50  0000 L CNN
+F 0 "C14" H 3875 3850 50  0000 L CNN
 F 1 "22uF, 35V" H 3875 3650 50  0000 L CNN
 F 2 "Capacitor_SMD:C_1206_3216Metric" H 3888 3600 50  0001 C CNN
@@
 $EndComp
 $Comp
-L Device:Ferrite_Bead L3
+L Device:Ferrite_Bead L4
 U 1 1 5BA24C16
 P 9450 3450
-F 0 "L3" V 9300 3475 50  0000 C CNN
+F 0 "L4" V 9300 3475 50  0000 C CNN
 F 1 "500mA Fuse" V 9600 3450 50  0000 C CNN
 F 2 "Resistor_SMD:R_0603_1608Metric" V 9380 3450 50  0001 C CNN
@@
 $EndComp
 $Comp
-L Device:Ferrite_Bead L1
+L Device:Ferrite_Bead L2
 U 1 1 5BA2521F
 P 3300 3450
-F 0 "L1" V 3150 3475 50  0000 C CNN
+F 0 "L2" V 3150 3475 50  0000 C CNN
 F 1 "500mA Fuse" V 3450 3450 50  0000 C CNN
 F 2 "Resistor_SMD:R_0603_1608Metric" V 3230 3450 50  0001 C CNN
@@
 Connection ~ 4350 4450
 $Comp
-L power:GND #PWR0104
+L power:GND #PWR04
 U 1 1 5BA25F94
 P 5750 4650
-F 0 "#PWR0104" H 5750 4400 50  0001 C CNN
+F 0 "#PWR04" H 5750 4400 50  0001 C CNN
 F 1 "GND" H 5750 4500 50  0000 C CNN
 F 2 "" H 5750 4650 50  0001 C CNN

Commit message: Corrects anotation of Helios Master
Parts:
- renumbered C14 to C13, C15 to C14, C16 to C15, C17 to C16, D6 to D5, L2 to L1, L3 to L2, L4 to L3, R12 to R6, R13 to R7, U7 to U4
Changed lines of the file:
@@
 $EndDescr
 $Comp
-L fort:MIC4680YM U7
+L fort:MIC4680YM U4
 U 1 1 5BA10D91
 P 5150 3650
-F 0 "U7" H 4950 3150 60  0000 C CNN
+F 0 "U4" H 4950 3150 60  0000 C CNN
 F 1 "MIC4680YM" H 5150 4000 60  0000 C CNN
 F 2 "Package_SO:SOIC-8_3.9x4.9mm_P1.27mm" H 5050 3550 60  0001 C CNN
@@
 $EndComp
 $Comp
-L Device:D_Schottky D6
+L Device:D_Schottky D5
 U 1 1 5BA10E06
 P 6150 3850
-F 0 "D6" H 6150 3950 50  0000 C CNN
+F 0 "D5" H 6150 3950 50  0000 C CNN
 F 1 "B260, 60V, 2A" H 6150 3750 50  0000 C CNN
 F 2 "Diode_SMD:D_SMB" H 6150 3850 50  0001 C CNN
@@
 $EndComp
 $Comp
-L Device:L L3
+L Device:L L2
 U 1 1 5BA10FBE
 P 6700 3450
-F 0 "L3" V 6650 3450 50  0000 C CNN
+F 0 "L2" V 6650 3450 50  0000 C CNN
 F 1 "68uH, 560mA" V 6775 3450 50  0000 C CNN
 F 2 "Inductor_SMD:L_Wuerth_WE-PD2-Typ-MS" H 6700 3450 50  0001 C CNN
@@
 $EndComp
 $Comp
-L Device:R R12
+L Device:R R6
 U 1 1 5BA11005
 P 7250 3750
-F 0 "R12" V 7330 3750 50  0000 C CNN
+F 0 "R6" V 7330 3750 50  0000 C CNN
 F 1 "15k" V 7250 3750 50  0000 C CNN
 F 2 "Resistor_SMD:R_0603_1608Metric" V 7180 3750 50  0001 C CNN
@@
 $EndComp
 $Comp
-L Device:R R13
+L Device:R R7
 U 1 1 5BA1109C
 P 7250 4200
-F 0 "R13" V 7330 4200 50  0000 C CNN
+F 0 "R7" V 7330 4200 50  0000 C CNN
 F 1 "4k87" V 7250 4200 50  0000 C CNN
 F 2 "Resistor_SMD:R_0603_1608Metric" V 7180 4200 50  0001 C CNN
@@
 $EndComp
 $Comp
-L Device:CP C15
+L Device:CP C14
 U 1 1 5BA110CE
 P 7750 3800
-F 0 "C15" H 7775 3900 50  0000 L CNN
+F 0 "C14" H 7775 3900 50  0000 L CNN
 F 1 "470u, 6.3V" H 7775 3700 50  0000 L CNN
 F 2 "Capacitor_Tantalum_SMD:CP_EIA-7343-31_Kemet-D" H 7788 3650 50  0001 C CNN
@@
 $EndComp
 $Comp
-L Device:C C16
+L Device:C C15
 U 1 1 5BA11119
 P 8300 3800
-F 0 "C16" H 8325 3900 50  0000 L CNN
+F 0 "C15" H 8325 3900 50  0000 L CNN
 F 1 "4u7, 6.3V" H 8325 3700 50  0000 L CNN
 F 2 "Capacitor_SMD:C_0603_1608Metric" H 8338 3650 50  0001 C CNN
@@
 $EndComp
 $Comp
-L Device:C C17
+L Device:C C16
 U 1 1 5BA11162
 P 8850 3800
-F 0 "C17" H 8875 3900 50  0000 L CNN
+F 0 "C16" H 8875 3900 50  0000 L CNN
 F 1 "100n" H 8875 3700 50  0000 L CNN
 F 2 "Capacitor_SMD:C_0603_1608Metric" H 8888 3650 50  0001 C CNN
@@
 $EndComp
 $Comp
-L Device:C C14
+L Device:C C13
 U 1 1 5BA11196
 P 3850 3750
-F 0 "C14" H 3875 3850 50  0000 L CNN
+F 0 "C13" H 3875 3850 50  0000 L CNN
 F 1 "22uF, 35V" H 3875 3650 50  0000 L CNN
 F 2 "Capacitor_SMD:C_1206_3216Metric" H 3888 3600 50  0001 C CNN
@@
 $EndComp
 $Comp
-L Device:Ferrite_Bead L4
+L Device:Ferrite_Bead L3
 U 1 1 5BA24C16
 P 9450 3450
-F 0 "L4" V 9300 3475 50  0000 C CNN
+F 0 "L3" V 9300 3475 50  0000 C CNN
 F 1 "500mA Fuse" V 9600 3450 50  0000 C CNN
 F 2 "Resistor_SMD:R_0603_1608Metric" V 9380 3450 50  0001 C CNN
@@
 $EndComp
 $Comp
-L Device:Ferrite_Bead L2
+L Device:Ferrite_Bead L1
 U 1 1 5BA2521F
 P 3300 3450
-F 0 "L2" V 3150 3475 50  0000 C CNN
+F 0 "L1" V 3150 3475 50  0000 C CNN
 F 1 "500mA Fuse" V 3450 3450 50  0000 C CNN
 F 2 "Resistor_SMD:R_0603_1608Metric" V 3230 3450 50  0001 C CNN
@@
 Connection ~ 4350 4450
 $Comp
-L power:GND #PWR04
+L power:GND #PWR0102
 U 1 1 5BA25F94
 P 5750 4650
-F 0 "#PWR04" H 5750 4400 50  0001 C CNN
+F 0 "#PWR0102" H 5750 4400 50  0001 C CNN
 F 1 "GND" H 5750 4500 50  0000 C CNN
 F 2 "" H 5750 4650 50  0001 C CNN

Commit message: Updates board for manufacturing
Parts:
- C13: value 22uF, 35V -> 22uF, 25V
Other:
- note added: "VIN: 7V-25V\nVload: 500mA"
- note removed: "VIN: 7V-34V\nVload: 500mA"
Changed lines of the file:
@@
 P 3850 3750
 F 0 "C13" H 3875 3850 50  0000 L CNN
-F 1 "22uF, 35V" H 3875 3650 50  0000 L CNN
+F 1 "22uF, 25V" H 3875 3650 50  0000 L CNN
 F 2 "Capacitor_SMD:C_1206_3216Metric" H 3888 3600 50  0001 C CNN
 F 3 "" H 3850 3750 50  0001 C CNN
@@
 VIN_PROTECTED
 Text Notes 2900 3100 0    60   ~ 0
-VIN: 7V-34V\nVload: 500mA
+VIN: 7V-25V\nVload: 500mA
 Wire Wire Line
 	3850 3450 4700 3450

Commit message: Makes all electronics production ready
Parts:
- C15: Part Number CL10A475KQ8NNNC -> GPC0603475
- C16: Part Number CC0603KRX7R8BB104 -> GPC0603104
- R6: Part Number RMCF0603FT15K0 -> GPR060315k
Changed lines of the file:
@@
 $Descr A4 11693 8268
 encoding utf-8
-Sheet 4 6
+Sheet 4 8
 Title "5V Buck Converter w/o LDO"
 Date "20/11/2018"
@@
 F 2 "Resistor_SMD:R_0603_1608Metric" V 7180 3750 50  0001 C CNN
 F 3 "" H 7250 3750 50  0001 C CNN
-F 4 "RMCF0603FT15K0" H 7250 3750 60  0001 C CNN "Part Number"
+F 4 "GPR060315k" H 7250 3750 60  0001 C CNN "Part Number"
 	1    7250 3750
 	1    0    0    -1
@@
 F 2 "Capacitor_SMD:C_0603_1608Metric" H 8338 3650 50  0001 C CNN
 F 3 "" H 8300 3800 50  0001 C CNN
-F 4 "CL10A475KQ8NNNC" H 8300 3800 60  0001 C CNN "Part Number"
+F 4 "GPC0603475" H 8300 3800 60  0001 C CNN "Part Number"
 	1    8300 3800
 	1    0    0    -1
@@
 F 2 "Capacitor_SMD:C_0603_1608Metric" H 8888 3650 50  0001 C CNN
 F 3 "" H 8850 3800 50  0001 C CNN
-F 4 "CC0603KRX7R8BB104" H 8850 3800 60  0001 C CNN "Part Number"
+F 4 "GPC0603104" H 8850 3800 60  0001 C CNN "Part Number"
 	1    8850 3800
 	1    0    0    -1
