File: ecad/common/Fan_controller.kicad_sch (KiCad schematic)
At the start: 10 parts, among them U6 EMC2302-1-AIZL-TR

Commit message: fixup! Updates Celaeno for production
Parts:
- D1, D7: MPN (none) -> CPDT-5V0USP-HF
- R16, R17: MPN (none) -> GPR060347K
- R18, R19, R20, R21: MPN (none) -> GPR06032K2
- U6: MPN (none) -> EMC2302-1-AIZL-TR
Changed lines of the file:
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@@
 			)
 		)
-		(property "MPN" ""
+		(property "MPN" "EMC2302-1-AIZL-TR"
 			(at 102.87 87.63 0)
 			(effects
@@
 			)
 		)
-		(property "MPN" ""
+		(property "MPN" "GPR060347K"
 			(at 143.51 76.2 0)
 			(effects
@@
 			)
 		)
-		(property "MPN" ""
+		(property "MPN" "GPR060347K"
 			(at 151.13 76.2 0)
 			(effects
@@
 			)
 		)
-		(property "MPN" ""
+		(property "MPN" "GPR06032K2"
 			(at 166.37 80.01 0)
 			(effects
@@
 			)
 		)
-		(property "MPN" ""
+		(property "MPN" "CPDT-5V0USP-HF"
 			(at 180.34 109.22 0)
 			(effects
@@
 			)
 		)
-		(property "MPN" ""
+		(property "MPN" "CPDT-5V0USP-HF"
 			(at 204.47 109.22 0)
 			(effects
@@
 			)
 		)
-		(property "MPN" ""
+		(property "MPN" "GPR06032K2"
 			(at 166.37 85.09 0)
 			(effects
@@
 			)
 		)
-		(property "MPN" ""
+		(property "MPN" "GPR06032K2"
 			(at 166.37 90.17 0)
 			(effects
@@
 			)
 		)
-		(property "MPN" ""
+		(property "MPN" "GPR06032K2"
 			(at 166.37 95.25 0)
 			(effects
