File: ecad/climate/zeus/12V_low_side_switch.sch (KiCad schematic (older format))
At the start: 3 parts, among them Q1 PMV45EN

Commit message: Small Correction for Production
Parts:
- D1: value MCL4148 -> 1N4148WS; footprint Diode_SMD:D_MicroMELF -> Diode_SMD:D_SOD-323F; Part Number MCL4148-TR -> 1N4148WS
Changed lines of the file:
@@
 AR Path="/5BBA23F4/5BBA266C" Ref="Q1"  Part="1"
 AR Path="/5BB2B93A/5BBA266C" Ref="Q2"  Part="1"
-F 0 "Q2" H 5800 4300 50  0000 L CNN
+F 0 "Q1" H 5800 4300 50  0000 L CNN
 F 1 "PMV45EN" H 5800 4200 50  0000 L CNN
 F 2 "Package_TO_SOT_SMD:SOT-23" H 5800 4350 50  0001 C CNN
@@
 AR Path="/5BBA23F4/5BBA2674" Ref="D1"  Part="1"
 AR Path="/5BB2B93A/5BBA2674" Ref="D2"  Part="1"
-F 0 "D2" H 6500 3750 50  0000 C CNN
-F 1 "MCL4148" H 6500 3550 50  0000 C CNN
-F 2 "Diode_SMD:D_MicroMELF" H 6500 3650 50  0001 C CNN
+F 0 "D1" H 6500 3750 50  0000 C CNN
+F 1 "1N4148WS" H 6500 3550 50  0000 C CNN
+F 2 "Diode_SMD:D_SOD-323F" H 6500 3650 50  0001 C CNN
 F 3 "" H 6500 3650 50  0001 C CNN
-F 4 "MCL4148-TR" H 6500 3650 60  0001 C CNN "Part Number"
+F 4 "1N4148WS" H 6500 3650 60  0001 C CNN "Part Number"
 	1    6500 3650
 	0    1    1    0
@@
 AR Path="/5BBA23F4/5BBA267B" Ref="#PWR0109"  Part="1"
 AR Path="/5BB2B93A/5BBA267B" Ref="#PWR0111"  Part="1"
-F 0 "#PWR0111" H 6500 2850 50  0001 C CNN
+F 0 "#PWR0109" H 6500 2850 50  0001 C CNN
 F 1 "+12V" H 6500 3140 50  0000 C CNN
 F 2 "" H 6500 3000 50  0001 C CNN
@@
 AR Path="/5BBA23F4/5BBA2691" Ref="#PWR0110"  Part="1"
 AR Path="/5BB2B93A/5BBA2691" Ref="#PWR0112"  Part="1"
-F 0 "#PWR0112" H 5700 4500 50  0001 C CNN
+F 0 "#PWR0110" H 5700 4500 50  0001 C CNN
 F 1 "GND" H 5700 4600 50  0000 C CNN
 F 2 "" H 5700 4750 50  0001 C CNN
@@
 AR Path="/5BBA23F4/5BBA6C7D" Ref="R20"  Part="1"
 AR Path="/5BB2B93A/5BBA6C7D" Ref="R21"  Part="1"
-F 0 "R21" V 5330 4500 50  0000 C CNN
+F 0 "R20" V 5330 4500 50  0000 C CNN
 F 1 "47k5" V 5250 4500 50  0000 C CNN
 F 2 "Resistor_SMD:R_0603_1608Metric" V 5180 4500 50  0001 C CNN

Commit message: Licenses Climate PCB under OHL v1.2
Other:
- note added: "© 2018 Université de Lausanne\n\nThis documentation describes Open Hardware and is licensed under the\nCERN OHL v. 1.2.\n\nYou may redistribute and modify this documentation under the terms of\nthe CERN OHL v.1.2. (http://ohwr.org/cernohl). This documentation is\ndistributed WITHOUT ANY EXPRESS OR IMPLIED WARRANTY,\nINCLUDING OF MERCHANTABILITY, SATISFACTORY QUALITY AND\nFITNESS FOR A PARTICULAR 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"
Changed lines of the file:
@@
 encoding utf-8
 Sheet 9 10
-Title ""
-Date ""
-Rev ""
-Comp ""
-Comment1 ""
-Comment2 ""
+Title "12V Low Side Sitch w/ free-whiling diode"
+Date "06/11/2018"
+Rev "A"
+Comp "Université de Lausanne"
+Comment1 "Author: Alexandre Tuleu"
+Comment2 "Licensed under the CERN OHL v1.2"
 Comment3 ""
 Comment4 ""
@@
 Wire Wire Line
 	6500 4000 7200 4000
+Text Notes 550  7750 0    50   ~ 0
+© 2018 Université de Lausanne\n\nThis documentation describes Open Hardware and is licensed under the\nCERN OHL v. 1.2.\n\nYou may redistribute and modify this documentation under the terms of\nthe CERN OHL v.1.2. (http://ohwr.org/cernohl). This documentation is\ndistributed WITHOUT ANY EXPRESS OR IMPLIED WARRANTY,\nINCLUDING OF MERCHANTABILITY, SATISFACTORY QUALITY AND\nFITNESS FOR A PARTICULAR PURPOSE. Please see the CERN OHL v.1.2\nfor applicable conditions
 $EndSCHEMATC

Commit message: Updates board for manufacturing
Parts:
- R20: value 47k5 -> 47k; Part Number GPR060347k5 -> GPR060347K
Changed lines of the file:
@@
 AR Path="/5BB2B93A/5BBA6C7D" Ref="R21"  Part="1"
 F 0 "R20" V 5330 4500 50  0000 C CNN
-F 1 "47k5" V 5250 4500 50  0000 C CNN
+F 1 "47k" V 5250 4500 50  0000 C CNN
 F 2 "Resistor_SMD:R_0603_1608Metric" V 5180 4500 50  0001 C CNN
 F 3 "" H 5250 4500 50  0001 C CNN
-F 4 "GPR060347k5" H 5250 4500 60  0001 C CNN "Part Number"
+F 4 "GPR060347K" H 5250 4500 60  0001 C CNN "Part Number"
 	1    5250 4500
 	-1   0    0    1
