File: ecad/climate/zeus/UC.sch (KiCad schematic (older format))
At the start: 18 parts, among them J14 68000-212HLF, J15 68000-212HLF, J4 M20-8760342, SW1 1825910-6, U2 AT90CAN128-16AU, Y1 16MHz

Commit message: Makes pleiades zeus again
Parts:
- removed J14, J15: 68000-212HLF, Connector_PinHeader_2.54mm:PinHeader_1x12_P2.54mm_Vertical, symbol Connector_Generic:Conn_01x12
Connections:
- net labels removed: +12V, +3V3, RELAY_1, RELAY_2
- wire segments 115 -> 81
- no-connect marks 24 -> 42
Changed lines of the file:
@@
 EESchema Schematic File Version 4
-LIBS:pleiades-cache
+LIBS:zeus-cache
 EELAYER 26 0
 EELAYER END
 $Descr A4 11693 8268
 encoding utf-8
-Sheet 6 12
+Sheet 6 10
 Title ""
 Date ""
@@
 	5800 6450 5800 6400
 $Comp
-L Connector_Generic:Conn_01x12 J14
-U 1 1 5BB5BBE4
-P 10450 2450
-F 0 "J14" H 10530 2442 50  0000 L CNN
-F 1 "68000-212HLF" H 10530 2351 50  0000 L CNN
-F 2 "Connector_PinHeader_2.54mm:PinHeader_1x12_P2.54mm_Vertical" H 10450 2450 50  0001 C CNN
-F 3 "~" H 10450 2450 50  0001 C CNN
-F 4 "68000-212HLF" H 10450 2450 50  0001 C CNN "Part Number"
-	1    10450 2450
-	1    0    0    -1
-$EndComp
-$Comp
 L MCU_Microchip_AVR:AT90CAN128-16AU U2
 U 1 1 5BA92DFF
 P 5800 3950
 F 0 "U2" H 5300 5900 50  0000 L BNN
-F 1 "AT90CAN128-16AU" H 6950 2000 50  0000 R BNN
+F 1 "AT90CAN128-16AU" H 5600 1950 50  0000 R BNN
 F 2 "Package_QFP:TQFP-64_14x14mm_P0.8mm" H 5850 3950 50  0001 C CNN
 F 3 "" H 5800 3950 50  0001 C CNN
@@
 Wire Wire Line
 	6400 3250 7700 3250
-$Comp
-L Connector_Generic:Conn_01x12 J15
-U 1 1 5BB63291
-P 10450 4250
-F 0 "J15" H 10530 4242 50  0000 L CNN
-F 1 "68000-212HLF" H 10530 4151 50  0000 L CNN
-F 2 "Connector_PinHeader_2.54mm:PinHeader_1x12_P2.54mm_Vertical" H 10450 4250 50  0001 C CNN
-F 3 "~" H 10450 4250 50  0001 C CNN
-F 4 "68000-212HLF" H 10450 4250 50  0001 C CNN "Part Number"
-	1    10450 4250
-	1    0    0    -1
-$EndComp
-Wire Wire Line
-	6400 2250 10250 2250
-Wire Wire Line
-	6400 2350 10250 2350
-Wire Wire Line
-	6400 2450 10250 2450
-Wire Wire Line
-	6400 2550 10250 2550
-Wire Wire Line
-	6400 2650 10250 2650
-Wire Wire Line
-	6400 2750 10250 2750
-Wire Wire Line
-	6400 2850 10250 2850
-Wire Wire Line
-	6400 2950 10250 2950
-Wire Wire Line
-	6400 4050 10250 4050
-Wire Wire Line
-	6400 4150 10250 4150
-Wire Wire Line
-	6400 4250 10250 4250
-Wire Wire Line
-	6400 4350 10250 4350
-Wire Wire Line
-	6400 4450 10250 4450
-Wire Wire Line
-	6400 4550 10250 4550
-Wire Wire Line
-	6400 4650 10250 4650
-Wire Wire Line
-	6400 4750 10250 4750
-$Comp
-L power:GND #PWR0101
-U 1 1 5BB6711B
-P 10100 3150
-F 0 "#PWR0101" H 10100 2900 50  0001 C CNN
-F 1 "GND" H 10105 2977 50  0000 C CNN
-F 2 "" H 10100 3150 50  0001 C CNN
-F 3 "" H 10100 3150 50  0001 C CNN
-	1    10100 3150
-	1    0    0    -1
-$EndComp
-Wire Wire Line
-	10100 3050 10250 3050
-$Comp
-L power:GND #PWR0102
-U 1 1 5BB69978
-P 10100 5000
-F 0 "#PWR0102" H 10100 4750 50  0001 C CNN
-F 1 "GND" H 10105 4827 50  0000 C CNN
-F 2 "" H 10100 5000 50  0001 C CNN
-F 3 "" H 10100 5000 50  0001 C CNN
-	1    10100 5000
-	1    0    0    -1
-$EndComp
-Wire Wire Line
-	10100 5000 10100 4850
-Wire Wire Line
-	10100 4850 10250 4850
-$Comp
-L power:+12V #PWR0103
-U 1 1 5BB6C373
-P 10100 1800
-F 0 "#PWR0103" H 10100 1650 50  0001 C CNN
-F 1 "+12V" H 10115 1973 50  0000 C CNN
-F 2 "" H 10100 1800 50  0001 C CNN
-F 3 "" H 10100 1800 50  0001 C CNN
-	1    10100 1800
-	1    0    0    -1
-$EndComp
-Wire Wire Line
-	10100 1800 10100 1950
-Wire Wire Line
-	10100 1950 10250 1950
-$Comp
-L power:+5V #PWR0104
-U 1 1 5BB6EEB4
-P 9900 1800
-F 0 "#PWR0104" H 9900 1650 50  0001 C CNN
-F 1 "+5V" H 9915 1973 50  0000 C CNN
-F 2 "" H 9900 1800 50  0001 C CNN
-F 3 "" H 9900 1800 50  0001 C CNN
-	1    9900 1800
-	1    0    0    -1
-$EndComp
-$Comp
-L power:+3V3 #PWR0105
-U 1 1 5BB71A1D
-P 9650 1800
-F 0 "#PWR0105" H 9650 1650 50  0001 C CNN
-F 1 "+3V3" H 9665 1973 50  0000 C CNN
-F 2 "" H 9650 1800 50  0001 C CNN
-F 3 "" H 9650 1800 50  0001 C CNN
-	1    9650 1800
-	1    0    0    -1
-$EndComp
-Wire Wire Line
-	9650 1800 9650 2150
-Wire Wire Line
-	9650 2150 10250 2150
-Wire Wire Line
-	10250 2050 9900 2050
-Wire Wire Line
-	9900 2050 9900 1800
-$Comp
-L power:+12V #PWR0106
-U 1 1 5BB77434
-P 10100 3600
-F 0 "#PWR0106" H 10100 3450 50  0001 C CNN
-F 1 "+12V" H 10115 3773 50  0000 C CNN
-F 2 "" H 10100 3600 50  0001 C CNN
-F 3 "" H 10100 3600 50  0001 C CNN
-	1    10100 3600
-	1    0    0    -1
-$EndComp
-Wire Wire Line
-	10100 3600 10100 3750
-Wire Wire Line
-	10100 3750 10250 3750
-$Comp
-L power:+5V #PWR0107
-U 1 1 5BB7743C
-P 9900 3600
-F 0 "#PWR0107" H 9900 3450 50  0001 C CNN
-F 1 "+5V" H 9915 3773 50  0000 C CNN
-F 2 "" H 9900 3600 50  0001 C CNN
-F 3 "" H 9900 3600 50  0001 C CNN
-	1    9900 3600
-	1    0    0    -1
-$EndComp
-$Comp
-L power:+3V3 #PWR0108
-U 1 1 5BB77442
-P 9650 3600
-F 0 "#PWR0108" H 9650 3450 50  0001 C CNN
-F 1 "+3V3" H 9665 3773 50  0000 C CNN
-F 2 "" H 9650 3600 50  0001 C CNN
-F 3 "" H 9650 3600 50  0001 C CNN
-	1    9650 3600
-	1    0    0    -1
-$EndComp
-Wire Wire Line
-	9650 3600 9650 3950
-Wire Wire Line
-	9650 3950 10250 3950
-Wire Wire Line
-	10250 3850 9900 3850
-Wire Wire Line
-	9900 3850 9900 3600
-Wire Wire Line
-	10100 3150 10100 3050
-Text HLabel 4600 4650 0    50   Output ~ 0
-RELAY_1
-Text HLabel 4600 4750 0    50   Output ~ 0
-RELAY_2
-Wire Wire Line
-	4600 4650 5200 4650
-Wire Wire Line
-	4600 4750 5200 4750
+NoConn ~ 5200 4650
+NoConn ~ 5200 4750
+NoConn ~ 6400 2250
+NoConn ~ 6400 2350
+NoConn ~ 6400 2450
+NoConn ~ 6400 2550
+NoConn ~ 6400 2650
+NoConn ~ 6400 2750
+NoConn ~ 6400 2850
+NoConn ~ 6400 2950
+NoConn ~ 6400 4050
+NoConn ~ 6400 4150
+NoConn ~ 6400 4250
+NoConn ~ 6400 4350
+NoConn ~ 6400 4450
+NoConn ~ 6400 4550
+NoConn ~ 6400 4650
+NoConn ~ 6400 4750
 $EndSCHEMATC

Commit message: Licenses Climate PCB under OHL v1.2
Other:
- note added: "© 2018 Université de Lausanne\n\nThis documentation describes Open Hardware and is licensed under the\nCERN OHL v. 1.2.\n\nYou may redistribute and modify this documentation under the terms of\nthe CERN OHL v.1.2. (http://ohwr.org/cernohl). This documentation is\ndistributed WITHOUT ANY EXPRESS OR IMPLIED WARRANTY,\nINCLUDING OF MERCHANTABILITY, SATISFACTORY QUALITY AND\nFITNESS FOR A PARTICULAR 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"
Changed lines of the file:
@@
 encoding utf-8
 Sheet 6 10
-Title ""
-Date ""
-Rev ""
-Comp ""
-Comment1 ""
-Comment2 ""
+Title "AT90CAN128 - Climate Controller"
+Date "06/11/2018"
+Rev "A"
+Comp "Université de Lausanne"
+Comment1 "Author: Alexandre Tuleu"
+Comment2 "Licensed under the CERN OHL v1.2"
 Comment3 ""
 Comment4 ""
@@
 NoConn ~ 6400 4650
 NoConn ~ 6400 4750
+Text Notes 550  7750 0    50   ~ 0
+© 2018 Université de Lausanne\n\nThis documentation describes Open Hardware and is licensed under the\nCERN OHL v. 1.2.\n\nYou may redistribute and modify this documentation under the terms of\nthe CERN OHL v.1.2. (http://ohwr.org/cernohl). This documentation is\ndistributed WITHOUT ANY EXPRESS OR IMPLIED WARRANTY,\nINCLUDING OF MERCHANTABILITY, SATISFACTORY QUALITY AND\nFITNESS FOR A PARTICULAR PURPOSE. Please see the CERN OHL v.1.2\nfor applicable conditions
 $EndSCHEMATC

Commit message: Makes all electronics production ready
Parts:
- C10, C11: Part Number C0603C180K5GACTU -> GPC0603180
- C7, C8, C9: Part Number CC0603KRX7R8BB104 -> GPC0603104
- R5: Part Number RMCF0603FT100K -> GPR0603100K
Changed lines of the file:
@@
 F 2 "Capacitor_SMD:C_0603_1608Metric" H 5188 1350 50  0001 C CNN
 F 3 "" H 5150 1500 50  0001 C CNN
-F 4 "CC0603KRX7R8BB104" H 5150 1500 60  0001 C CNN "Part Number"
+F 4 "GPC0603104" H 5150 1500 60  0001 C CNN "Part Number"
 	1    5150 1500
 	1    0    0    -1
@@
 F 2 "Capacitor_SMD:C_0603_1608Metric" H 5588 1350 50  0001 C CNN
 F 3 "" H 5550 1500 50  0001 C CNN
-F 4 "CC0603KRX7R8BB104" H 5550 1500 60  0001 C CNN "Part Number"
+F 4 "GPC0603104" H 5550 1500 60  0001 C CNN "Part Number"
 	1    5550 1500
 	1    0    0    -1
@@
 F 2 "Capacitor_SMD:C_0603_1608Metric" H 6238 1350 50  0001 C CNN
 F 3 "" H 6200 1500 50  0001 C CNN
-F 4 "CC0603KRX7R8BB104" H 6200 1500 60  0001 C CNN "Part Number"
+F 4 "GPC0603104" H 6200 1500 60  0001 C CNN "Part Number"
 	1    6200 1500
 	1    0    0    -1
@@
 F 2 "Capacitor_SMD:C_0603_1608Metric" H 3138 2050 50  0001 C CNN
 F 3 "" H 3100 2200 50  0001 C CNN
-F 4 "C0603C180K5GACTU" H 3100 2200 60  0001 C CNN "Part Number"
+F 4 "GPC0603180" H 3100 2200 60  0001 C CNN "Part Number"
 	1    3100 2200
 	0    -1   1    0
@@
 F 2 "Capacitor_SMD:C_0603_1608Metric" H 3138 2850 50  0001 C CNN
 F 3 "" H 3100 3000 50  0001 C CNN
-F 4 "C0603C180K5GACTU" H 3100 3000 60  0001 C CNN "Part Number"
+F 4 "GPC0603180" H 3100 3000 60  0001 C CNN "Part Number"
 	1    3100 3000
 	0    -1   1    0
@@
 F 2 "Resistor_SMD:R_0603_1608Metric" V 2780 1700 50  0001 C CNN
 F 3 "" H 2850 1700 50  0001 C CNN
-F 4 "RMCF0603FT100K" H 2850 1700 60  0001 C CNN "Part Number"
+F 4 "GPR0603100K" H 2850 1700 60  0001 C CNN "Part Number"
 	1    2850 1700
 	1    0    0    -1

Commit message: Updates ecad for assembly production
Parts:
- U2: value AT90CAN128-16AU -> AT90CAN32-16AU; Part Number AT90CAN128-16AU -> AT90CAN32-16AU
Changed lines of the file:
@@
 P 5800 3950
 F 0 "U2" H 5300 5900 50  0000 L BNN
-F 1 "AT90CAN128-16AU" H 5600 1950 50  0000 R BNN
+F 1 "AT90CAN32-16AU" H 5600 1950 50  0000 R BNN
 F 2 "Package_QFP:TQFP-64_14x14mm_P0.8mm" H 5850 3950 50  0001 C CNN
 F 3 "" H 5800 3950 50  0001 C CNN
-F 4 "AT90CAN128-16AU" H 5800 3950 60  0001 C CNN "Part Number"
+F 4 "AT90CAN32-16AU" H 5800 3950 60  0001 C CNN "Part Number"
 	1    5800 3950
 	1    0    0    -1

Commit message: Updates kicad data.
Parts:
- U2: symbol MCU_Microchip_AVR:AT90CAN128-16AU -> zeus-rescue:AT90CAN128-16AU-MCU_Microchip_AVR
Changed lines of the file:
@@
 	5800 6450 5800 6400
 $Comp
-L MCU_Microchip_AVR:AT90CAN128-16AU U2
+L zeus-rescue:AT90CAN128-16AU-MCU_Microchip_AVR U2
 U 1 1 5BA92DFF
 P 5800 3950
+AR Path="/5BA92DFF" Ref="U2"  Part="1"
+AR Path="/5BA4D58C/5BA92DFF" Ref="U2"  Part="1"
 F 0 "U2" H 5300 5900 50  0000 L BNN
 F 1 "AT90CAN32-16AU" H 5600 1950 50  0000 R BNN
