File: ecad/climate/zeus/zeus.sch (KiCad schematic (older format))
At the start: 11 parts, among them J1 MCV 1,5/ 2-G-3,5, J10 47053-1000, J11 47053-1000, J2 MCV 1,5/ 2-G-3,5, J3 5566-02A, J5 47053-1000, J6 47053-1000, J7 215079-8, J8 640454-2, J9 640454-2

Commit message: Updates ecad for assembly production
Parts:
- J8, J9: value 640454-2 -> 6410-02A; footprint FORT:640454-2 -> Connector_Molex:Molex_KK-254_AE-6410-02A_1x02_P2.54mm_Vertical; Part Number 640454-2 -> 22-27-2021
Connections:
- net 12V Low Side 1/12V_SW+: now also J8.2 (Pin_2); no longer J8.1 (Pin_1)
- net 12V Low Side 1/12V_SW-: now also J8.1 (Pin_1); no longer J8.2 (Pin_2)
- net 12V Low Side 2/12V_SW+: now also J9.2 (Pin_2); no longer J9.1 (Pin_1)
- net 12V Low Side 2/12V_SW-: now also J9.1 (Pin_1); no longer J9.2 (Pin_2)
Other:
- moved on the sheet: J1, J2
Changed lines of the file:
@@
 $EndComp
 $Sheet
-S 1550 3950 1850 350
+S 1900 3950 1850 350
 U 5BA4C5E7
 F0 "CAN Transceiver" 60
 F1 "../../common/CAN_transceiver.sch" 60
-F2 "CAN+" B L 1550 4050 60
-F3 "CAN-" B L 1550 4150 60
-F4 "TXD" I R 3400 4050 60
-F5 "RXD" O R 3400 4150 60
+F2 "CAN+" B L 1900 4050 60
+F3 "CAN-" B L 1900 4150 60
+F4 "TXD" I R 3750 4050 60
+F5 "RXD" O R 3750 4150 60
 $EndSheet
 $Sheet
@@
 L Connector_Generic:Conn_01x02 J8
 U 1 1 5BA51183
-P 10550 1200
-F 0 "J8" H 10550 1300 50  0000 C CNN
-F 1 "640454-2" H 10550 1000 50  0000 C CNN
-F 2 "FORT:640454-2" H 10550 1200 50  0001 C CNN
-F 3 "" H 10550 1200 50  0001 C CNN
-F 4 "640454-2" H 10550 1200 60  0001 C CNN "Part Number"
-	1    10550 1200
-	1    0    0    -1
-$EndComp
-$Comp
-L Connector_Generic:Conn_01x02 J9
-U 1 1 5BA51439
-P 10550 1650
-F 0 "J9" H 10550 1750 50  0000 C CNN
-F 1 "640454-2" H 10550 1450 50  0000 C CNN
-F 2 "FORT:640454-2" H 10550 1650 50  0001 C CNN
-F 3 "" H 10550 1650 50  0001 C CNN
-F 4 "640454-2" H 10550 1650 60  0001 C CNN "Part Number"
-	1    10550 1650
-	1    0    0    -1
+P 10550 1300
+F 0 "J8" H 10550 1400 50  0000 C CNN
+F 1 "6410-02A" H 10550 1100 50  0000 C CNN
+F 2 "Connector_Molex:Molex_KK-254_AE-6410-02A_1x02_P2.54mm_Vertical" H 10550 1300 50  0001 C CNN
+F 3 "" H 10550 1300 50  0001 C CNN
+F 4 "22-27-2021" H 10550 1300 60  0001 C CNN "Part Number"
+	1    10550 1300
+	1    0    0    1
 $EndComp
 Text Notes 11150 1650 1    60   ~ 0
@@
 L Connector_Generic:Conn_01x02 J2
 U 1 1 5BA55E48
-P 700 4500
-F 0 "J2" H 700 4600 50  0000 C CNN
-F 1 "MCV 1,5/ 2-G-3,5" H 700 4300 50  0000 C CNN
-F 2 "Connector_Phoenix_MC:PhoenixContact_MCV_1,5_2-G-3.5_1x02_P3.50mm_Vertical" H 700 4500 50  0001 C CNN
-F 3 "" H 700 4500 50  0001 C CNN
-F 4 "MCV 1,5/ 2-G-3,5" H 700 4500 60  0001 C CNN "Part Number"
-	1    700  4500
+P 1050 4500
+F 0 "J2" H 1050 4600 50  0000 C CNN
+F 1 "MCV 1,5/ 2-G-3,5" H 1050 4300 50  0000 C CNN
+F 2 "Connector_Phoenix_MC:PhoenixContact_MCV_1,5_2-G-3.5_1x02_P3.50mm_Vertical" H 1050 4500 50  0001 C CNN
+F 3 "" H 1050 4500 50  0001 C CNN
+F 4 "MCV 1,5/ 2-G-3,5" H 1050 4500 60  0001 C CNN "Part Number"
+	1    1050 4500
 	-1   0    0    -1
 $EndComp
@@
 L Connector_Generic:Conn_01x02 J1
 U 1 1 5BA560A5
-P 700 4050
-F 0 "J1" H 700 4150 50  0000 C CNN
-F 1 "MCV 1,5/ 2-G-3,5" H 700 3850 50  0000 C CNN
-F 2 "Connector_Phoenix_MC:PhoenixContact_MCV_1,5_2-G-3.5_1x02_P3.50mm_Vertical" H 700 4050 50  0001 C CNN
-F 3 "" H 700 4050 50  0001 C CNN
-F 4 "MCV 1,5/ 2-G-3,5" H 700 4050 60  0001 C CNN "Part Number"
-	1    700  4050
+P 1050 4050
+F 0 "J1" H 1050 4150 50  0000 C CNN
+F 1 "MCV 1,5/ 2-G-3,5" H 1050 3850 50  0000 C CNN
+F 2 "Connector_Phoenix_MC:PhoenixContact_MCV_1,5_2-G-3.5_1x02_P3.50mm_Vertical" H 1050 4050 50  0001 C CNN
+F 3 "" H 1050 4050 50  0001 C CNN
+F 4 "MCV 1,5/ 2-G-3,5" H 1050 4050 60  0001 C CNN "Part Number"
+	1    1050 4050
 	-1   0    0    -1
 $EndComp
@@
 3V3\nSDA\nSCL\nGND
 $Sheet
-S 3600 3150 1250 1600
+S 3950 3150 1250 1600
 U 5BA4D58C
 F0 "UC" 60
 F1 "UC.sch" 60
-F2 "CAN_TX" O L 3600 4050 60
-F3 "CAN_RX" I L 3600 4150 60
-F4 "~FAN_ALERT" I R 4850 4100 60
-F5 "HEAT1" O R 4850 3800 60
-F6 "HEAT2" O R 4850 3900 60
-F7 "SDA_5V" B R 4850 4200 60
-F8 "SCL_5V" O R 4850 4300 60
+F2 "CAN_TX" O L 3950 4050 60
+F3 "CAN_RX" I L 3950 4150 60
+F4 "~FAN_ALERT" I R 5200 4100 60
+F5 "HEAT1" O R 5200 3800 60
+F6 "HEAT2" O R 5200 3900 60
+F7 "SDA_5V" B R 5200 4200 60
+F8 "SCL_5V" O R 5200 4300 60
 $EndSheet
 $Comp
@@
 	9800 4800 10400 4800
 Wire Wire Line
-	900  4050 1200 4050
-Wire Wire Line
-	900  4150 1300 4150
-Wire Wire Line
-	1200 4050 1200 4500
-Wire Wire Line
-	1200 4500 900  4500
-Connection ~ 1200 4050
-Wire Wire Line
-	1300 4150 1300 4600
-Wire Wire Line
-	1300 4600 900  4600
-Connection ~ 1300 4150
+	1250 4050 1550 4050
+Wire Wire Line
+	1250 4150 1650 4150
+Wire Wire Line
+	1550 4050 1550 4500
+Wire Wire Line
+	1550 4500 1250 4500
+Connection ~ 1550 4050
+Wire Wire Line
+	1650 4150 1650 4600
+Wire Wire Line
+	1650 4600 1250 4600
+Connection ~ 1650 4150
 Connection ~ 2200 1500
 Wire Wire Line
@@
 	2000 1600 2000 1800
 Wire Wire Line
-	3400 4050 3600 4050
-Wire Wire Line
-	3400 4150 3600 4150
+	3750 4050 3950 4050
+Wire Wire Line
+	3750 4150 3950 4150
 Wire Wire Line
 	10200 3050 10400 3050
@@
 	10200 3500 10200 3350
 Wire Wire Line
-	4850 4200 6100 4200
-Wire Wire Line
-	4850 4300 6100 4300
-Wire Wire Line
 	8050 4250 8500 4250
 Wire Wire Line
@@
 	10200 4100 10200 4700
 Wire Wire Line
-	1200 4050 1550 4050
-Wire Wire Line
-	1300 4150 1550 4150
+	1550 4050 1900 4050
+Wire Wire Line
+	1650 4150 1900 4150
 Wire Wire Line
 	2200 1500 2350 1500
@@
 	10250 1300 10350 1300
 Wire Wire Line
-	4850 4100 6100 4100
-Wire Wire Line
-	4850 3900 5900 3900
+	5200 3900 5900 3900
 Wire Wire Line
 	5900 3900 5900 2850
@@
 	9000 1700 9100 1700
 Wire Wire Line
-	4850 3800 5800 3800
+	5200 3800 5800 3800
 Wire Wire Line
 	5800 3800 5800 2750
@@
 Wire Wire Line
 	9450 3750 9450 3650
+Wire Wire Line
+	5200 4100 6100 4100
+Wire Wire Line
+	5200 4200 6100 4200
+Wire Wire Line
+	5200 4300 6100 4300
+$Comp
+L Connector_Generic:Conn_01x02 J9
+U 1 1 5C7D38B0
+P 10550 1750
+F 0 "J9" H 10550 1850 50  0000 C CNN
+F 1 "6410-02A" H 10550 1550 50  0000 C CNN
+F 2 "Connector_Molex:Molex_KK-254_AE-6410-02A_1x02_P2.54mm_Vertical" H 10550 1750 50  0001 C CNN
+F 3 "" H 10550 1750 50  0001 C CNN
+F 4 "22-27-2021" H 10550 1750 60  0001 C CNN "Part Number"
+	1    10550 1750
+	1    0    0    1
+$EndComp
 $EndSCHEMATC

Commit message: Updates kicad data.
Parts:
- J7: value 215079-8 -> 215079-4
Changed lines of the file:
@@
 P 10600 3150
 F 0 "J7" H 10600 3350 50  0000 C CNN
-F 1 "215079-8" H 10600 2850 50  0000 C CNN
+F 1 "215079-4" H 10600 2850 50  0000 C CNN
 F 2 "FORT:Micro-Match_4_TH" H 10600 3150 50  0001 C CNN
 F 3 "" H 10600 3150 50  0001 C CNN
