File: ecad/climate/prometheus/prometheus.sch (KiCad schematic (older format))
At the start: 11 parts, among them J1 2.5mm I.D. 5.5mm O.D., J2 5566-02A, J3 5566-02A, J4 5566-02A, J5 5566-02A

Commit message: Updates board for manufacturing
Parts:
- added J6: 5566-02A, Connector_Molex:Molex_Mini-Fit_Jr_5566-02A_2x01_P4.20mm_Vertical, symbol Connector_Generic:Conn_01x02
Connections:
- wire segments 23 -> 27
Changed lines of the file:
@@
 Connection ~ 6200 3650
 Wire Wire Line
-	6200 3900 6200 4150
-Wire Wire Line
-	6200 4150 6400 4150
-Connection ~ 6200 3900
+	6200 4400 6400 4400
 $Comp
 L power:GND #PWR06
 U 1 1 5C00493A
-P 6300 4550
-F 0 "#PWR06" H 6300 4300 50  0001 C CNN
-F 1 "GND" H 6305 4377 50  0000 C CNN
-F 2 "" H 6300 4550 50  0001 C CNN
-F 3 "" H 6300 4550 50  0001 C CNN
-	1    6300 4550
+P 6300 4800
+F 0 "#PWR06" H 6300 4550 50  0001 C CNN
+F 1 "GND" H 6305 4627 50  0000 C CNN
+F 2 "" H 6300 4800 50  0001 C CNN
+F 3 "" H 6300 4800 50  0001 C CNN
+	1    6300 4800
 	1    0    0    -1
 $EndComp
 Wire Wire Line
-	6300 4550 6300 4250
+	6300 4800 6300 4500
 Wire Wire Line
-	6300 4250 6400 4250
+	6300 4500 6400 4500
 Wire Wire Line
-	6300 4250 6300 4000
+	6300 4500 6300 4250
 Wire Wire Line
 	6300 4000 6400 4000
-Connection ~ 6300 4250
+Connection ~ 6300 4500
 Wire Wire Line
 	6300 4000 6300 3750
 Wire Wire Line
 	6300 3750 6400 3750
-Connection ~ 6300 4000
 Wire Wire Line
 	6300 3750 6300 3500
@@
 	1    0    0    -1
 $EndComp
+$Comp
+L Connector_Generic:Conn_01x02 J6
+U 1 1 5C019117
+P 6600 4400
+F 0 "J6" H 6680 4392 50  0000 L CNN
+F 1 "5566-02A" H 6680 4301 50  0000 L CNN
+F 2 "Connector_Molex:Molex_Mini-Fit_Jr_5566-02A_2x01_P4.20mm_Vertical" H 6600 4400 50  0001 C CNN
+F 3 "~" H 6600 4400 50  0001 C CNN
+F 4 "39-28-1023" H 6600 4400 50  0001 C CNN "Part Number"
+	1    6600 4400
+	1    0    0    -1
+$EndComp
+Wire Wire Line
+	6300 4250 6400 4250
+Wire Wire Line
+	6300 4250 6300 4000
+Connection ~ 6300 4250
+Connection ~ 6300 4000
+Wire Wire Line
+	6200 3900 6200 4150
+Connection ~ 6200 3900
+Wire Wire Line
+	6200 4150 6400 4150
+Connection ~ 6200 4150
+Wire Wire Line
+	6200 4150 6200 4400
 $EndSCHEMATC
