File: ecad/climate/prometheus/prometheus.kicad_pcb (KiCad board)
At the start: 2 copper layers, 34 x 44 mm, 13 parts, among them J1 2.5mm I.D. 5.5mm O.D., J2 5566-02A, J3 5566-02A, J4 5566-02A, J5 5566-02A

Commit message: Updates board for manufacturing
Parts:
- added J6: 5566-02A, Connector_Molex:Molex_Mini-Fit_Jr_5566-02A_2x01_P4.20mm_Vertical, F.Cu at (127.0, 116.0)
- moved G*** 4.12 mm to (118.0, 77.5)
- moved REF** 4.12 mm to (118.0, 84.0)
- moved J2 4.00 mm to (127.0, 84.0)
- moved J3 4.00 mm to (127.0, 92.0)
- moved J4 4.00 mm to (127.0, 100.0)
- moved J5 4.00 mm to (127.0, 108.0)
- moved MH1 4.00 mm to (106.0, 77.0)
- moved MH2 4.00 mm to (106.0, 123.0)
- moved MH3 4.00 mm to (134.0, 77.0)
- moved MH4 4.00 mm to (134.0, 123.0)
Routing:
- net GND: track 73.5 -> 88.2 mm
- net +12V: track 48.5 -> 56.5 mm
Other:
- board size 34 x 44 mm -> 34 x 52 mm

Commit message: Updates kicad data.
Other:
- board text added: "FORT Prometheus rev B ©2018 Université de Lausanne"
- board text removed: "FORT Prometheus rev A ©2018 Université de Lausanne"
Changed lines of the file:
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@@
-(kicad_pcb (version 20171130) (host pcbnew 5.0.0+dfsg1-2~bpo9+1)
+(kicad_pcb (version 20171130) (host pcbnew 5.0.2+dfsg1-1~bpo9+1)
   (general
     (thickness 1.6)
@@
   )
   (setup
-    (last_trace_width 1.5)
+    (last_trace_width 0.5)
     (user_trace_width 0.5)
     (user_trace_width 1.5)
@@
     (pad_drill 0.762)
     (pad_to_mask_clearance 0.2)
+    (solder_mask_min_width 0.25)
     (aux_axis_origin 0 0)
     (visible_elements FFFFFF7F)
@@
       (xy -4.198507 1.271524)) (layer F.SilkS) (width 0.01))
   )
-  (gr_text "FORT Prometheus rev A\n©2018 \nUniversité de Lausanne" (at 120.25 123) (layer F.SilkS)
+  (gr_text "FORT Prometheus rev B\n©2018 \nUniversité de Lausanne" (at 120.25 123) (layer F.SilkS)
     (effects (font (size 1 1) (thickness 0.25)))
   )

Commit message: Updates PCBs
Parts:
- removed G***: LOGO, FORT:UNIL-LOGO_13.8x5.1mm
- removed J5, J6: 5566-02A, Connector_Molex:Molex_Mini-Fit_Jr_5566-02A_2x01_P4.20mm_Vertical
- removed MH1, MH2, MH3, MH4: MountingHole, MountingHole:MountingHole_3.2mm_M3_DIN965
- J2, J3: value 5566-02A -> JST PH; footprint Connector_Molex:Molex_Mini-Fit_Jr_5566-02A_2x01_P4.20mm_Vertical -> FORT:JST_PH_B4B-PH-SM4-TB_1x04-1MP_P2.00mm_Vertical
- J4: value 5566-02A -> Phoenix MCV_1,5; footprint Connector_Molex:Molex_Mini-Fit_Jr_5566-02A_2x01_P4.20mm_Vertical -> Connector_Phoenix_MC:PhoenixContact_MCV_1,5_2-G-3.5_1x02_P3.50mm_Vertical
- REF**: moved to B.Cu
- moved J4 27.6 mm to (106.8, 81.2), turned to -90 degrees
- moved J1 22.1 mm to (133.7, 85.5), turned to -90 degrees
- moved R1 16.1 mm to (107.6, 75.9)
- moved D1 14.8 mm to (107.6, 77.4), turned to 180 degrees
- moved J3 11.2 mm to (124.8, 81.0)
- moved J2 11.1 mm to (116.3, 81.0)
- moved REF** 0.54 mm to (118.5, 83.8), turned to 0 degrees
Connections:
- J4 pad 1: +12V -> GND
- J4 pad 2: GND -> +12V
Routing:
- net GND: track 88.2 -> 34.8 mm
- net +12V: track 56.5 -> 70.8 mm
- net /CAN-: track 0.00 -> 9.23 mm
- net /CAN+: track 0.00 -> 9.23 mm
- removed copper zone on F.Cu, net GND
Other:
- board size 34 x 52 mm -> 36 x 14 mm
- net class Default removed
- rule pad_to_mask_clearance: 0.2 -> 0
- board text added: "FORT Prometheus rev C ©2018 UNIL ©2024 UNIGE"
- board text removed: "FORT Prometheus rev B ©2018 Université de Lausanne"
