File: ecad/climate/arke/UC.sch (KiCad schematic (older format))
At the start: 18 parts, among them J4 M20-8760342, SW1 1825910-6, U2 ATMEGA16M1-AU, Y1 16MHz

Commit message: Updates Arke to KiCad 5
Parts:
- C10, C11, C7, C8, C9: footprint Capacitors_SMD:C_0603 -> Capacitor_SMD:C_0603_1608Metric; symbol C -> Device:C
- D1, D2, D3: footprint LEDs:LED_0603 -> LED_SMD:LED_0603_1608Metric; symbol LED -> Device:LED
- D4: footprint Diodes_SMD:D_SOT-23_ANK -> Diode_SMD:D_SOT-23_ANK; symbol D_Schottky -> Device:D_Schottky
- J4: footprint Pin_Headers:Pin_Header_Straight_2x03_Pitch2.54mm_SMD -> Connector_PinHeader_2.54mm:PinHeader_2x03_P2.54mm_Vertical_SMD; symbol Conn_02x03_Odd_Even -> Connector_Generic:Conn_02x03_Odd_Even
- R1, R2, R3, R4, R5: footprint Resistors_SMD:R_0603 -> Resistor_SMD:R_0603_1608Metric; symbol R -> Device:R
- SW1: footprint Buttons_Switches_THT:SW_PUSH_6mm -> Button_Switch_THT:SW_PUSH_6mm; symbol SW_Push -> Switch:SW_Push
- U2: footprint Housings_QFP:TQFP-32_7x7mm_Pitch0.8mm -> Package_QFP:TQFP-32_7x7mm_P0.8mm; symbol ATMEGA16M1-AU -> MCU_Microchip_ATmega:ATmega16M1-AU
- Y1: footprint Crystals:Crystal_SMD_SeikoEpson_FA238-4pin_3.2x2.5mm -> Crystal:Crystal_SMD_SeikoEpson_FA238-4Pin_3.2x2.5mm; symbol Crystal_GND24 -> Device:Crystal_GND24
Connections:
- net GND: now also R4.1; no longer R4.2
- net GNDA: now also R4.2; no longer R4.1
Other:
- moved on the sheet: C10, C11, C7, C8, C9, D4, J4, R1, R2, R3, R4, R5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

Commit message: Licenses Climate PCB under OHL v1.2
Other:
- note added: "© 2018 Université de Lausanne\n\nThis documentation describes Open Hardware and is licensed under the\nCERN OHL v. 1.2.\n\nYou may redistribute and modify this documentation under the terms of\nthe CERN OHL v.1.2. (http://ohwr.org/cernohl). This documentation is\ndistributed WITHOUT ANY EXPRESS OR IMPLIED WARRANTY,\nINCLUDING OF MERCHANTABILITY, SATISFACTORY QUALITY AND\nFITNESS FOR A PARTICULAR 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"
Changed lines of the file:
@@
 encoding utf-8
 Sheet 3 5
-Title ""
-Date ""
-Rev ""
-Comp ""
-Comment1 ""
-Comment2 ""
+Title "ATMega16M1 SLCAN Transceiver"
+Date "06/11/2018"
+Rev "A"
+Comp "Université de Lausanne"
+Comment1 "Author: Alexandre Tuleu"
+Comment2 "Licensed under the CERN OHL v1.2"
 Comment3 ""
 Comment4 ""
@@
 Wire Wire Line
 	4100 1700 5700 1700
+Text Notes 550  7750 0    50   ~ 0
+© 2018 Université de Lausanne\n\nThis documentation describes Open Hardware and is licensed under the\nCERN OHL v. 1.2.\n\nYou may redistribute and modify this documentation under the terms of\nthe CERN OHL v.1.2. (http://ohwr.org/cernohl). This documentation is\ndistributed WITHOUT ANY EXPRESS OR IMPLIED WARRANTY,\nINCLUDING OF MERCHANTABILITY, SATISFACTORY QUALITY AND\nFITNESS FOR A PARTICULAR PURPOSE. Please see the CERN OHL v.1.2\nfor applicable conditions
 $EndSCHEMATC

Commit message: Makes all electronics production ready
Parts:
- C10, C11: Part Number C0603C180K5GACTU -> GP0603180
- C7, C8, C9: Part Number CC0603KRX7R8BB104 -> GPC0603104
- R1, R2, R3: Part Number RMCF0603FT1K00 -> GPR06031k
- R5: Part Number RMCF0603FT100K -> GPR0603100k
Changed lines of the file:
@@
 F 2 "Capacitor_SMD:C_0603_1608Metric" H 4138 1750 50  0001 C CNN
 F 3 "" H 4100 1900 50  0001 C CNN
-F 4 "CC0603KRX7R8BB104" H 4100 1900 60  0001 C CNN "Part Number"
+F 4 "GPC0603104" H 4100 1900 60  0001 C CNN "Part Number"
 	1    4100 1900
 	1    0    0    -1
@@
 F 2 "Capacitor_SMD:C_0603_1608Metric" H 4438 2050 50  0001 C CNN
 F 3 "" H 4400 2200 50  0001 C CNN
-F 4 "CC0603KRX7R8BB104" H 4400 2200 60  0001 C CNN "Part Number"
+F 4 "GPC0603104" H 4400 2200 60  0001 C CNN "Part Number"
 	1    4400 2200
 	1    0    0    -1
@@
 F 2 "Capacitor_SMD:C_0603_1608Metric" H 4688 2450 50  0001 C CNN
 F 3 "" H 4650 2600 50  0001 C CNN
-F 4 "CC0603KRX7R8BB104" H 4650 2600 60  0001 C CNN "Part Number"
+F 4 "GPC0603104" H 4650 2600 60  0001 C CNN "Part Number"
 	1    4650 2600
 	1    0    0    -1
@@
 F 2 "Capacitor_SMD:C_0603_1608Metric" H 8438 4700 50  0001 C CNN
 F 3 "" H 8400 4850 50  0001 C CNN
-F 4 "C0603C180K5GACTU" H 8400 4850 60  0001 C CNN "Part Number"
+F 4 "GP0603180" H 8400 4850 60  0001 C CNN "Part Number"
 	1    8400 4850
 	0    1    1    0
@@
 F 2 "Capacitor_SMD:C_0603_1608Metric" H 8438 5500 50  0001 C CNN
 F 3 "" H 8400 5650 50  0001 C CNN
-F 4 "C0603C180K5GACTU" H 8400 5650 60  0001 C CNN "Part Number"
+F 4 "GP0603180" H 8400 5650 60  0001 C CNN "Part Number"
 	1    8400 5650
 	0    1    1    0
@@
 F 2 "Resistor_SMD:R_0603_1608Metric" V 9980 5100 50  0001 C CNN
 F 3 "" H 10050 5100 50  0001 C CNN
-F 4 "RMCF0603FT100K" H 10050 5100 60  0001 C CNN "Part Number"
+F 4 "GPR0603100k" H 10050 5100 60  0001 C CNN "Part Number"
 	1    10050 5100
 	1    0    0    -1
@@
 F 2 "Resistor_SMD:R_0603_1608Metric" V 8680 2500 50  0001 C CNN
 F 3 "" H 8750 2500 50  0001 C CNN
-F 4 "RMCF0603FT1K00" H 8750 2500 60  0001 C CNN "Part Number"
+F 4 "GPR06031k" H 8750 2500 60  0001 C CNN "Part Number"
 	1    8750 2500
 	0    1    1    0
@@
 F 2 "Resistor_SMD:R_0603_1608Metric" V 8680 2850 50  0001 C CNN
 F 3 "" H 8750 2850 50  0001 C CNN
-F 4 "RMCF0603FT1K00" H 8750 2850 60  0001 C CNN "Part Number"
+F 4 "GPR06031k" H 8750 2850 60  0001 C CNN "Part Number"
 	1    8750 2850
 	0    1    1    0
@@
 F 2 "Resistor_SMD:R_0603_1608Metric" V 8680 3200 50  0001 C CNN
 F 3 "" H 8750 3200 50  0001 C CNN
-F 4 "RMCF0603FT1K00" H 8750 3200 60  0001 C CNN "Part Number"
+F 4 "GPR06031k" H 8750 3200 60  0001 C CNN "Part Number"
 	1    8750 3200
 	0    1    1    0
