File: ecad/climate/arke/rs232_isolator.sch (KiCad schematic (older format))
At the start: 7 parts, among them U1 ADM3251E

Commit message: Updates Arke to KiCad 5
Parts:
- C1, C2, C3, C4, C5, C6: footprint Capacitors_SMD:C_0603 -> Capacitor_SMD:C_0603_1608Metric; symbol C -> Device:C
- U1: footprint Housings_SOIC:SOIC-20W_7.5x12.8mm_Pitch1.27mm -> Package_SO:SOIC-20W_7.5x12.8mm_P1.27mm; symbol ADM3251E -> fort:ADM3251E
Changed lines of the file:
@@
-EESchema Schematic File Version 2
+EESchema Schematic File Version 4
 LIBS:power
-LIBS:device
-LIBS:switches
-LIBS:relays
-LIBS:motors
-LIBS:transistors
-LIBS:conn
-LIBS:linear
-LIBS:regul
 LIBS:74xx
-LIBS:cmos4000
-LIBS:adc-dac
-LIBS:memory
-LIBS:xilinx
-LIBS:microcontrollers
-LIBS:dsp
-LIBS:microchip
-LIBS:analog_switches
-LIBS:motorola
-LIBS:texas
-LIBS:intel
-LIBS:audio
-LIBS:interface
-LIBS:digital-audio
-LIBS:philips
-LIBS:display
-LIBS:cypress
-LIBS:siliconi
-LIBS:opto
-LIBS:atmel
-LIBS:contrib
-LIBS:valves
 LIBS:fort
-LIBS:kerykeion-cache
-EELAYER 25 0
+LIBS:arke-cache
+EELAYER 26 0
 EELAYER END
 $Descr A4 11693 8268
@@
 $EndDescr
 $Comp
-L ADM3251E U1
+L fort:ADM3251E U1
 U 1 1 5BA26332
 P 5300 3700
 F 0 "U1" H 4850 4450 60  0000 C CNN
 F 1 "ADM3251E" H 4900 2950 60  0000 C CNN
-F 2 "Housings_SOIC:SOIC-20W_7.5x12.8mm_Pitch1.27mm" H 4750 4350 60  0001 C CNN
+F 2 "Package_SO:SOIC-20W_7.5x12.8mm_P1.27mm" H 4750 4350 60  0001 C CNN
 F 3 "" H 4850 4450 60  0001 C CNN
 F 4 "ADM3251E" H 4950 4550 60  0001 C CNN "Part Number"
@@
 	4150 3800 4600 3800
 $Comp
-L GND #PWR05
+L power:GND #PWR05
 U 1 1 5BA263FA
 P 5150 4800
@@
 	5150 4800 5150 4600
 $Comp
-L C C1
+L Device:C C1
 U 1 1 5BA26629
 P 4400 2950
 F 0 "C1" H 4425 3050 50  0000 L CNN
 F 1 "100n" H 4425 2850 50  0000 L CNN
-F 2 "Capacitors_SMD:C_0603" H 4438 2800 50  0001 C CNN
+F 2 "Capacitor_SMD:C_0603_1608Metric" H 4438 2800 50  0001 C CNN
 F 3 "" H 4400 2950 50  0001 C CNN
 F 4 "CC0603KRX7R8BB104" H 4400 2950 60  0001 C CNN "Part Number"
@@
 $EndComp
 $Comp
-L GND #PWR06
+L power:GND #PWR06
 U 1 1 5BA26630
 P 4400 3200
@@
 	4400 3200 4400 3100
 $Comp
-L C C2
+L Device:C C2
 U 1 1 5BA26706
 P 6400 3100
 F 0 "C2" V 6450 3150 50  0000 L CNN
 F 1 "100n" V 6450 2850 50  0000 L CNN
-F 2 "Capacitors_SMD:C_0603" H 6438 2950 50  0001 C CNN
+F 2 "Capacitor_SMD:C_0603_1608Metric" H 6438 2950 50  0001 C CNN
 F 3 "" H 6400 3100 50  0001 C CNN
 F 4 "CC0603KRX7R8BB104" H 6400 3100 60  0001 C CNN "Part Number"
@@
 $EndComp
 $Comp
-L C C5
+L Device:C C5
 U 1 1 5BA268C2
 P 6400 3300
 F 0 "C5" V 6450 3350 50  0000 L CNN
 F 1 "100n" V 6450 3050 50  0000 L CNN
-F 2 "Capacitors_SMD:C_0603" H 6438 3150 50  0001 C CNN
+F 2 "Capacitor_SMD:C_0603_1608Metric" H 6438 3150 50  0001 C CNN
 F 3 "" H 6400 3300 50  0001 C CNN
 F 4 "CC0603KRX7R8BB104" H 6400 3300 60  0001 C CNN "Part Number"
@@
 	6700 3300 6550 3300
 $Comp
-L C C3
+L Device:C C3
 U 1 1 5BA26B07
 P 7050 3200
 F 0 "C3" H 7075 3300 50  0000 L CNN
 F 1 "100n" H 7075 3100 50  0000 L CNN
-F 2 "Capacitors_SMD:C_0603" H 7088 3050 50  0001 C CNN
+F 2 "Capacitor_SMD:C_0603_1608Metric" H 7088 3050 50  0001 C CNN
 F 3 "" H 7050 3200 50  0001 C CNN
 F 4 "CC0603KRX7R8BB104" H 7050 3200 60  0001 C CNN "Part Number"
@@
 	5450 2800 5450 2750
 Wire Wire Line
-	5450 2750 7400 2750
+	5450 2750 7050 2750
 Wire Wire Line
 	7050 2750 7050 3050
@@
 	7050 3500 7050 3350
 $Comp
-L C C4
+L Device:C C4
 U 1 1 5BA26BE9
 P 7400 3200
 F 0 "C4" H 7425 3300 50  0000 L CNN
 F 1 "100n" H 7425 3100 50  0000 L CNN
-F 2 "Capacitors_SMD:C_0603" H 7438 3050 50  0001 C CNN
+F 2 "Capacitor_SMD:C_0603_1608Metric" H 7438 3050 50  0001 C CNN
 F 3 "" H 7400 3200 50  0001 C CNN
 F 4 "CC0603KRX7R8BB104" H 7400 3200 60  0001 C CNN "Part Number"
@@
 	7400 3350 7400 4800
 Wire Wire Line
-	5450 4800 7700 4800
+	5450 4800 7050 4800
 Wire Wire Line
 	5450 4800 5450 4600
 $Comp
-L C C6
+L Device:C C6
 U 1 1 5BA26C69
 P 7050 4100
 F 0 "C6" H 7075 4200 50  0000 L CNN
 F 1 "100n" H 7075 4000 50  0000 L CNN
-F 2 "Capacitors_SMD:C_0603" H 7088 3950 50  0001 C CNN
+F 2 "Capacitor_SMD:C_0603_1608Metric" H 7088 3950 50  0001 C CNN
 F 3 "" H 7050 4100 50  0001 C CNN
 F 4 "CC0603KRX7R8BB104" H 7050 4100 60  0001 C CNN "Part Number"
@@
 	4400 2700 5150 2700
 Wire Wire Line
-	5150 2550 5150 2800
-$Comp
-L +5V #PWR07
+	5150 2550 5150 2700
+$Comp
+L power:+5V #PWR07
 U 1 1 5BA26D6E
 P 5150 2550
@@
 GND_ISO
 Connection ~ 7400 4800
+Wire Wire Line
+	7050 2750 7400 2750
+Wire Wire Line
+	7050 4800 7400 4800
+Wire Wire Line
+	5150 2700 5150 2800
+Wire Wire Line
+	7400 4800 7700 4800
 $EndSCHEMATC

Commit message: Licenses Climate PCB under OHL v1.2
Other:
- note added: "© 2018 Université de Lausanne\n\nThis documentation describes Open Hardware and is licensed under the\nCERN OHL v. 1.2.\n\nYou may redistribute and modify this documentation under the terms of\nthe CERN OHL v.1.2. (http://ohwr.org/cernohl). This documentation is\ndistributed WITHOUT ANY EXPRESS OR IMPLIED WARRANTY,\nINCLUDING OF MERCHANTABILITY, SATISFACTORY QUALITY AND\nFITNESS FOR A PARTICULAR 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"
Changed lines of the file:
@@
 encoding utf-8
 Sheet 2 5
-Title ""
-Date ""
-Rev ""
-Comp ""
-Comment1 ""
-Comment2 ""
+Title "RS232 Isolator"
+Date "06/11/2018"
+Rev "A"
+Comp "Université de Lausanne"
+Comment1 "Author: Alexandre Tuleu"
+Comment2 "Licensed under the CERN OHL v1.2"
 Comment3 ""
 Comment4 ""
@@
 Wire Wire Line
 	7400 4800 7700 4800
+Text Notes 550  7750 0    50   ~ 0
+© 2018 Université de Lausanne\n\nThis documentation describes Open Hardware and is licensed under the\nCERN OHL v. 1.2.\n\nYou may redistribute and modify this documentation under the terms of\nthe CERN OHL v.1.2. (http://ohwr.org/cernohl). This documentation is\ndistributed WITHOUT ANY EXPRESS OR IMPLIED WARRANTY,\nINCLUDING OF MERCHANTABILITY, SATISFACTORY QUALITY AND\nFITNESS FOR A PARTICULAR PURPOSE. Please see the CERN OHL v.1.2\nfor applicable conditions
 $EndSCHEMATC

Commit message: Makes all electronics production ready
Parts:
- C1, C2, C3, C4, C5, C6: Part Number CC0603KRX7R8BB104 -> GPC0603104
Changed lines of the file:
@@
 F 2 "Capacitor_SMD:C_0603_1608Metric" H 4438 2800 50  0001 C CNN
 F 3 "" H 4400 2950 50  0001 C CNN
-F 4 "CC0603KRX7R8BB104" H 4400 2950 60  0001 C CNN "Part Number"
+F 4 "GPC0603104" H 4400 2950 60  0001 C CNN "Part Number"
 	1    4400 2950
 	1    0    0    -1
@@
 F 2 "Capacitor_SMD:C_0603_1608Metric" H 6438 2950 50  0001 C CNN
 F 3 "" H 6400 3100 50  0001 C CNN
-F 4 "CC0603KRX7R8BB104" H 6400 3100 60  0001 C CNN "Part Number"
+F 4 "GPC0603104" H 6400 3100 60  0001 C CNN "Part Number"
 	1    6400 3100
 	0    -1   -1   0
@@
 F 2 "Capacitor_SMD:C_0603_1608Metric" H 6438 3150 50  0001 C CNN
 F 3 "" H 6400 3300 50  0001 C CNN
-F 4 "CC0603KRX7R8BB104" H 6400 3300 60  0001 C CNN "Part Number"
+F 4 "GPC0603104" H 6400 3300 60  0001 C CNN "Part Number"
 	1    6400 3300
 	0    -1   -1   0
@@
 F 2 "Capacitor_SMD:C_0603_1608Metric" H 7088 3050 50  0001 C CNN
 F 3 "" H 7050 3200 50  0001 C CNN
-F 4 "CC0603KRX7R8BB104" H 7050 3200 60  0001 C CNN "Part Number"
+F 4 "GPC0603104" H 7050 3200 60  0001 C CNN "Part Number"
 	1    7050 3200
 	1    0    0    -1
@@
 F 2 "Capacitor_SMD:C_0603_1608Metric" H 7438 3050 50  0001 C CNN
 F 3 "" H 7400 3200 50  0001 C CNN
-F 4 "CC0603KRX7R8BB104" H 7400 3200 60  0001 C CNN "Part Number"
+F 4 "GPC0603104" H 7400 3200 60  0001 C CNN "Part Number"
 	1    7400 3200
 	1    0    0    -1
@@
 F 2 "Capacitor_SMD:C_0603_1608Metric" H 7088 3950 50  0001 C CNN
 F 3 "" H 7050 4100 50  0001 C CNN
-F 4 "CC0603KRX7R8BB104" H 7050 4100 60  0001 C CNN "Part Number"
+F 4 "GPC0603104" H 7050 4100 60  0001 C CNN "Part Number"
 	1    7050 4100
 	1    0    0    -1
