File: ecad/misc/schmitt-trigger-test/schmitt-trigger-test.kicad_pcb (KiCad board)
At the start: 2 copper layers, 4 parts, among them J1 Conn_01x03, J2 Conn_01x03, U1 74LVC1G17

Commit message: Makes all electronics production ready
Parts:
- added C2: 1nF, Capacitor_SMD:C_0603_1608Metric_Pad1.05x0.95mm_HandSolder, F.Cu at (150.6, 99.0)
- added D1: 1N4148WS, Diode_SMD:D_SOD-323, F.Cu at (147.2, 97.2)
- added R1: 10k, Resistor_SMD:R_0603_1608Metric, F.Cu at (150.6, 95.6)
- added R2: 10k, Resistor_SMD:R_0603_1608Metric, F.Cu at (149.0, 97.2)
- moved J1 2.60 mm to (142.4, 94.5)
Connections:
- net Net-(J2-Pad2) renamed /Filtered
- J1 pad 2: Net-(J1-Pad2) -> /RAW
- U1 pad 2: Net-(J1-Pad2) -> Net-(C2-Pad1)
Routing:
- net GND: track 53.0 -> 38.0 mm
- net /RAW: track 0.00 -> 9.13 mm
- net Net-(J1-Pad2): track 8.65 -> 0.00 mm
- net Net-(C2-Pad1): track 0.00 -> 6.67 mm
- net VCC: track 26.2 -> 28.8 mm
Other:
- board text added: "< Fgbber"
- board text added: "Helios >"
