File: ecad/misc/schmitt-trigger-test/schmitt-trigger-test.sch (KiCad schematic (older format))
At the start: 4 parts, among them J1 Conn_01x03, J2 Conn_01x03, U1 74LVC1G17

Commit message: Makes all electronics production ready
Parts:
- added C2: 1nF, Capacitor_SMD:C_0603_1608Metric_Pad1.05x0.95mm_HandSolder, symbol Device:C
- added D1: 1N4148WS, Diode_SMD:D_SOD-323, symbol Diode:1N4148WS
- added R1, R2: 10k, Resistor_SMD:R_0603_1608Metric, symbol Device:R
Connections:
- net labels added: Filtered, RAW
- wire segments 12 -> 26
Changed lines of the file:
@@
 EESchema Schematic File Version 4
+LIBS:schmitt-trigger-test-cache
 EELAYER 26 0
 EELAYER END
@@
 L Connector_Generic:Conn_01x03 J1
 U 1 1 5BFD5FA3
-P 3450 3650
-F 0 "J1" H 3370 3967 50  0000 C CNN
-F 1 "Conn_01x03" H 3370 3876 50  0000 C CNN
-F 2 "Connector_Phoenix_MC:PhoenixContact_MCV_1,5_3-G-3.5_1x03_P3.50mm_Vertical" H 3450 3650 50  0001 C CNN
-F 3 "~" H 3450 3650 50  0001 C CNN
-	1    3450 3650
+P 2550 3650
+F 0 "J1" H 2470 3967 50  0000 C CNN
+F 1 "Conn_01x03" H 2470 3876 50  0000 C CNN
+F 2 "Connector_Phoenix_MC:PhoenixContact_MCV_1,5_3-G-3.5_1x03_P3.50mm_Vertical" H 2550 3650 50  0001 C CNN
+F 3 "~" H 2550 3650 50  0001 C CNN
+	1    2550 3650
 	-1   0    0    -1
 $EndComp
@@
 L power:VCC #PWR0105
 U 1 1 5BFD6442
-P 3950 3350
-F 0 "#PWR0105" H 3950 3200 50  0001 C CNN
-F 1 "VCC" H 3967 3523 50  0000 C CNN
-F 2 "" H 3950 3350 50  0001 C CNN
-F 3 "" H 3950 3350 50  0001 C CNN
-	1    3950 3350
-	1    0    0    -1
-$EndComp
-Wire Wire Line
-	3950 3350 3950 3550
-Wire Wire Line
-	3950 3550 3650 3550
+P 3050 3350
+F 0 "#PWR0105" H 3050 3200 50  0001 C CNN
+F 1 "VCC" H 3067 3523 50  0000 C CNN
+F 2 "" H 3050 3350 50  0001 C CNN
+F 3 "" H 3050 3350 50  0001 C CNN
+	1    3050 3350
+	1    0    0    -1
+$EndComp
+Wire Wire Line
+	3050 3350 3050 3550
+Wire Wire Line
+	3050 3550 2750 3550
 $Comp
 L power:GND #PWR0106
 U 1 1 5BFD64B0
-P 4000 3850
-F 0 "#PWR0106" H 4000 3600 50  0001 C CNN
-F 1 "GND" H 4005 3677 50  0000 C CNN
-F 2 "" H 4000 3850 50  0001 C CNN
-F 3 "" H 4000 3850 50  0001 C CNN
-	1    4000 3850
-	1    0    0    -1
-$EndComp
-Wire Wire Line
-	3650 3750 4000 3750
-Wire Wire Line
-	4000 3750 4000 3850
-Wire Wire Line
-	3650 3650 5050 3650
+P 3100 3850
+F 0 "#PWR0106" H 3100 3600 50  0001 C CNN
+F 1 "GND" H 3105 3677 50  0000 C CNN
+F 2 "" H 3100 3850 50  0001 C CNN
+F 3 "" H 3100 3850 50  0001 C CNN
+	1    3100 3850
+	1    0    0    -1
+$EndComp
+Wire Wire Line
+	2750 3750 3100 3750
+Wire Wire Line
+	3100 3750 3100 3850
+Wire Wire Line
+	2750 3650 3950 3650
 Wire Wire Line
 	5600 3650 6900 3650
+Text Label 3000 3650 0    50   ~ 0
+RAW
+Text Label 5650 3650 0    50   ~ 0
+Filtered
+$Comp
+L Diode:1N4148WS D1
+U 1 1 5C0FDD66
+P 4300 3300
+F 0 "D1" H 4300 3083 50  0000 C CNN
+F 1 "1N4148WS" H 4300 3174 50  0000 C CNN
+F 2 "Diode_SMD:D_SOD-323" H 4300 3125 50  0001 C CNN
+F 3 "https://www.vishay.com/docs/85751/1n4148ws.pdf" H 4300 3300 50  0001 C CNN
+	1    4300 3300
+	-1   0    0    1
+$EndComp
+$Comp
+L Device:C C2
+U 1 1 5C0FDE2D
+P 4700 3900
+F 0 "C2" H 4815 3946 50  0000 L CNN
+F 1 "1nF" H 4815 3855 50  0000 L CNN
+F 2 "Capacitor_SMD:C_0603_1608Metric_Pad1.05x0.95mm_HandSolder" H 4738 3750 50  0001 C CNN
+F 3 "~" H 4700 3900 50  0001 C CNN
+	1    4700 3900
+	1    0    0    -1
+$EndComp
+$Comp
+L Device:R R1
+U 1 1 5C0FDEB2
+P 3950 2950
+F 0 "R1" H 4020 2996 50  0000 L CNN
+F 1 "10k" H 4020 2905 50  0000 L CNN
+F 2 "Resistor_SMD:R_0603_1608Metric" V 3880 2950 50  0001 C CNN
+F 3 "~" H 3950 2950 50  0001 C CNN
+	1    3950 2950
+	1    0    0    -1
+$EndComp
+$Comp
+L Device:R R2
+U 1 1 5C0FDF1B
+P 4300 3650
+F 0 "R2" V 4093 3650 50  0000 C CNN
+F 1 "10k" V 4184 3650 50  0000 C CNN
+F 2 "Resistor_SMD:R_0603_1608Metric" V 4230 3650 50  0001 C CNN
+F 3 "~" H 4300 3650 50  0001 C CNN
+	1    4300 3650
+	0    1    1    0
+$EndComp
+Wire Wire Line
+	3950 3100 3950 3300
+Connection ~ 3950 3650
+Wire Wire Line
+	3950 3650 4150 3650
+$Comp
+L power:VCC #PWR01
+U 1 1 5C0FE4A2
+P 3950 2500
+F 0 "#PWR01" H 3950 2350 50  0001 C CNN
+F 1 "VCC" H 3967 2673 50  0000 C CNN
+F 2 "" H 3950 2500 50  0001 C CNN
+F 3 "" H 3950 2500 50  0001 C CNN
+	1    3950 2500
+	1    0    0    -1
+$EndComp
+Wire Wire Line
+	3950 2500 3950 2800
+Wire Wire Line
+	3950 3300 4150 3300
+Connection ~ 3950 3300
+Wire Wire Line
+	3950 3300 3950 3650
+Wire Wire Line
+	4450 3300 4700 3300
+Wire Wire Line
+	4700 3300 4700 3450
+Wire Wire Line
+	4450 3650 4700 3650
+Connection ~ 4700 3650
+Wire Wire Line
+	4700 3650 4700 3750
+Wire Wire Line
+	4700 3450 4850 3450
+Wire Wire Line
+	4850 3450 4850 3650
+Wire Wire Line
+	4850 3650 5050 3650
+Connection ~ 4700 3450
+Wire Wire Line
+	4700 3450 4700 3650
+$Comp
+L power:GND #PWR02
+U 1 1 5C0FECB3
+P 4700 4100
+F 0 "#PWR02" H 4700 3850 50  0001 C CNN
+F 1 "GND" H 4705 3927 50  0000 C CNN
+F 2 "" H 4700 4100 50  0001 C CNN
+F 3 "" H 4700 4100 50  0001 C CNN
+	1    4700 4100
+	1    0    0    -1
+$EndComp
+Wire Wire Line
+	4700 4100 4700 4050
 $EndSCHEMATC
