File: ecad/climate/notus/notus.sch (KiCad schematic (older format))
At the start: 5 parts, among them J1 640454-2

Commit message: Updates ecad for assembly production
Parts:
- removed D1: 1N4001, Diode_THT:D_DO-41_SOD81_P10.16mm_Horizontal, symbol Diode:1N4001
- added J2: 6410-02A, Connector_Molex:Molex_KK-254_AE-6410-02A_1x02_P2.54mm_Vertical, symbol Connector_Generic:Conn_01x02
- added MH3, MH4: MountingHole, MountingHole:MountingHole_4.3mm_M4_DIN965, symbol Mechanical:MountingHole
- added R2, R3: 20R, 20W, Resistor_THT:R_Axial_Power_L60.0mm_W14.0mm_P71.12mm, symbol Device:Heater
- added R4: 10R, 20W, Resistor_THT:R_Axial_Power_L60.0mm_W14.0mm_P71.12mm, symbol Device:Heater
- J1: value 640454-2 -> 6410-02A; footprint FORT:640454-2 -> Connector_Molex:Molex_KK-254_AE-6410-02A_1x02_P2.54mm_Vertical; Part Number 640454-2 -> 22-27-2021
Connections:
- net labels added: GNDA, PWM_A, PWM_B
- net labels removed: PWM_+
- wire segments 14 -> 26
Changed lines of the file:
@@
 EESchema Schematic File Version 4
+LIBS:notus-cache
 EELAYER 26 0
 EELAYER END
@@
 L Device:Heater R1
 U 1 1 5BF5BA91
-P 5450 3700
-F 0 "R1" V 5600 3600 50  0000 L CNN
-F 1 "10R, 20W" V 5300 3550 50  0000 L CNN
-F 2 "Resistor_THT:R_Axial_Power_L60.0mm_W14.0mm_P71.12mm" V 5380 3700 50  0001 C CNN
-F 3 "~" H 5450 3700 50  0001 C CNN
-F 4 "SQP20AJB-10R" H 5450 3700 50  0001 C CNN "Part Number"
-	1    5450 3700
+P 3800 3700
+F 0 "R1" V 3950 3600 50  0000 L CNN
+F 1 "10R, 20W" V 3650 3550 50  0000 L CNN
+F 2 "Resistor_THT:R_Axial_Power_L60.0mm_W14.0mm_P71.12mm" V 3730 3700 50  0001 C CNN
+F 3 "~" H 3800 3700 50  0001 C CNN
+F 4 "SQP20AJB-10R" H 3800 3700 50  0001 C CNN "Part Number"
+	1    3800 3700
 	0    1    1    0
 $EndComp
@@
 L Connector_Generic:Conn_01x02 J1
 U 1 1 5BF692D0
-P 4400 3700
-F 0 "J1" H 4400 3450 50  0000 C CNN
-F 1 "640454-2" H 4450 3850 50  0000 C CNN
-F 2 "FORT:640454-2" H 4400 3700 50  0001 C CNN
-F 3 "~" H 4400 3700 50  0001 C CNN
-F 4 "640454-2" H 4400 3700 50  0001 C CNN "Part Number"
-	1    4400 3700
+P 2750 3700
+F 0 "J1" H 2750 3450 50  0000 C CNN
+F 1 "6410-02A" H 2800 3850 50  0000 C CNN
+F 2 "Connector_Molex:Molex_KK-254_AE-6410-02A_1x02_P2.54mm_Vertical" H 2750 3700 50  0001 C CNN
+F 3 "~" H 2750 3700 50  0001 C CNN
+F 4 "22-27-2021" H 2750 3700 50  0001 C CNN "Part Number"
+	1    2750 3700
 	-1   0    0    -1
 $EndComp
@@
 L Mechanical:MountingHole MH1
 U 1 1 5BF69646
-P 5600 3100
-F 0 "MH1" H 5700 3146 50  0000 L CNN
-F 1 "MountingHole" H 5700 3055 50  0000 L CNN
-F 2 "MountingHole:MountingHole_4.3mm_M4_DIN965" H 5600 3100 50  0001 C CNN
-F 3 "~" H 5600 3100 50  0001 C CNN
-	1    5600 3100
+P 6500 5500
+F 0 "MH1" H 6600 5546 50  0000 L CNN
+F 1 "MountingHole" H 6600 5455 50  0000 L CNN
+F 2 "MountingHole:MountingHole_4.3mm_M4_DIN965" H 6500 5500 50  0001 C CNN
+F 3 "~" H 6500 5500 50  0001 C CNN
+	1    6500 5500
 	1    0    0    -1
 $EndComp
@@
 L Mechanical:MountingHole MH2
 U 1 1 5BF696E5
-P 5650 4500
-F 0 "MH2" H 5750 4546 50  0000 L CNN
-F 1 "MountingHole" H 5750 4455 50  0000 L CNN
-F 2 "MountingHole:MountingHole_4.3mm_M4_DIN965" H 5650 4500 50  0001 C CNN
-F 3 "~" H 5650 4500 50  0001 C CNN
-	1    5650 4500
-	1    0    0    -1
-$EndComp
-Wire Wire Line
-	4600 3700 5150 3700
-Wire Wire Line
-	5600 3700 5750 3700
-Wire Wire Line
-	5900 4200 4850 4200
-Wire Wire Line
-	4650 4200 4650 3800
-Wire Wire Line
-	4650 3800 4600 3800
-Text Label 4800 3700 0    50   ~ 0
-PWM_+
+P 6500 5250
+F 0 "MH2" H 6600 5296 50  0000 L CNN
+F 1 "MountingHole" H 6600 5205 50  0000 L CNN
+F 2 "MountingHole:MountingHole_4.3mm_M4_DIN965" H 6500 5250 50  0001 C CNN
+F 3 "~" H 6500 5250 50  0001 C CNN
+	1    6500 5250
+	1    0    0    -1
+$EndComp
+Wire Wire Line
+	4250 4200 3200 4200
+Wire Wire Line
+	3000 4200 3000 3800
+Wire Wire Line
+	3000 3800 2950 3800
+Text Label 3150 3700 0    50   ~ 0
+PWM_A
 $Comp
 L power:GND #PWR0101
 U 1 1 5BF6A01B
-P 4850 4350
-F 0 "#PWR0101" H 4850 4100 50  0001 C CNN
-F 1 "GND" H 4855 4177 50  0000 C CNN
-F 2 "" H 4850 4350 50  0001 C CNN
-F 3 "" H 4850 4350 50  0001 C CNN
-	1    4850 4350
-	1    0    0    -1
-$EndComp
-Wire Wire Line
-	4850 4350 4850 4200
-Connection ~ 4850 4200
-Wire Wire Line
-	4850 4200 4650 4200
-Wire Wire Line
-	5900 3700 5900 4200
-$Comp
-L Diode:1N4001 D1
-U 1 1 5BF6C3E1
-P 5450 4050
-F 0 "D1" H 5450 4266 50  0000 C CNN
-F 1 "1N4001" H 5450 4175 50  0000 C CNN
-F 2 "Diode_THT:D_DO-41_SOD81_P10.16mm_Horizontal" H 5450 3875 50  0001 C CNN
-F 3 "http://www.vishay.com/docs/88503/1n4001.pdf" H 5450 4050 50  0001 C CNN
-	1    5450 4050
-	1    0    0    -1
-$EndComp
-Wire Wire Line
-	5300 4050 5150 4050
-Wire Wire Line
-	5150 4050 5150 3700
-Connection ~ 5150 3700
-Wire Wire Line
-	5150 3700 5300 3700
-Wire Wire Line
-	5600 4050 5750 4050
-Wire Wire Line
-	5750 4050 5750 3700
-Connection ~ 5750 3700
-Wire Wire Line
-	5750 3700 5900 3700
+P 3200 4350
+F 0 "#PWR0101" H 3200 4100 50  0001 C CNN
+F 1 "GND" H 3205 4177 50  0000 C CNN
+F 2 "" H 3200 4350 50  0001 C CNN
+F 3 "" H 3200 4350 50  0001 C CNN
+	1    3200 4350
+	1    0    0    -1
+$EndComp
+Wire Wire Line
+	3200 4350 3200 4200
+Connection ~ 3200 4200
+Wire Wire Line
+	3200 4200 3000 4200
+Wire Wire Line
+	4250 3700 4250 4200
+$Comp
+L Mechanical:MountingHole MH4
+U 1 1 5C6B2F1A
+P 7800 5550
+F 0 "MH4" H 7900 5596 50  0000 L CNN
+F 1 "MountingHole" H 7900 5505 50  0000 L CNN
+F 2 "MountingHole:MountingHole_4.3mm_M4_DIN965" H 7800 5550 50  0001 C CNN
+F 3 "~" H 7800 5550 50  0001 C CNN
+	1    7800 5550
+	1    0    0    -1
+$EndComp
+$Comp
+L Mechanical:MountingHole MH3
+U 1 1 5C6B2F58
+P 7800 5250
+F 0 "MH3" H 7900 5296 50  0000 L CNN
+F 1 "MountingHole" H 7900 5205 50  0000 L CNN
+F 2 "MountingHole:MountingHole_4.3mm_M4_DIN965" H 7800 5250 50  0001 C CNN
+F 3 "~" H 7800 5250 50  0001 C CNN
+	1    7800 5250
+	1    0    0    -1
+$EndComp
+Wire Wire Line
+	2950 3700 3500 3700
+Wire Wire Line
+	3950 3700 4250 3700
+$Comp
+L Device:Heater R2
+U 1 1 5C6B2FC0
+P 3800 3350
+F 0 "R2" V 3950 3250 50  0000 L CNN
+F 1 "20R, 20W" V 3650 3200 50  0000 L CNN
+F 2 "Resistor_THT:R_Axial_Power_L60.0mm_W14.0mm_P71.12mm" V 3730 3350 50  0001 C CNN
+F 3 "~" H 3800 3350 50  0001 C CNN
+F 4 "SQP20AJB-10R" H 3800 3350 50  0001 C CNN "Part Number"
+	1    3800 3350
+	0    1    1    0
+$EndComp
+Wire Wire Line
+	3500 3700 3500 3350
+Wire Wire Line
+	3500 3350 3650 3350
+Connection ~ 3500 3700
+Wire Wire Line
+	3500 3700 3650 3700
+Wire Wire Line
+	3950 3350 4250 3350
+Wire Wire Line
+	4250 3350 4250 3700
+Connection ~ 4250 3700
+$Comp
+L Device:Heater R4
+U 1 1 5C6B39CE
+P 6000 3700
+F 0 "R4" V 6150 3600 50  0000 L CNN
+F 1 "10R, 20W" V 5850 3550 50  0000 L CNN
+F 2 "Resistor_THT:R_Axial_Power_L60.0mm_W14.0mm_P71.12mm" V 5930 3700 50  0001 C CNN
+F 3 "~" H 6000 3700 50  0001 C CNN
+F 4 "SQP20AJB-10R" H 6000 3700 50  0001 C CNN "Part Number"
+	1    6000 3700
+	0    1    1    0
+$EndComp
+$Comp
+L Connector_Generic:Conn_01x02 J2
+U 1 1 5C6B39D6
+P 4950 3700
+F 0 "J2" H 4950 3450 50  0000 C CNN
+F 1 "6410-02A" H 5000 3850 50  0000 C CNN
+F 2 "Connector_Molex:Molex_KK-254_AE-6410-02A_1x02_P2.54mm_Vertical" H 4950 3700 50  0001 C CNN
+F 3 "~" H 4950 3700 50  0001 C CNN
+F 4 "22-27-2021" H 4950 3700 50  0001 C CNN "Part Number"
+	1    4950 3700
+	-1   0    0    -1
+$EndComp
+Wire Wire Line
+	6450 4200 5400 4200
+Wire Wire Line
+	5200 4200 5200 3800
+Wire Wire Line
+	5200 3800 5150 3800
+Text Label 5350 3700 0    50   ~ 0
+PWM_B
+Connection ~ 5400 4200
+Wire Wire Line
+	5400 4200 5200 4200
+Wire Wire Line
+	6450 3700 6450 4200
+Wire Wire Line
+	5150 3700 5700 3700
+Wire Wire Line
+	6150 3700 6450 3700
+$Comp
+L Device:Heater R3
+U 1 1 5C6B39EE
+P 6000 3350
+F 0 "R3" V 6150 3250 50  0000 L CNN
+F 1 "20R, 20W" V 5850 3200 50  0000 L CNN
+F 2 "Resistor_THT:R_Axial_Power_L60.0mm_W14.0mm_P71.12mm" V 5930 3350 50  0001 C CNN
+F 3 "~" H 6000 3350 50  0001 C CNN
+F 4 "SQP20AJB-10R" H 6000 3350 50  0001 C CNN "Part Number"
+	1    6000 3350
+	0    1    1    0
+$EndComp
+Wire Wire Line
+	5700 3700 5700 3350
+Wire Wire Line
+	5700 3350 5850 3350
+Connection ~ 5700 3700
+Wire Wire Line
+	5700 3700 5850 3700
+Wire Wire Line
+	6150 3350 6450 3350
+Wire Wire Line
+	6450 3350 6450 3700
+Connection ~ 6450 3700
+$Comp
+L power:GNDA #PWR0102
+U 1 1 5C6AE913
+P 5400 4400
+F 0 "#PWR0102" H 5400 4150 50  0001 C CNN
+F 1 "GNDA" H 5405 4227 50  0000 C CNN
+F 2 "" H 5400 4400 50  0001 C CNN
+F 3 "" H 5400 4400 50  0001 C CNN
+	1    5400 4400
+	1    0    0    -1
+$EndComp
+Wire Wire Line
+	5400 4200 5400 4400
 $EndSCHEMATC
