File: ecad/nyx/micro_coupling_simulation.kicad_sch (KiCad schematic)
At the start: 12 parts

Commit message: Works on faulty simulation
Parts:
- removed V1: VPULSE, symbol Simulation_SPICE:VPULSE
- added R6, R7, R8, R9: 0.150, symbol Device:R
- added V1: VSIN, symbol Simulation_SPICE:VSIN
Connections:
- net GND: now also R7.1, R9.2, V1.2; no longer L1.2, L2.2
- net at L1.1: now also R8.1
- net at L3.2: now also R6.1; no longer L2.1
- new net: L2.2, R7.2
- new net: R8.2, V1.1
- new net: L2.1, R6.2
- new net: L1.2, R9.1
