File: ecad/climate/anemoi/anemoi.kicad_sch (KiCad schematic)
At the start: 15 parts, among them J1 215079-4, SW1 219-3MST, U1 TMP1075DGK, U2 MMA8453Q, U3 HIH6131-021-001

Commit message: WIP
Parts:
- removed C2, C3: 100nF, Capacitors_SMD:C_0603, symbol Device:C
- removed R1, R2, R3: 100K, Resistors_SMD:R_0603, symbol Device:R
- removed SW1: 219-3MST, Buttons_Switches_SMD:SW_DIP_x3_W8.61mm_Slide_LowProfile, symbol Switch:SW_DIP_x03
- removed U1: TMP1075DGK, Housings_SSOP:TSSOP-8_3x3mm_Pitch0.65mm, symbol fort:TMP1075DGK
- removed U2: MMA8453Q, FORT:Freescale_98ASA00063D_3x3mm_Pitch_0.5mm, symbol fort:MMA8453Q
- removed U3: HIH6131-021-001, Housings_SOIC:SOIC-8_3.9x4.9mm_Pitch1.27mm, symbol fort:HIH6131-021-001
- added C1: 100n, Capacitor_SMD:C_0402_1005Metric, symbol Device:C
- added U1: MMA8653FCR1, Package_DFN_QFN:DFN-10_2x2mm_P0.4mm, symbol Sensor_Motion:MMA8653FCR1
- added U2: SHT4x, Sensor_Humidity:Sensirion_DFN-4_1.5x1.5mm_P0.8mm_SHT4x_NoCentralPad, symbol Sensor_Humidity:SHT4x
- C3: renamed from C1; value 4.7uF -> 1u; footprint Capacitors_SMD:C_0603 -> Capacitor_SMD:C_0603_1608Metric
- C4: value 100nF -> 100n; footprint Capacitors_SMD:C_0603 -> Capacitor_SMD:C_0402_1005Metric; now not fitted
- C5, C6: value 100nF -> 100n; footprint Capacitors_SMD:C_0603 -> Capacitor_SMD:C_0402_1005Metric
Connections:
- net VCORE is gone; now on net BYP: C4.1
- net BYP: now also U1.4 (BYP); no longer C6.1
- net GND: now also C1.2, U1.6 (GND), U1.7 (GND), U1.9 (GND), U2.4 (VSS)
- net SCL: now also U1.2 (SCL), U2.2 (SCL)
- net SDA: now also U1.10 (SDA), U2.1 (SDA)
- net +3.3V renamed +3V3
- net +3V3: now also C6.1, C1.1, U1.1 (VDD), U1.8 (VDDIO), U2.3 (VDD)
- no-connect marks 5 -> 2
Other:
- note removed: "Accelerometer"
- note removed: "Temperature"
- note removed: "Temperature and Humidity"
- moved on the sheet: C3, C5, C6, D1, J1

Commit message: Updates PCBs
Parts:
- J1: footprint FORT:Micro-Match_4_TH -> FORT:TE_Micro-MaTch_188275-4_2x02_P1.27mm_Vertical
Changed lines of the file:
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@@
 			)
 		)
-		(property "Footprint" "FORT:Micro-Match_4_TH"
+		(property "Footprint" "FORT:TE_Micro-MaTch_188275-4_2x02_P1.27mm_Vertical"
 			(at 43.18 91.44 0)
 			(effects
